File: Hardware/Board/Raspberry.sch (KiCad schematic (older format))
At the start: 9 parts, among them J6 Raspberry_Pi_2_3, U13 ESP-12F

Commit message: Trennung MCU und Rest, Footprints fast alles zugewiesen, GSM Modul integriert, viel Kleinkram
Parts:
- added D20, D21, D22: B230, Diode_SMD:D_SMB, symbol Diode:B230
- J1: renamed from J?; footprint (none) -> Connector_PinHeader_2.54mm:PinHeader_1x06_P2.54mm_Vertical
- J15: renamed from J?; footprint (none) -> Connector_PinSocket_2.54mm:PinSocket_1x06_P2.54mm_Horizontal
- gave numbers to parts that had none: 2
Connections:
- net +4V: now also D22.1 (K)
- net +5VD: now also D20.2 (A)
- new net: D20.1 (K), D21.2 (A)
- new net: D21.1 (K), D22.2 (A)
Changed lines of the file:
@@
 Connection ~ 7950 1350
 $Comp
-L Connector_Generic:Conn_01x06 J?
+L Connector_Generic:Conn_01x06 J1
 U 1 1 60626CBA
 P 7450 4800
-F 0 "J?" H 7350 5250 50  0000 L CNN
+F 0 "J1" H 7350 5250 50  0000 L CNN
 F 1 "Conn_01x06" H 7250 5150 50  0000 L CNN
-F 2 "" H 7450 4800 50  0001 C CNN
+F 2 "Connector_PinHeader_2.54mm:PinHeader_1x06_P2.54mm_Vertical" H 7450 4800 50  0001 C CNN
 F 3 "~" H 7450 4800 50  0001 C CNN
 	1    7450 4800
@@
 $EndComp
 $Comp
-L Connector_Generic:Conn_01x06 J?
+L Connector_Generic:Conn_01x06 J15
 U 1 1 60626D7E
 P 8400 4800
-F 0 "J?" H 8320 5217 50  0000 C CNN
+F 0 "J15" H 8320 5217 50  0000 C CNN
 F 1 "Conn_01x06" H 8320 5126 50  0000 C CNN
-F 2 "" H 8400 4800 50  0001 C CNN
+F 2 "Connector_PinSocket_2.54mm:PinSocket_1x06_P2.54mm_Horizontal" H 8400 4800 50  0001 C CNN
 F 3 "~" H 8400 4800 50  0001 C CNN
 	1    8400 4800
@@
 $EndComp
 $Comp
-L power:GND #PWR?
+L power:GND #PWR0139
 U 1 1 606274EA
 P 7100 5150
-F 0 "#PWR?" H 7100 4900 50  0001 C CNN
+F 0 "#PWR0139" H 7100 4900 50  0001 C CNN
 F 1 "GND" H 7105 4977 50  0000 C CNN
 F 2 "" H 7100 5150 50  0001 C CNN
@@
 $EndComp
 $Comp
-L stmbl:+4V #PWR?
+L stmbl:+4V #PWR0145
 U 1 1 60627B42
 P 7100 4350
-F 0 "#PWR?" H 7100 4200 50  0001 C CNN
+F 0 "#PWR0145" H 7100 4200 50  0001 C CNN
 F 1 "+4V" H 7115 4523 50  0000 C CNN
 F 2 "" H 7100 4350 50  0001 C CNN
@@
 $EndComp
 $Comp
-L Device:C C?
+L Device:C C88
 U 1 1 60627C50
 P 6550 5300
-F 0 "C?" H 6665 5346 50  0000 L CNN
+F 0 "C88" H 6665 5346 50  0000 L CNN
 F 1 "10u" H 6665 5255 50  0000 L CNN
 F 2 "Capacitor_SMD:C_1210_3225Metric" H 6588 5150 50  0001 C CNN
@@
 $EndComp
 $Comp
-L power:GND #PWR?
+L power:GND #PWR0235
 U 1 1 60627C57
 P 6550 5450
-F 0 "#PWR?" H 6550 5200 50  0001 C CNN
+F 0 "#PWR0235" H 6550 5200 50  0001 C CNN
 F 1 "GND" H 6555 5277 50  0000 C CNN
 F 2 "" H 6550 5450 50  0001 C CNN
@@
 $EndComp
 $Comp
-L Device:C C?
+L Device:C C87
 U 1 1 60628290
 P 6150 5300
-F 0 "C?" H 6265 5346 50  0000 L CNN
+F 0 "C87" H 6265 5346 50  0000 L CNN
 F 1 "10u" H 6265 5255 50  0000 L CNN
 F 2 "Capacitor_SMD:C_1210_3225Metric" H 6188 5150 50  0001 C CNN
@@
 $EndComp
 $Comp
-L power:GND #PWR?
+L power:GND #PWR0236
 U 1 1 60628297
 P 6150 5450
-F 0 "#PWR?" H 6150 5200 50  0001 C CNN
+F 0 "#PWR0236" H 6150 5200 50  0001 C CNN
 F 1 "GND" H 6155 5277 50  0000 C CNN
 F 2 "" H 6150 5450 50  0001 C CNN
@@
 Text Notes 7650 4650 0    50   ~ 0
 SIM800L Modul\n
+$Comp
+L power:+5VD #PWR0372
+U 1 1 5D9A02CF
+P 7300 5750
+F 0 "#PWR0372" H 7300 5600 50  0001 C CNN
+F 1 "+5VD" H 7315 5923 50  0000 C CNN
+F 2 "" H 7300 5750 50  0001 C CNN
+F 3 "" H 7300 5750 50  0001 C CNN
+	1    7300 5750
+	1    0    0    -1
+$EndComp
+$Comp
+L Diode:B230 D20
+U 1 1 5D9A0C60
+P 7650 5800
+F 0 "D20" H 7650 5584 50  0000 C CNN
+F 1 "B230" H 7650 5675 50  0000 C CNN
+F 2 "Diode_SMD:D_SMB" H 7650 5625 50  0001 C CNN
+F 3 "http://www.jameco.com/Jameco/Products/ProdDS/1538777.pdf" H 7650 5800 50  0001 C CNN
+	1    7650 5800
+	-1   0    0    1
+$EndComp
+$Comp
+L Diode:B230 D21
+U 1 1 5D9A0DCB
+P 7950 5800
+F 0 "D21" H 7950 5584 50  0000 C CNN
+F 1 "B230" H 7950 5675 50  0000 C CNN
+F 2 "Diode_SMD:D_SMB" H 7950 5625 50  0001 C CNN
+F 3 "http://www.jameco.com/Jameco/Products/ProdDS/1538777.pdf" H 7950 5800 50  0001 C CNN
+	1    7950 5800
+	-1   0    0    1
+$EndComp
+$Comp
+L Diode:B230 D22
+U 1 1 5D9A175A
+P 8250 5800
+F 0 "D22" H 8250 5584 50  0000 C CNN
+F 1 "B230" H 8250 5675 50  0000 C CNN
+F 2 "Diode_SMD:D_SMB" H 8250 5625 50  0001 C CNN
+F 3 "http://www.jameco.com/Jameco/Products/ProdDS/1538777.pdf" H 8250 5800 50  0001 C CNN
+	1    8250 5800
+	-1   0    0    1
+$EndComp
+$Comp
+L stmbl:+4V #PWR0373
+U 1 1 5D9A20CD
+P 8550 5750
+F 0 "#PWR0373" H 8550 5600 50  0001 C CNN
+F 1 "+4V" H 8565 5923 50  0000 C CNN
+F 2 "" H 8550 5750 50  0001 C CNN
+F 3 "" H 8550 5750 50  0001 C CNN
+	1    8550 5750
+	1    0    0    -1
+$EndComp
+Wire Wire Line
+	7500 5800 7300 5800
+Wire Wire Line
+	7300 5800 7300 5750
+Wire Wire Line
+	8400 5800 8550 5800
+Wire Wire Line
+	8550 5800 8550 5750
 $EndSCHEMATC

Commit message: Footprints zuweisungen
Parts:
- J15: footprint Connector_PinSocket_2.54mm:PinSocket_1x06_P2.54mm_Horizontal -> Connector_PinSocket_2.54mm:PinSocket_1x06_P2.54mm_Vertical
Changed lines of the file:
@@
 F 0 "J15" H 8320 5217 50  0000 C CNN
 F 1 "Conn_01x06" H 8320 5126 50  0000 C CNN
-F 2 "Connector_PinSocket_2.54mm:PinSocket_1x06_P2.54mm_Horizontal" H 8400 4800 50  0001 C CNN
+F 2 "Connector_PinSocket_2.54mm:PinSocket_1x06_P2.54mm_Vertical" H 8400 4800 50  0001 C CNN
 F 3 "~" H 8400 4800 50  0001 C CNN
 	1    8400 4800

Commit message: Komplete enummerierung Geändert, Schaltplan zusammengefasst, Layout nochmals reset. BOM zu 75% fertig gestellt
Parts:
- removed C58: 47u, Capacitor_SMD:C_1210_3225Metric, symbol Device:C
- removed C59, C60, C87, C88: 10u, Capacitor_SMD:C_1210_3225Metric, symbol Device:C
- removed D20, D21, D22: B230, Diode_SMD:D_SMB, symbol Diode:B230
- removed J1: Conn_01x06, Connector_PinHeader_2.54mm:PinHeader_1x06_P2.54mm_Vertical, symbol Connector_Generic:Conn_01x06
- removed J15: Conn_01x06, Connector_PinSocket_2.54mm:PinSocket_1x06_P2.54mm_Vertical, symbol Connector_Generic:Conn_01x06
- removed J6: Raspberry_Pi_2_3, Connector_IDC:IDC-Header_2x20_P2.54mm_Vertical, symbol Connector:Raspberry_Pi_2_3
- removed U13: ESP-12F, RF_Module:ESP-12E, symbol RF_Module:ESP-12F
Other:
- note removed: "SIM800L Modul\n"
