File: Hardware/Board/IO.sch (KiCad schematic (older format))
At the start: 86 parts, among them U200 TJA1029T, U201 TJA1029T, U202 TJA1029T, U203 TJA1049T-3, U204 MAX3072E, U205 DS2482S-800+, U206 PCF8574A, U207 PCF8574A, U208 MAX11615

Commit message: Alle Busse aus dem Prozessor geroutet, Multplexing der LIN, RS485 und TTY Busse, diverse Aufräumarbeiten.
Parts:
- added C? (x3): 100nF, Capacitor_SMD:C_0603_1608Metric, symbol Device:C
- added D? (x3): NUP2105L, Package_TO_SOT_SMD:SOT-23, symbol Device:D_TVS_x2_AAC
- added D? (x2): SP0504BAJT, Package_TO_SOT_SMD:SOT-353_SC-70-5, symbol Power_Protection:SP0504BAJT
- added FB? (x14): 100R, Inductor_SMD:L_0603_1608Metric, symbol Device:Ferrite_Bead_Small
- added R? (x3): 120R, Resistor_SMD:R_0603_1608Metric, symbol Device:R
- added R? (x6): 10R, Resistor_SMD:R_0603_1608Metric, symbol Device:R
- added U? (x3): MAX3072E, Package_SO:SOIC-8_3.9x4.9mm_P1.27mm, symbol Interface_UART:MAX3072E
- added U?: 4052, symbol 4xxx_IEEE:4052
Connections:
- net +3V3: now also C?.2, C?.2, C?.2, U?.8 (VCC), U?.8 (VCC), U?.8 (VCC)
- net GND: now also U?.15 (GND2), U?.15 (GND2), U?.2 (GND1), U?.2 (GND1), U?.8 (GND1), U?.8 (GND1), U?.9 (GND2), U?.9 (GND2), C?.1, C?.1, C?.1, D?.2 (A), D?.2 (A), D?.3 (common), D?.3 (common), D?.3 (common), U?.5 (GND), U?.5 (GND), U?.5 (GND)
- net LPUART_RTS_DE_RS485: now also U?.2 (~RE~), U?.2 (~RE~), U?.2 (~RE~), U?.3 (DE), U?.3 (DE), U?.3 (DE)
- net RX_SER3: no longer U?.15 (X2)
- net RX_SER4: no longer U?.11 (X3)
- net SER_SEL_A0: now also U?.10 (A0); no longer U?.10 (A0)
- net SER_SEL_A1: now also U?.9 (A1); no longer U?.9 (A1)
- net SER_SEL_EN: now also U?.6 (~E); no longer U?.6 (~E)
- net TX_SER4: no longer U?.4 (Y3)
- net USART3_RX_SER: now also U?.13 (X); no longer U?.13 (X)
- net USART3_TX_SER: now also U?.3 (Y); no longer U?.3 (Y)
- net VEE: now also U?.7 (VEE)
- net Vdd: now also U?.16 (Vdd)
- net Vss: now also U?.8 (Vss)
- net at U?.11 (B4): now also D?.5 (K), FB?.2 (x2)
- net at U?.12 (B3): now also D?.4 (K), FB?.2 (x2)
- net at U?.13 (B2): now also D?.3 (K), FB?.2 (x2)
- net at U?.14 (B1): now also D?.1 (K), FB?.2 (x2)
- net *LPUART_RX_RS485 renamed RX_RS485_2
- net RX_RS485_2: now also U?.14 (X1), U?.15 (X2)
- net LPUART_TX_RS485 renamed TX_RS485_2
- net TX_RS485_2: now also U?.5 (Y1)
- net RS485-A renamed RS485_2_A
- net RS485_2_A: now also FB?.1, FB?.1
- net RS485-B renamed RS485_2_B
- net RS485_2_B: now also FB?.1, FB?.1
- net RX_SER1 renamed RX_RS485_1
- net RX_RS485_1: now also U?.1 (RO); no longer U?.5 (A3)
- net RX_SER2 renamed RX_SER_2
- net RX_SER_2: now also U?.14 (X1); no longer U?.14 (X1)
- net TX_SER1 renamed TX_RS485_1
- net TX_RS485_1: now also U?.4 (DI); no longer U?.3 (A1)
- net TX_SER2 renamed TX_SER_2
- net TX_SER_2: now also U?.5 (Y1); no longer U?.5 (Y1)
- net TX_SER3 renamed TX_RS485_3
- net TX_RS485_3: now also U?.4 (DI); no longer U?.3 (A1)
- net USART2_RX_LIN renamed UART4_RX_LIN
- net USART2_TX_LIN renamed UART4_TX_LIN
- new net: R?.2, U?.6 (A) (x3)
- new net: R?.2, U?.7 (B) (x3)
- new net: D?.2 (A2), FB?.2, R?.1, R?.1 (x3)
- new net: D?.1 (A1), FB?.2, R?.1, R?.2 (x3)
- new net LPUART3_TX_RS485: U?.3 (Y)
- new net LPUART_RX_RS485: U?.13 (X)
- new net RS485_1_A: FB?.1
- new net RS485_1_B: FB?.1
- new net RS485_SEL_A0: U?.10 (A0)
- new net RS485_SEL_A1: U?.9 (A1)
- new net RS485_SEL_EN: U?.6 (~E)
- new net RX_RS485_3: U?.1 (RO)
- new net RX_RS485_4: U?.1 (RO), U?.11 (X3)
- new net RX_SER_1: U?.12 (X0), U?.5 (A3)
- new net RX_SER_3: U?.15 (X2)
- new net RX_SER_4: U?.11 (X3)
- new net TTY_RX_1: FB?.1
- new net TTY_RX_2: FB?.1
- new net TTY_RX_3: FB?.1
- new net TTY_RX_4: FB?.1
- new net TTY_TX_1: FB?.1
- new net TTY_TX_2: FB?.1
- new net TTY_TX_3: FB?.1
- new net TTY_TX_4: FB?.1
- new net TX_RS485_4: U?.4 (DI), U?.4 (Y3)
- new net TX_SER_1: U?.1 (Y0), U?.3 (A1)
- new net TX_SER_3: U?.2 (Y2), U?.3 (A1)
- new net TX_SER_4: U?.4 (Y3)
Other:
- moved on the sheet: C200, C201, C202, C203, C204, C205, C211, C?, D200, D201, D202, D204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

Commit message: Prozessor Pins zugeordnet, 4 bistabile Relais, CAN Control Interface, CAN Debug Adapter, Lagesensor zugefügt, Umwelt Sensor, ISM 868 MHz Tranceiver, ESP and Control Bus. UID Eprom. Etliche Aufräum Arbeiten.
Parts:
- removed U? (x3): 4052, symbol 4xxx_IEEE:4052
- added C? (x4): 100nF, Capacitor_SMD:C_0603_1608Metric, symbol Device:C
- added R? (x8): 47k, Resistor_SMD:R_0603_1608Metric, symbol Device:R
- added U? (x4): SN74LV4052A, symbol 4xxx:4052
Connections:
- net +3.3VA: now also C211.2, C?.2, C?.2, C?.2, U204.8 (VCC), U?.8 (VCC), U?.8 (VCC), U?.8 (VCC), C?.1, C?.1, C?.1, C?.1, R?.1, R?.1, R?.1, R?.1, U?.16 (VDD), U?.16 (VDD), U?.16 (VDD), U?.16 (VDD)
- net +3V3: no longer C211.2, C?.2, C?.2, C?.2, U204.8 (VCC), U?.8 (VCC), U?.8 (VCC), U?.8 (VCC)
- net GND: now also C?.2, C?.2, C?.2, C?.2, R?.2, R?.2, R?.2, R?.2, U?.7 (VEE), U?.7 (VEE), U?.7 (VEE), U?.7 (VEE), U?.8 (VSS), U?.8 (VSS), U?.8 (VSS), U?.8 (VSS)
- net LIN_SEL_A0: now also U?.10 (A)
- net LIN_SEL_A1: now also U?.9 (B)
- net LIN_SEL_EN: now also U?.6 (Inh)
- net LPUART3_TX_RS485: now also U?.3 (Y)
- net LPUART_RTS_DE_RS485: now also U?.3 (Y); no longer U204.2 (~RE~), U204.3 (DE), U?.2 (~RE~), U?.2 (~RE~), U?.2 (~RE~), U?.3 (DE), U?.3 (DE), U?.3 (DE)
- net LPUART_RX_RS485: now also U?.13 (X)
- net RS485_2_A: no longer FB?.1, FB?.1
- net RS485_2_B: no longer FB?.1, FB?.1
- net RS485_SEL_A0: now also U?.10 (A), U?.10 (A)
- net RS485_SEL_A1: now also U?.9 (B), U?.9 (B)
- net RS485_SEL_EN: now also U?.6 (Inh), U?.6 (Inh)
- net RX_LIN1: now also U?.12 (X0)
- net RX_LIN2: now also U?.14 (X1)
- net RX_LIN3: now also U?.15 (X2)
- net RX_LIN4: now also U?.11 (X3)
- net RX_RS485_1: now also U?.12 (X0)
- net RX_RS485_2: now also U?.14 (X1), U?.15 (X2)
- net RX_RS485_4: now also U?.11 (X3)
- net RX_SER_1: now also U?.12 (X0)
- net RX_SER_2: now also U?.14 (X1)
- net RX_SER_3: now also U?.15 (X2)
- net RX_SER_4: now also U?.11 (X3)
- net SER_SEL_A0: now also U?.10 (A)
- net SER_SEL_A1: now also U?.9 (B)
- net SER_SEL_EN: now also U?.6 (Inh)
- net TX_LIN1: now also U?.1 (Y0)
- net TX_LIN2: now also U?.5 (Y1)
- net TX_LIN3: now also U?.2 (Y2)
- net TX_LIN4: now also U?.4 (Y3)
- net TX_RS485_1: now also U?.1 (Y0), U?.1 (Y0)
- net TX_RS485_2: now also U?.5 (Y1), U?.5 (Y1)
- net TX_RS485_3: now also U?.2 (Y2), U?.2 (Y2)
- net TX_RS485_4: now also U?.4 (Y3), U?.4 (Y3)
- net TX_SER_1: now also U?.1 (Y0)
- net TX_SER_2: now also U?.5 (Y1)
- net TX_SER_3: now also U?.2 (Y2)
- net TX_SER_4: now also U?.4 (Y3)
- net UART4_RX_LIN: now also U?.13 (X)
- net UART4_TX_LIN: now also U?.3 (Y)
- net USART3_RX_SER: now also U?.13 (X)
- net USART3_TX_SER: now also U?.3 (Y)
- new net DE_RS485_1: R?.1, U?.3 (DE)
- new net DE_RS485_2: R?.1, U204.3 (DE)
- new net DE_RS485_3: R?.1, U?.3 (DE)
- new net DE_RS485_4: R?.1, U?.3 (DE)
- new net RE_RS485: U?.13 (X)
- new net RE_RS485_1: R?.2, U?.12 (X0), U?.2 (~RE~)
- new net RE_RS485_2: R?.2, U204.2 (~RE~), U?.14 (X1)
- new net RE_RS485_3: R?.2, U?.15 (X2), U?.2 (~RE~)
- new net RE_RS485_4: R?.2, U?.11 (X3), U?.2 (~RE~)
- new net RS485_3_A: FB?.1
- new net RS485_3_B: FB?.1
- new net RS485_4_A: FB?.1
- new net RS485_4_B: FB?.1
