File: Hardware/Board/Womo.kicad_pcb (KiCad board)
At the start: 2 copper layers, 157 parts, among them J10 WAGO_Klemmleiste_8-pol, J13 WAGO_Klemmleiste_6-pol, J7 WAGO_Klemmleiste_6-pol, J8 WAGO_Klemmleiste_4-pol, J9 WAGO_Klemmleiste_8-pol, U1 STM32L475VGTx, U10 MAX17572, U11 MAX17572, U12 MAX17574, U13 ESP-12F, U14 DS2482S-800+, U2 AT25SF081-XMHD-X, U3 TJA1029T, U4 TJA1029T, U5 TJA1029T, U6 TJA1049T-3, U7 MAX3072E, U8 MAX17572, U9 MAX17572

Commit message: Footprints zuweisungen
Parts:
- added BT1: Battery_Cell, Battery:BatteryHolder_Keystone_1058_1x2032, F.Cu at (240.0, 191.8)
- added C100: 10u, Capacitor_SMD:C_1210_3225Metric, F.Cu at (35.2, 53.3)
- added C101: 1uF, Capacitor_SMD:C_0603_1608Metric, F.Cu at (110.6, 28.7)
- added C102: 1uF, Capacitor_SMD:C_0603_1608Metric, F.Cu at (285.0, 59.7)
- added C63: 100nF, Capacitor_SMD:C_0603_1608Metric, F.Cu at (270.2, 24.2)
- added C64: 100nF, Capacitor_SMD:C_0603_1608Metric, F.Cu at (273.2, 24.2)
- added C65: 100n, Capacitor_SMD:C_0603_1608Metric, F.Cu at (172.5, 97.4)
- added C66: 10n, Capacitor_SMD:C_0603_1608Metric, F.Cu at (169.5, 97.4)
- added C67: 4u7, Capacitor_SMD:C_0603_1608Metric, F.Cu at (173.2, 95.4)
- added C68: 10n, Capacitor_SMD:C_0603_1608Metric, F.Cu at (165.1, 102.0)
- added C69: 4u7, Capacitor_SMD:C_0603_1608Metric, F.Cu at (173.2, 93.9)
- added C70: 1uF, Capacitor_SMD:C_0603_1608Metric, F.Cu at (39.0, 54.0)
- added C71: 100n, Capacitor_SMD:C_0603_1608Metric, F.Cu at (266.9, 60.1)
- added C72: 100n, Capacitor_SMD:C_0603_1608Metric, F.Cu at (39.0, 52.5)
- added C73: 100n, Capacitor_SMD:C_0603_1608Metric, F.Cu at (269.9, 60.1)
- added C74: 100n, Capacitor_SMD:C_0603_1608Metric, F.Cu at (83.9, 42.2)
- added C75: 100n, Capacitor_SMD:C_0603_1608Metric, F.Cu at (57.9, 74.1)
- added C76: 100n, Capacitor_SMD:C_0603_1608Metric, F.Cu at (72.0, 58.5)
- added C77: 100n, Capacitor_SMD:C_0603_1608Metric, F.Cu at (279.0, 60.1)
- added C78: 2u2, Capacitor_SMD:C_0603_1608Metric, F.Cu at (86.9, 42.2)
- added C79: 10uF, Capacitor_SMD:C_1210_3225Metric, F.Cu at (71.0, 48.4)
- added C80: 100nF, Capacitor_SMD:C_0603_1608Metric, F.Cu at (282.0, 59.7)
- added C81: 100nF, Capacitor_SMD:C_0603_1608Metric, F.Cu at (83.9, 43.7)
- added C82: 100nF, Capacitor_SMD:C_0603_1608Metric, F.Cu at (72.0, 54.4)
- added C83: 1uF, Capacitor_SMD:C_0603_1608Metric, F.Cu at (51.2, 79.3)
- added C84: 100nF, Capacitor_SMD:C_0603_1608Metric, F.Cu at (72.0, 55.9)
- added C85: 100nF, Capacitor_SMD:C_0603_1608Metric, F.Cu at (276.0, 60.1)
- added C86: 100nF, Capacitor_SMD:C_0603_1608Metric, F.Cu at (89.9, 43.7)
- added C87: 10u, Capacitor_SMD:C_1210_3225Metric, F.Cu at (206.7, 19.4)
- added C88: 10u, Capacitor_SMD:C_1210_3225Metric, F.Cu at (202.1, 19.4)
- added C89: 100pF, Capacitor_SMD:C_0603_1608Metric, F.Cu at (43.4, 149.6)
- added C90: 100pF, Capacitor_SMD:C_0603_1608Metric, F.Cu at (71.7, 119.1)
- added C91: 100pF, Capacitor_SMD:C_0603_1608Metric, F.Cu at (37.3, 152.9)
- added C92: 100pF, Capacitor_SMD:C_0603_1608Metric, F.Cu at (119.4, 90.3)
- added C93: 100pF, Capacitor_SMD:C_0603_1608Metric, F.Cu at (43.4, 152.6)
- added C94: 100pF, Capacitor_SMD:C_0603_1608Metric, F.Cu at (40.8, 146.5)
- added C95: 100pF, Capacitor_SMD:C_0603_1608Metric, F.Cu at (40.8, 143.5)
- added C96: 100pF, Capacitor_SMD:C_0603_1608Metric, F.Cu at (37.8, 145.0)
- added C97: 1uF, Capacitor_SMD:C_0603_1608Metric, F.Cu at (54.2, 79.3)
- added C98: 100n, Capacitor_SMD:C_0603_1608Metric, F.Cu at (86.9, 45.2)
- added C99: 1uF, Capacitor_SMD:C_0603_1608Metric, F.Cu at (89.9, 42.2)
- added D14: SP0504BAJT, Package_TO_SOT_SMD:SOT-353_SC-70-5, F.Cu at (271.7, 22.1)
- added D15: SP0504BAJT, Package_TO_SOT_SMD:SOT-353_SC-70-5, F.Cu at (271.7, 19.2)
- added D16: SP0504BAJT, Package_TO_SOT_SMD:SOT-353_SC-70-5, F.Cu at (28.3, 155.6)
- added D17: SP0504BAJT, Package_TO_SOT_SMD:SOT-353_SC-70-5, F.Cu at (71.8, 116.9)
- added D18: SP0504BAJT, Package_TO_SOT_SMD:SOT-353_SC-70-5, F.Cu at (31.5, 155.6)
- added D19: LED, LED_SMD:LED_1206_3216Metric, F.Cu at (267.8, 58.2)
- added D20: B230, Diode_SMD:D_SMB, F.Cu at (181.4, 20.1)
- added D21: B230, Diode_SMD:D_SMB, F.Cu at (196.1, 20.1)
- added D22: B230, Diode_SMD:D_SMB, F.Cu at (188.7, 20.1)
- added FB16: 100R, Inductor_SMD:L_0603_1608Metric, F.Cu at (165.1, 103.5)
- added FB17: 100R, Inductor_SMD:L_0603_1608Metric, F.Cu at (171.6, 99.0)
- added FB18: 100R, Inductor_SMD:L_0603_1608Metric, F.Cu at (58.6, 138.1)
- added FB19: 100R, Inductor_SMD:L_0603_1608Metric, F.Cu at (55.6, 141.1)
- added FB20: 100R, Inductor_SMD:L_0603_1608Metric, F.Cu at (40.7, 155.6)
- added FB21: 100R, Inductor_SMD:L_0603_1608Metric, F.Cu at (71.7, 123.6)
- added FB22: 100R, Inductor_SMD:L_0603_1608Metric, F.Cu at (40.7, 154.1)
- added FB23: 100R, Inductor_SMD:L_0603_1608Metric, F.Cu at (71.7, 122.1)
- added FB24: 100R, Inductor_SMD:L_0603_1608Metric, F.Cu at (58.6, 135.1)
- added FB25: 100R, Inductor_SMD:L_0603_1608Metric, F.Cu at (74.7, 119.1)
- added FB26: 100R, Inductor_SMD:L_0603_1608Metric, F.Cu at (46.8, 145.0)
- added FB27: 100R, Inductor_SMD:L_0603_1608Metric, F.Cu at (49.8, 145.0)
- added FB28: 100R, Inductor_SMD:L_0603_1608Metric, F.Cu at (37.3, 151.4)
- added FB29: 100R, Inductor_SMD:L_0603_1608Metric, F.Cu at (43.8, 143.5)
- added FB30: 100R, Inductor_SMD:L_0603_1608Metric, F.Cu at (34.7, 154.4)
- added FB31: 100R, Inductor_SMD:L_0603_1608Metric, F.Cu at (43.8, 145.0)
- added FB32: 100R, Inductor_SMD:L_0603_1608Metric, F.Cu at (40.8, 148.0)
- added FB33: 100R, Inductor_SMD:L_0603_1608Metric, F.Cu at (34.3, 152.9)
- added FB34: 100R, Inductor_SMD:L_0603_1608Metric, F.Cu at (40.3, 149.6)
- added FB35: 100R, Inductor_SMD:L_0603_1608Metric, F.Cu at (43.8, 146.5)
- added FB36: 100R, Inductor_SMD:L_0603_1608Metric, F.Cu at (34.7, 155.9)
- added FB37: 100R, Inductor_SMD:L_0603_1608Metric, F.Cu at (46.8, 143.5)
- added FB38: 100R, Inductor_SMD:L_0603_1608Metric, F.Cu at (46.4, 149.6)
- added FB39: 100R, Inductor_SMD:L_0603_1608Metric, F.Cu at (37.8, 148.0)
- added FB40: 100R, Inductor_SMD:L_0603_1608Metric, F.Cu at (37.8, 143.5)
- added FB41: 100R, Inductor_SMD:L_0603_1608Metric, F.Cu at (37.3, 149.9)
- added FB42: 100R, Inductor_SMD:L_0603_1608Metric, F.Cu at (55.6, 135.1)
- added FB43: 100R, Inductor_SMD:L_0603_1608Metric, F.Cu at (34.3, 151.4)
- added FB44: 100R, Inductor_SMD:L_0603_1608Metric, F.Cu at (34.3, 149.9)
- added FB45: Ferrite, Inductor_SMD:L_0603_1608Metric, F.Cu at (273.0, 60.1)
- added FB46: Ferrite, Inductor_SMD:L_0603_1608Metric, F.Cu at (66.1, 65.5)
- added FB47: Ferrite, Inductor_SMD:L_0603_1608Metric, F.Cu at (83.9, 46.7)
- added FB48: Ferrite, Inductor_SMD:L_0603_1608Metric, F.Cu at (51.2, 80.8)
- added FB49: Ferrite, Inductor_SMD:L_0603_1608Metric, F.Cu at (86.9, 43.7)
- added IC1: MX25LM51245GXDI00, SamacSys_Parts:BGA24C100P5X5_600X800X35, F.Cu at (237.5, 144.8)
- added IC2: IS66WVH8M8BLL-100B1LI_0, SamacSys_Parts:BGA24C100P5X5_600X800X35, F.Cu at (226.1, 144.8)
- added IC3: TSC2007, Package_SO:TSSOP-16_4.4x5mm_P0.65mm, F.Cu at (284.5, 56.1)
- added J1: Conn_01x06, Connector_PinHeader_2.54mm:PinHeader_1x06_P2.54mm_Vertical, F.Cu at (163.5, 19.6)
- added J11: RJ12, Connector_RJ:RJ12_Amphenol_54601, F.Cu at (43.1, 117.3)
- added J12: RJ45, Connector_RJ:RJ45_Amphenol_54602-x08_Horizontal, F.Cu at (57.6, 119.8)
- added J14: 52271-0679, SamacSys_Parts:52271-0679, F.Cu at (63.5, 56.0)
- added J15: Conn_01x06, Connector_PinSocket_2.54mm:PinSocket_1x06_P2.54mm_Horizontal, F.Cu at (240.0, 6.35)
- added J18: WAGO_Klemmleiste_8-pol, WAGO Klemmleisten:WAGO_Klemmleiste_Hebel4mm²Vertikal_RM5mm_8-pol, F.Cu at (79.2, 93.3)
- added J19: WAGO_Klemmleiste_8-pol, WAGO Klemmleisten:WAGO_Klemmleiste_Hebel4mm²Vertikal_RM5mm_8-pol, F.Cu at (36.7, 93.3)
- added J2: Conn_02x25_Odd_Even, Connector_PinSocket_2.54mm:PinSocket_2x25_P2.54mm_Vertical, F.Cu at (31.0, 91.4)
- added J20: Conn_02x03_Top_Bottom, Connectors_Molex:Molex_Microfit3_Header_02x03_Straight_43045-0628, F.Cu at (49.5, 139.9)
- added J21: Conn_02x10_Odd_Even, Connector_PinHeader_2.54mm:PinHeader_2x10_P2.54mm_Vertical, F.Cu at (34.6, 117.3)
- added J22: Conn_02x06_Odd_Even, Connector_PinHeader_2.54mm:PinHeader_2x06_P2.54mm_Vertical, F.Cu at (250.2, 62.2)
- added J23: Conn_02x25_Odd_Even, Connector_PinHeader_2.54mm:PinHeader_2x25_P2.54mm_Vertical, F.Cu at (284.5, 86.4)
- added J3: USB_B_Micro, Connector_USB:USB_Micro-B_Molex-105017-0001, F.Cu at (270.5, 88.9)
- added J4: 54104-4031, SamacSys_Parts:54104-4031, F.Cu at (246.4, 87.6)
- added J5: Conn_ARM_JTAG_SWD_20, Connector_IDC:IDC-Header_2x10_P2.54mm_Vertical, F.Cu at (264.2, 73.7)
- added J6: Raspberry_Pi_2_3, Connector_IDC:IDC-Header_2x20_P2.54mm_Vertical, F.Cu at (155.7, 23.4)
- added L1: 15uH, Inductor_SMD:L_Coilcraft_XxL4040, F.Cu at (152.1, 100.7)
- added L2: 15uH, Inductor_SMD:L_Coilcraft_XxL4040, F.Cu at (161.4, 91.9)
- added L3: 15uH, Inductor_SMD:L_Coilcraft_XxL4040, F.Cu at (156.7, 100.7)
- added L4: L_Core_Ferrite, Inductor_SMD:L_Coilcraft_XxL4020, F.Cu at (161.4, 96.4)
- added L5: 10uH, SamacSys_Parts:XAL8080, F.Cu at (154.0, 94.0)
- added L6: 15uH, Inductor_SMD:L_Coilcraft_XxL4040, F.Cu at (166.0, 91.9)
- added L7: 4uH7, Inductor_SMD:L_Coilcraft_XxL4030, F.Cu at (161.3, 101.0)
- added Q1: 2N7002, Package_TO_SOT_SMD:SOT-23, F.Cu at (170.0, 91.4)
- added Q2: 2N7002, Package_TO_SOT_SMD:SOT-23, F.Cu at (173.4, 91.4)
- added Q3: 2N7002, Package_TO_SOT_SMD:SOT-23, F.Cu at (170.0, 94.9)
- added Q4: 2N7002, Package_TO_SOT_SMD:SOT-23, F.Cu at (165.4, 99.5)
- added Q5: 2N7002, Package_TO_SOT_SMD:SOT-23, F.Cu at (34.5, 147.3)
- added Q6: 2N7002, Package_TO_SOT_SMD:SOT-23, F.Cu at (34.5, 143.8)
- added R48: 10K, Resistor_SMD:R_0603_1608Metric, F.Cu at (264.2, 24.2)
- added R49: 10K, Resistor_SMD:R_0603_1608Metric, F.Cu at (267.2, 24.2)
- added R50: 100K, Resistor_SMD:R_0603_1608Metric, F.Cu at (168.1, 102.0)
- added R51: 10R 1%, Resistor_SMD:R_0603_1608Metric, F.Cu at (168.6, 100.5)
- added R52: 32k4, Resistor_SMD:R_0603_1608Metric, F.Cu at (168.6, 99.0)
- added R53: 1K, Resistor_SMD:R_0603_1608Metric, F.Cu at (71.7, 120.6)
- added R54: 1K, Resistor_SMD:R_0603_1608Metric, F.Cu at (37.7, 155.9)
- added R55: 1K, Resistor_SMD:R_0603_1608Metric, F.Cu at (43.8, 148.0)
- added R56: 1K, Resistor_SMD:R_0603_1608Metric, F.Cu at (46.8, 146.5)
- added R57: 1K, Resistor_SMD:R_0603_1608Metric, F.Cu at (49.8, 143.5)
- added R58: 1K, Resistor_SMD:R_0603_1608Metric, F.Cu at (37.7, 154.4)
- added R59: 1K, Resistor_SMD:R_0603_1608Metric, F.Cu at (61.6, 135.1)
- added R60: 1K, Resistor_SMD:R_0603_1608Metric, F.Cu at (43.4, 151.1)
- added R61: 10k, Resistor_SMD:R_0603_1608Metric, F.Cu at (46.8, 148.0)
- added R62: 10k, Resistor_SMD:R_0603_1608Metric, F.Cu at (40.8, 145.0)
- added R63: 10k, Resistor_SMD:R_0603_1608Metric, F.Cu at (37.8, 146.5)
- added R64: 10k, Resistor_SMD:R_0603_1608Metric, F.Cu at (40.3, 151.1)
- added R65: 10k, Resistor_SMD:R_0603_1608Metric, F.Cu at (55.6, 136.6)
- added R66: 10k, Resistor_SMD:R_0603_1608Metric, F.Cu at (74.9, 116.3)
- added R67: 10k, Resistor_SMD:R_0603_1608Metric, F.Cu at (119.4, 91.9)
- added R68: 10k, Resistor_SMD:R_0603_1608Metric, F.Cu at (77.9, 116.3)
- added R69: 1K, Resistor_SMD:R_0603_1608Metric, F.Cu at (58.6, 136.6)
- added R70: 10k, Resistor_SMD:R_0603_1608Metric, F.Cu at (55.6, 138.1)
- added R71: 10k, Resistor_SMD:R_0603_1608Metric, F.Cu at (40.3, 152.6)
- added R72: 1K, Resistor_SMD:R_0603_1608Metric, F.Cu at (55.6, 139.6)
- added R73: 10k, Resistor_SMD:R_0603_1608Metric, F.Cu at (77.7, 117.8)
- added R74: 10k, Resistor_SMD:R_0603_1608Metric, F.Cu at (74.7, 120.6)
- added R75: 10K, Resistor_SMD:R_0603_1608Metric, F.Cu at (86.9, 46.7)
- added R76: 10K, Resistor_SMD:R_0603_1608Metric, F.Cu at (288.0, 59.7)
- added R77: 10K, Resistor_SMD:R_0603_1608Metric, F.Cu at (83.9, 45.2)
- added R78: 10K, Resistor_SMD:R_0603_1608Metric, F.Cu at (66.1, 64.0)
- added U15: MAX11615, Package_SO:QSOP-16_3.9x4.9mm_P0.635mm, F.Cu at (266.4, 20.7)
- added U16: STLD40D, Package_DFN_QFN:DFN-8-1EP_3x3mm_P0.65mm_EP1.55x2.4mm, F.Cu at (165.8, 95.9)
- added U17: STM32L4R9ZITx, Package_QFP:LQFP-144_20x20mm_P0.5mm, F.Cu at (242.6, 120.7)
- added U18: USBLC6-2SC6, Package_TO_SOT_SMD:SOT-23-6, F.Cu at (72.4, 51.8)
- added U19: MOD-nRF8001, RF_Module:MOD-nRF8001, F.Cu at (274.3, 185.4)
- C12, C13: value 5p1 -> 3p3
- C2, C3: value 8p2 -> 6p8
- C4, C5, C6, C7: value C -> 100n
- C8: value 100nF -> 100n
- D1: value SP0504BAJT -> DIODE
- U1: value STM32L475VGTx -> PCF8574A
- U2: value AT25SF081-XMHD-X -> PCF8574A
Connections:
- net RxD-RS485 renamed *LPUART_RX_RS485
- C1 pad 1: Net-(C1-Pad1) -> RESET
- C1 pad 2: GND -> GND1
- C10 pad 1: Net-(C10-Pad1) -> +3V3
- C10 pad 2: GND -> GND1
- C11 pad 1: Net-(C10-Pad1) -> +3V3
- C11 pad 2: GND -> GND1
- C12 pad 1: GND -> GND1
- C13 pad 1: GND -> GND1
- C14 pad 1: +3V3 -> GND
- C14 pad 2: GND -> +3V3
- C15 pad 1: +5VL -> +VSW
- C15 pad 2: GND -> GND1
- C2 pad 2: GND -> GND1
- C3 pad 2: GND -> GND1
- C4 pad 2: GND -> GND1
- C5 pad 2: GND -> GND1
- C55 pad 1: +5VL -> +VSW
- C6 pad 2: GND -> GND1
- C60 pad 1: Net-(C60-Pad1) -> +3.3VA
- C7 pad 2: GND -> GND1
- C8 pad 2: GND -> GND1
- C9 pad 2: GND -> GND1
- D1 pad 1: Disp_SCK -> Net-(D1-Pad1)
- D1 pad 2: GND -> LCD_LED-A
- D1 pad 3: Disp_MOSI -> (no net)
- D1 pad 4: Disp_INT -> (no net)
- D1 pad 5: Disp_Audio_L -> (no net)
- D12 pad 1: Net-(D12-Pad1) -> P0
- D12 pad 3: Net-(D12-Pad3) -> P1
- D12 pad 4: Net-(D12-Pad4) -> P2
- D12 pad 5: Net-(D12-Pad5) -> P3
- D13 pad 1: Net-(D13-Pad1) -> AIN0
- D13 pad 3: Net-(D13-Pad3) -> AIN1
- D13 pad 4: Net-(D13-Pad4) -> AIN2
- D13 pad 5: Net-(D13-Pad5) -> AIN3
- D2 pad 1: +5VL -> Net-(D2-Pad1)
- D2 pad 3: Disp_MISO -> Net-(D2-Pad3)
- D2 pad 4: Disp_CS -> Net-(D2-Pad4)
- D2 pad 5: Disp_PD -> Net-(D2-Pad5)
- D3 pad 3: USB_D+ -> Net-(D3-Pad3)
- D3 pad 4: USB_D- -> Net-(D3-Pad4)
- D3 pad 5: USB_ID -> Net-(D3-Pad5)
- D7 pad 2: GND -> Net-(D7-Pad2)
- FB10 pad 2: Net-(D13-Pad3) -> Net-(D3-Pad3)
- FB11 pad 2: Net-(D12-Pad3) -> Net-(D2-Pad3)
- FB12 pad 2: Net-(D13-Pad4) -> Net-(D3-Pad4)
- FB13 pad 2: Net-(D12-Pad4) -> Net-(D2-Pad4)
- FB14 pad 2: Net-(D13-Pad5) -> Net-(D3-Pad5)
- FB15 pad 2: Net-(D12-Pad5) -> Net-(D2-Pad5)
- FB8 pad 2: Net-(D13-Pad1) -> Net-(D3-Pad1)
- FB9 pad 2: Net-(D12-Pad1) -> Net-(D2-Pad1)
- R1 pad 2: RxD-LIN1 -> USART1_RX_LIN1
- R2 pad 2: RxD-LIN2 -> USART2_RX_LIN2
- R29 pad 2: 5V_Disp_EN -> VSW_Disp_EN
- R3 pad 2: RxD-LIN3 -> USART3_RX_LIN3
- R34 pad 1: +5VL -> +VSW
- R36 pad 1: +5VL -> +VSW
- R40 pad 2: Net-(D13-Pad1) -> Net-(D3-Pad1)
- R41 pad 2: Net-(D13-Pad3) -> Net-(D3-Pad3)
- R42 pad 2: Net-(D13-Pad4) -> Net-(D3-Pad4)
- R43 pad 2: Net-(D13-Pad5) -> Net-(D3-Pad5)
- R44 pad 2: Net-(D12-Pad1) -> Net-(D2-Pad1)
- R45 pad 2: Net-(D12-Pad3) -> Net-(D2-Pad3)
- R46 pad 2: Net-(D12-Pad4) -> Net-(D2-Pad4)
- R47 pad 2: Net-(D12-Pad5) -> Net-(D2-Pad5)
- U1 pad 1: Net-(U1-Pad1) -> +3V3
- U1 pad 10: GND -> 3VA_EN
- U1 pad 100: +3V3 -> (no net)
- U1 pad 11: +3V3 -> 5V_Raspi_EN
- U1 pad 12: Net-(C2-Pad1) -> VSW_Disp_EN
- U1 pad 13: Net-(C3-Pad1) -> Net-(U1-Pad13)
- U1 pad 14: Net-(C1-Pad1) -> I2C2_SCL
- U1 pad 15: Net-(U1-Pad15) -> I2C2_SDA
- U1 pad 16: Net-(U1-Pad16) -> +3V3
- U1 pad 17: Net-(U1-Pad17) -> (no net)
- U1 pad 18: Net-(U1-Pad18) -> (no net)
- U1 pad 19: Net-(U1-Pad19) -> (no net)
- U1 pad 2: Net-(U1-Pad2) -> GND
- U1 pad 20: Net-(U1-Pad20) -> (no net)
- U1 pad 21: Net-(U1-Pad21) -> (no net)
- U1 pad 22: Net-(C10-Pad1) -> (no net)
- U1 pad 23: Net-(U1-Pad23) -> (no net)
- U1 pad 24: Net-(U1-Pad24) -> (no net)
- U1 pad 25: Net-(U1-Pad25) -> (no net)
- U1 pad 26: Net-(U1-Pad26) -> (no net)
- U1 pad 27: GND -> (no net)
- U1 pad 28: +3V3 -> (no net)
- U1 pad 29: Net-(U1-Pad29) -> (no net)
- U1 pad 3: Net-(U1-Pad3) -> GND
- U1 pad 30: Disp_SCK -> (no net)
- U1 pad 31: Disp_MISO -> (no net)
- U1 pad 32: Disp_MOSI -> (no net)
- U1 pad 33: Net-(U1-Pad33) -> (no net)
- U1 pad 34: Net-(U1-Pad34) -> (no net)
- U1 pad 35: Net-(U1-Pad35) -> (no net)
- U1 pad 36: Net-(U1-Pad36) -> (no net)
- U1 pad 37: Net-(U1-Pad37) -> (no net)
- U1 pad 38: Net-(U1-Pad38) -> (no net)
- U1 pad 39: Net-(U1-Pad39) -> (no net)
- U1 pad 4: Net-(U1-Pad4) -> SLP-LIN1
- U1 pad 40: Net-(U1-Pad40) -> (no net)
- U1 pad 41: QuadSPI_CLK -> (no net)
- U1 pad 42: QuadSPI_NCS -> (no net)
- U1 pad 43: QuadSPI_IO0 -> (no net)
- U1 pad 44: QuadSPI_IO1 -> (no net)
- U1 pad 45: QuadSPI_IO2 -> (no net)
- U1 pad 46: QuadSPI_IO3 -> (no net)
- U1 pad 47: Net-(U1-Pad47) -> (no net)
- U1 pad 48: Net-(U1-Pad48) -> (no net)
- U1 pad 49: GND -> (no net)
- U1 pad 5: Net-(U1-Pad5) -> SLP-LIN2
- U1 pad 50: +3V3 -> (no net)
- U1 pad 51: Net-(U1-Pad51) -> (no net)
- U1 pad 52: Net-(U1-Pad52) -> (no net)
- U1 pad 53: Net-(U1-Pad53) -> (no net)
- U1 pad 54: Net-(U1-Pad54) -> (no net)
- U1 pad 55: Net-(U1-Pad55) -> (no net)
- U1 pad 56: Net-(U1-Pad56) -> (no net)
- U1 pad 57: Net-(U1-Pad57) -> (no net)
- U1 pad 58: Net-(U1-Pad58) -> (no net)
- U1 pad 59: Net-(U1-Pad59) -> (no net)
- U1 pad 6: Net-(U1-Pad6) -> SLP-LIN3
- U1 pad 60: Net-(U1-Pad60) -> (no net)
- U1 pad 61: Net-(U1-Pad61) -> (no net)
- U1 pad 62: Net-(U1-Pad62) -> (no net)
- U1 pad 63: Net-(U1-Pad63) -> (no net)
- U1 pad 64: Net-(U1-Pad64) -> (no net)
- U1 pad 65: Net-(U1-Pad65) -> (no net)
- U1 pad 66: Net-(U1-Pad66) -> (no net)
- U1 pad 67: USB_SOF -> (no net)
- U1 pad 68: Net-(U1-Pad68) -> (no net)
- U1 pad 69: USB_ID -> (no net)
- U1 pad 7: Net-(U1-Pad7) -> STB-CAN
- U1 pad 70: USB_D- -> (no net)
- U1 pad 71: USB_D+ -> (no net)
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
Commit message: Alle Footprints definiert, Libs angepasst, Layout gestartet mit Plazierung, Controller und Breakout Netzmäßig getrennt.
Parts:
- added J16: Conn_01x06, SamacSys_Parts:436500628, F.Cu at (61.9, 2.70)
- added J17: Conn_01x05, SamacSys_Parts:436500527, F.Cu at (58.4, 10.6)
- added J24: Conn_01x06, Connector_PinHeader_2.54mm:PinHeader_1x06_P2.54mm_Vertical, F.Cu at (158.8, 105.4)
- added SW1: Reset, Button_Switch_THT:SW_PUSH_6mm, F.Cu at (163.8, 152.4)
- added SW2: Boot, Button_Switch_THT:SW_PUSH_6mm, F.Cu at (163.8, 143.5)
- added SW3: Wakeup, Button_Switch_THT:SW_PUSH_6mm_H8.5mm, F.Cu at (163.8, 133.3)
- added Y1: 16 MHz, Crystal:Crystal_SMD_3225-4Pin_3.2x2.5mm, F.Cu at (226.1, 137.2)
- added Y2: 32.768, Crystal:Crystal_SMD_MicroCrystal_CC7V-T1A-2Pin_3.2x1.5mm, F.Cu at (233.7, 139.7)
- D1: footprint Package_TO_SOT_SMD:SOT-353_SC-70-5 -> Diode_SMD:D_SMB
- J10, J9: footprint TerminalBlock_WAGO:TerminalBlock_WAGO_236-108_1x08_P5.00mm_45Degree -> WAGO Klemmleisten:WAGO_Klemmleiste_Hebel4mm²Vertikal_RM5mm_8-pol
- J13, J7: footprint TerminalBlock_WAGO:TerminalBlock_WAGO_236-106_1x06_P5.00mm_45Degree -> WAGO Klemmleisten:WAGO_Klemmleiste_Hebel4mm²Vertikal_RM5mm_6-pol
- J15: footprint Connector_PinSocket_2.54mm:PinSocket_1x06_P2.54mm_Horizontal -> Connector_PinSocket_2.54mm:PinSocket_1x06_P2.54mm_Vertical
- J23: moved to B.Cu
- J8: footprint TerminalBlock_WAGO:TerminalBlock_WAGO_236-304_1x04_P10.00mm_45Degree -> WAGO Klemmleisten:WAGO_Klemmleiste_Hebel4mm²Vertikal_RM5mm_4-pol
- U1: footprint Package_QFP:LQFP-100_14x14mm_P0.5mm -> Package_SO:SOIC-16W_7.5x10.3mm_P1.27mm
- U2: footprint Package_SO:TSSOP-8_4.4x3mm_P0.65mm -> Package_SO:SOIC-16W_7.5x10.3mm_P1.27mm
- moved FB46 253.0 mm to (290.8, 181.6)
- moved FB48 250.7 mm to (280.7, 181.6), turned to 180 degrees
- moved C99 244.3 mm to (293.4, 177.3), turned to 270 degrees
- moved C76 241.0 mm to (276.9, 185.4), turned to 180 degrees
- moved FB47 234.4 mm to (280.7, 174.0), turned to 180 degrees
- moved FB49 232.1 mm to (280.7, 171.4), turned to 180 degrees
- moved C60 224.1 mm to (184.9, -50.5)
- moved C101 222.6 mm to (278.1, 175.3), turned to 270 degrees
- moved C72 220.0 mm to (248.9, 118.1), turned to 180 degrees
- moved C58 219.3 mm to (177.6, -42.7)
- moved C59 219.2 mm to (177.6, -45.9)
- moved C79 217.8 mm to (276.0, 122.1), turned to 180 degrees
- moved J14 216.7 mm to (240.0, 181.6)
- moved C98 209.1 mm to (246.4, 180.3)
- moved C100 205.0 mm to (204.5, 168.9), turned to 90 degrees
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Connections:
- C10 pad 1: +3V3 -> VCCQ
- C100 pad 1: +3.3VA -> +3.3VP
- C101 pad 1: +VSW -> VCC
- C102 pad 1: +3.3VA -> +3.3VP
- C11 pad 1: +3V3 -> VCCQ
- C15 pad 1: +VSW -> VCC
- C4 pad 1: +3V3 -> VCCQ
- C5 pad 1: +3V3 -> VCCQ
- C6 pad 1: +3V3 -> VCCQ
- C7 pad 1: +3V3 -> VCCQ
- C71 pad 1: +3V3 -> VCCQ
- C72 pad 1: +3V3 -> VCCQ
- C73 pad 1: +3V3 -> VCCQ
- C74 pad 1: +3V3 -> VCCQ
- C75 pad 2: +3V3 -> VCCQ
- C76 pad 2: +3V3 -> VCCQ
- C77 pad 2: +3V3 -> VCCQ
- C78 pad 2: RESET -> Net-(C78-Pad2)
- C79 pad 1: +3V3 -> VCCQ
- C8 pad 1: +3V3 -> VCCQ
- C80 pad 1: +3V3 -> VCCQ
- C81 pad 1: +3V3 -> VCCQ
- C82 pad 1: +3V3 -> VCCQ
- C83 pad 1: +VSW -> VCC
- C84 pad 1: +3V3 -> VCCQ
- C85 pad 1: +3V3 -> VCCQ
- C86 pad 1: +3V3 -> VCCQ
- C9 pad 1: +3V3 -> VCCQ
- C97 pad 1: +3V3 -> VCCQ
- C98 pad 2: +VSW -> VCC
- C99 pad 1: +3V3 -> VCCQ
- D16 pad 4: PA9 -> Net-(D16-Pad4)
- FB32 pad 2: PA9 -> Net-(D16-Pad4)
- FB45 pad 1: +3V3 -> VCCQ
- FB47 pad 2: +VSW -> VCC
- FB49 pad 2: +3.3VA -> +3.3VP
- IC1 pad B4: +3V3 -> VCCQ
- IC1 pad D1: +3V3 -> VCCQ
- IC1 pad E4: +3V3 -> VCCQ
- IC2 pad B4: +3V3 -> VCCQ
- IC2 pad D1: +3V3 -> VCCQ
- IC2 pad E4: +3V3 -> VCCQ
- IC3 pad 1: +VSW -> VCC
- J14 pad 1: +VSW -> VCC
- J2 pad 31: PA9 -> LCD_BL_CTR
- J22 pad 1: I2C2_SCL -> I2C3_SCL
- J22 pad 3: I2C2_SDA -> I2C3_SDA
- J23 pad 23: GND -> GND1
- J23 pad 24: GND -> GND1
- J23 pad 31: *PA9 -> *LCD_BL_CTR
- J4 pad 1: LCD_LED-K -> *LCD_LED-K
- J4 pad 2: LCD_LED-A -> *LCD_LED-A
- J4 pad 4: +VSW -> VCC
- J5 pad 2: +3V3 -> VCCQ
- R75 pad 2: Net-(R75-Pad2) -> GND1
- R76 pad 1: +3V3 -> VCCQ
- R77 pad 1: +VSW -> VCC
- R78 pad 1: +VSW -> VCC
- U17 pad 103: *PA9 -> PA9
- U17 pad 108: +3V3 -> VCCQ
- U17 pad 110: +3V3 -> VCCQ
- U17 pad 120: LCD_BL_CTRL -> PD4
- U17 pad 123: +3V3 -> VCCQ
- U17 pad 125: Net-(U17-Pad125) -> PD7
- U17 pad 131: +3V3 -> VCCQ
- U17 pad 144: +3V3 -> VCCQ
- U17 pad 17: +3V3 -> VCCQ
- U17 pad 29: +3V3 -> VCCQ
- U17 pad 30: +3V3 -> VCCQ
- U17 pad 36: +3V3 -> VCCQ
- U17 pad 38: LCD_BL_CTR -> *LCD_BL_CTR
- U17 pad 48: +3V3 -> VCCQ
- U17 pad 58: +3V3 -> VCCQ
- U17 pad 68: +3V3 -> VCCQ
- U17 pad 73: +3V3 -> VCCQ
- U17 pad 74: RESET -> Net-(C78-Pad2)
- U17 pad 80: RESET -> Net-(C78-Pad2)
- U17 pad 86: Net-(U17-Pad86) -> PD13
- U17 pad 88: +3V3 -> VCCQ
- U19 pad 1: +3.3VA -> +3.3VP
Other:
- rule pad_to_mask_clearance: 0.051 -> 0

Commit message: Kleinigkeiten
Parts:
- moved J2 294.4 mm to (277.7, 19.2)
- moved J9 246.4 mm to (240.2, -6.99), turned to 180 degrees
- moved J10 201.3 mm to (222.8, 35.7), turned to 180 degrees
- moved J7 193.1 mm to (256.3, 35.6), turned to 180 degrees
- moved J6 159.8 mm to (93.9, 105.4)
- moved C14 146.2 mm to (37.8, 74.1)
- moved C16 146.2 mm to (48.8, 61.4)
- moved C17 146.2 mm to (52.8, 59.2)
- moved C18 146.2 mm to (48.8, 62.9)
- moved C19 146.2 mm to (55.8, 58.8)
- moved C20 146.2 mm to (37.8, 75.6)
- moved C21 146.2 mm to (51.8, 61.1)
- moved C22 146.2 mm to (48.8, 64.4)
- moved C23 146.2 mm to (26.4, 84.2)
- moved C24 146.2 mm to (57.4, 56.0)
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
Commit message: Komplete enummerierung Geändert, Schaltplan zusammengefasst, Layout nochmals reset. BOM zu 75% fertig gestellt
Parts:
- removed C38, C55, C61, C79: 10uF, Capacitor_SMD:C_1210_3225Metric
- removed C39, C54, C57: 22uF, Capacitor_SMD:C_1210_3225Metric
- removed C40, C41, C42, C78: 2u2, Capacitor_SMD:C_0603_1608Metric
- removed C43, C47, C65, C71, C72, C73, C74, C75, C76, C77, C98: 100n, Capacitor_SMD:C_0603_1608Metric
- removed C44: 22nF, Capacitor_SMD:C_0603_1608Metric
- removed C45: 1u, Capacitor_SMD:C_0603_1608Metric
- removed C46: 5n6, Capacitor_SMD:C_0603_1608Metric
- removed C48, C50, C56, C62, C63, C64, C80, C81, C82, C84, C85, C86: 100nF, Capacitor_SMD:C_0603_1608Metric
- removed C49, C53, C58: 47u, Capacitor_SMD:C_1210_3225Metric
- removed C51, C59, C60, C87, C88: 10u, Capacitor_SMD:C_1210_3225Metric
- removed C52: 4u7, Capacitor_SMD:C_1210_3225Metric
- removed C66, C68: 10n, Capacitor_SMD:C_0603_1608Metric
- removed C67, C69: 4u7, Capacitor_SMD:C_0603_1608Metric
- removed C70, C83, C97, C99: 1uF, Capacitor_SMD:C_0603_1608Metric
- removed C89, C90, C91, C92, C93, C94, C95, C96: 100pF, Capacitor_SMD:C_0603_1608Metric
- removed D10: NUP2105L, Package_TO_SOT_SMD:SOT-23
- removed D11: SM712, Package_TO_SOT_SMD:SOT-23
- removed D12, D13, D14, D15, D16, D17, D18, D2, D3: SP0504BAJT, Package_TO_SOT_SMD:SOT-353_SC-70-5
- removed D19: LED, LED_SMD:LED_1206_3216Metric
- removed D20, D21, D22: B230, Diode_SMD:D_SMB
- removed D7, D8, D9: ESDLIN1524BJ, Diode_SMD:D_SOD-323
- removed FB10, FB11, FB12, FB13, FB14, FB15, FB16, FB17, FB18, FB19, FB20, FB21, FB22, FB23, FB24, FB25, FB26, FB27, FB28, FB29, FB30, FB31, FB32, FB33, FB34, FB35, FB36, FB37, FB38, FB39, FB40, FB41, FB42, FB43, FB44, FB6, FB7, FB8, FB9: 100R, Inductor_SMD:L_0603_1608Metric
- removed FB45, FB46, FB47, FB48, FB49: Ferrite, Inductor_SMD:L_0603_1608Metric
- removed J10, J18, J19, J9: WAGO_Klemmleiste_8-pol, WAGO Klemmleisten:WAGO_Klemmleiste_Hebel4mm²Vertikal_RM5mm_8-pol
- removed J11: RJ12, Connector_RJ:RJ12_Amphenol_54601
- removed J12: RJ45, Connector_RJ:RJ45_Amphenol_54602-x08_Horizontal
- removed J13: WAGO_Klemmleiste_6-pol, WAGO Klemmleisten:WAGO_Klemmleiste_Hebel4mm²Vertikal_RM5mm_6-pol
- removed J14: 52271-0679, SamacSys_Parts:52271-0679
- removed J15: Conn_01x06, Connector_PinSocket_2.54mm:PinSocket_1x06_P2.54mm_Vertical
- removed J16: Conn_01x06, SamacSys_Parts:436500628
- removed J17: Conn_01x05, SamacSys_Parts:436500527
- removed J20: Conn_02x03_Top_Bottom, Connectors_Molex:Molex_Microfit3_Header_02x03_Straight_43045-0628
- removed J21: Conn_02x10_Odd_Even, Connector_PinHeader_2.54mm:PinHeader_2x10_P2.54mm_Vertical
- removed J22: Conn_02x06_Odd_Even, Connector_PinHeader_2.54mm:PinHeader_2x06_P2.54mm_Vertical
- removed J23: Conn_02x25_Odd_Even, Connector_PinHeader_2.54mm:PinHeader_2x25_P2.54mm_Vertical
- removed J24: Conn_01x06, Connector_PinHeader_2.54mm:PinHeader_1x06_P2.54mm_Vertical
- removed J8: WAGO_Klemmleiste_4-pol, WAGO Klemmleisten:WAGO_Klemmleiste_Hebel4mm²Vertikal_RM5mm_4-pol
- removed L1, L2, L3, L6: 15uH, Inductor_SMD:L_Coilcraft_XxL4040
- removed L4: L_Core_Ferrite, Inductor_SMD:L_Coilcraft_XxL4020
- removed L5: 10uH, SamacSys_Parts:XAL8080
- removed L7: 4uH7, Inductor_SMD:L_Coilcraft_XxL4030
- removed Q1, Q2, Q3, Q4, Q5, Q6: 2N7002, Package_TO_SOT_SMD:SOT-23
- removed R10, R9: 60R, Resistor_SMD:R_0603_1608Metric
- removed R11: 120R, Resistor_SMD:R_0603_1608Metric
- removed R12, R13, R28, R29, R61, R62, R63, R64, R65, R66, R67, R68, R70, R71, R73, R74: 10k, Resistor_SMD:R_0603_1608Metric
- removed R14: 3M3, Resistor_SMD:R_0603_1608Metric
- removed R15: 432k, Resistor_SMD:R_0603_1608Metric
- removed R16, R17, R18, R19, R20, R30, R31, R33: 40k2, Resistor_SMD:R_0603_1608Metric
- removed R21, R34, R35: 4r7, Resistor_SMD:R_0603_1608Metric
- removed R22, R26: 86k6, Resistor_SMD:R_0603_1608Metric
- removed R23, R27, R52: 32k4, Resistor_SMD:R_0603_1608Metric
- removed R24, R36: 178k, Resistor_SMD:R_0603_1608Metric
- removed R25, R37: 39k, Resistor_SMD:R_0603_1608Metric
- removed R32: 49k9, Resistor_SMD:R_0603_1608Metric
- removed R38: 105k, Resistor_SMD:R_0603_1608Metric
- removed R39: 22k6, Resistor_SMD:R_0603_1608Metric
- removed R40, R41, R42, R43, R44, R45, R46, R47: 4k7, Resistor_SMD:R_0603_1608Metric
- removed R5, R53, R54, R55, R56, R57, R58, R59, R6, R60, R69, R72: 1K, Resistor_SMD:R_0603_1608Metric
- removed R50: 100K, Resistor_SMD:R_0603_1608Metric
- removed R51: 10R 1%, Resistor_SMD:R_0603_1608Metric
- removed R7, R8: 10R, Resistor_SMD:R_0603_1608Metric
- removed R75, R76, R77, R78: 10K, Resistor_SMD:R_0603_1608Metric
- removed U10, U11, U8, U9: MAX17572, Package_DFN_QFN:DFN-12-1EP_3x3mm_P0.5mm_EP2.05x2.86mm
- removed U12: MAX17574, Package_DFN_QFN:QFN-24-1EP_4x5mm_P0.5mm_EP2.65x3.65mm
- removed U13: ESP-12F, RF_Module:ESP-12E
- removed U14: DS2482S-800+, Package_SO:SOIC-16_3.9x9.9mm_P1.27mm
- removed U15: MAX11615, Package_SO:QSOP-16_3.9x4.9mm_P0.635mm
- removed U16: STLD40D, Package_DFN_QFN:DFN-8-1EP_3x3mm_P0.65mm_EP1.55x2.4mm
- removed U17: STM32L4R9ZITx, Package_QFP:LQFP-144_20x20mm_P0.5mm
- removed U18: USBLC6-2SC6, Package_TO_SOT_SMD:SOT-23-6
- removed U19: MOD-nRF8001, RF_Module:MOD-nRF8001
- removed U4, U5: TJA1029T, Package_SO:SOIC-8_3.9x4.9mm_P1.27mm
- removed U6: TJA1049T-3, Package_SO:SOIC-8_3.9x4.9mm_P1.27mm
- removed U7: MAX3072E, Package_SO:SOIC-8_3.9x4.9mm_P1.27mm
- added C104: 5n6, Capacitor_SMD:C_0603_1608Metric, F.Cu at (78.9, 159.1)
- added C105: 2u2, Capacitor_SMD:C_1210_3225Metric, F.Cu at (82.0, 159.0)
- added C106: 100n, Capacitor_SMD:C_0603_1608Metric, F.Cu at (80.7, 156.0)
- added C107: 100nF, Capacitor_SMD:C_0603_1608Metric, F.Cu at (64.6, 167.7)
- added C108: 10uF, Capacitor_SMD:C_1210_3225Metric, F.Cu at (48.8, 162.0)
- added C109: 4u7, Capacitor_SMD:C_1210_3225Metric, F.Cu at (58.1, 159.2)
- added C110: 5n6, Capacitor_SMD:C_0603_1608Metric, F.Cu at (72.9, 158.4)
- added C111: 2u2, Capacitor_SMD:C_1210_3225Metric, F.Cu at (75.1, 163.0)
- added C112: 100nF, Capacitor_SMD:C_0603_1608Metric, F.Cu at (69.9, 160.0)
- added C113: 22uF, Capacitor_SMD:C_1210_3225Metric, F.Cu at (48.8, 168.4)
- added C114: 5n6, Capacitor_SMD:C_0603_1608Metric, F.Cu at (74.7, 154.6)
- added C115: 100n, Capacitor_SMD:C_0603_1608Metric, F.Cu at (83.7, 145.8)
- added C116: 10n, Capacitor_SMD:C_0603_1608Metric, F.Cu at (76.2, 153.1)
- added C117: 4u7, Capacitor_SMD:C_1210_3225Metric, F.Cu at (61.6, 167.7)
- added C118: 10n, Capacitor_SMD:C_0603_1608Metric, F.Cu at (69.1, 163.6)
- added C119: 4u7, Capacitor_SMD:C_1210_3225Metric, F.Cu at (66.1, 162.7)
- added C120: 2u2, Capacitor_SMD:C_1210_3225Metric, F.Cu at (57.2, 169.8)
- added C121: 2u2, Capacitor_SMD:C_1210_3225Metric, F.Cu at (70.6, 166.6)
- added C122: 22nF, Capacitor_SMD:C_0603_1608Metric, F.Cu at (83.7, 155.4)
- added C123: 100nF, Capacitor_SMD:C_0603_1608Metric, F.Cu at (66.1, 164.2)
- added C124: 100nF, Capacitor_SMD:C_0603_1608Metric, F.Cu at (69.9, 158.5)
- added C125: 22uF, Capacitor_SMD:C_1210_3225Metric, F.Cu at (53.5, 159.2)
- added C126: 22uF, Capacitor_SMD:C_1210_3225Metric, F.Cu at (44.2, 165.2)
- added C127: 10u, Capacitor_SMD:C_1210_3225Metric, F.Cu at (72.1, 146.6)
- added C128: 100n, Capacitor_SMD:C_0603_1608Metric, F.Cu at (83.7, 153.8)
- added C129: 1u, Capacitor_SMD:C_0603_1608Metric, F.Cu at (80.9, 149.3)
- added C130: 47u, Capacitor_SMD:C_1210_3225Metric, F.Cu at (48.8, 165.2)
- added C131: 47u, Capacitor_SMD:C_1210_3225Metric, F.Cu at (58.5, 153.2)
- added C132: 2u2, Capacitor_SMD:C_1210_3225Metric, F.Cu at (64.6, 166.2)
- added C133: 5n6, Capacitor_SMD:C_0603_1608Metric, F.Cu at (81.1, 160.6)
- added C134: 100n, Capacitor_SMD:C_0603_1608Metric, F.Cu at (67.6, 167.2)
- added C135: 100nF, Capacitor_SMD:C_0603_1608Metric, F.Cu at (72.9, 159.9)
- added C136: 10uF, Capacitor_SMD:C_1210_3225Metric, F.Cu at (44.2, 168.4)
- added C137: 4u7, Capacitor_SMD:C_1210_3225Metric, F.Cu at (44.2, 162.0)
- added C200: 100nF, Capacitor_SMD:C_0603_1608Metric, F.Cu at (111.8, 11.1)
- added C201: 220pF, Capacitor_SMD:C_0603_1608Metric, F.Cu at (111.8, 12.7)
- added C202: 100nF, Capacitor_SMD:C_0603_1608Metric, F.Cu at (118.4, 6.06)
- added C203: 220pF, Capacitor_SMD:C_0603_1608Metric, F.Cu at (114.6, 14.2)
- added C204: 100nF, Capacitor_SMD:C_0603_1608Metric, F.Cu at (117.9, 12.4)
- added C205: 220pF, Capacitor_SMD:C_0603_1608Metric, F.Cu at (114.9, 10.9)
- added C206: 10uF, Capacitor_SMD:C_1210_3225Metric, F.Cu at (116.9, 0.24)
- added C207: 100nF, Capacitor_SMD:C_0603_1608Metric, F.Cu at (118.4, 7.57)
- added C208: 100nF, Capacitor_SMD:C_0603_1608Metric, F.Cu at (122.4, 2.85)
- added C209: 100nF, Capacitor_SMD:C_0603_1608Metric, F.Cu at (103.1, 22.0)
- added C210: 5n6, Capacitor_SMD:C_0603_1608Metric, F.Cu at (107.4, 19.2)
- added C211: 100nF, Capacitor_SMD:C_0603_1608Metric, F.Cu at (117.6, 13.9)
- added C212: 100nF, Capacitor_SMD:C_0603_1608Metric, F.Cu at (104.4, 20.5)
- added C213: 100nF, Capacitor_SMD:C_0603_1608Metric, F.Cu at (121.4, 10.4)
- added C214: 100nF, Capacitor_SMD:C_0603_1608Metric, F.Cu at (115.3, 7.86)
- added C300: 100pF, Capacitor_SMD:C_0603_1608Metric, F.Cu at (-4.37, 11.7)
- added C301: 100pF, Capacitor_SMD:C_0603_1608Metric, F.Cu at (-1.36, 11.7)
- added C302: 100pF, Capacitor_SMD:C_0603_1608Metric, F.Cu at (69.4, -69.1)
- added C303: 100pF, Capacitor_SMD:C_0603_1608Metric, F.Cu at (72.4, -69.1)
- added C304: 100pF, Capacitor_SMD:C_0603_1608Metric, F.Cu at (75.4, -69.1)
- added C305: 100pF, Capacitor_SMD:C_0603_1608Metric, F.Cu at (72.4, -66.1)
- added C306: 100pF, Capacitor_SMD:C_0603_1608Metric, F.Cu at (1.65, 11.7)
- added C307: 100pF, Capacitor_SMD:C_0603_1608Metric, F.Cu at (-10.4, 11.7)
- added C308: 47u, Capacitor_SMD:C_1210_3225Metric, F.Cu at (-56.5, -8.91)
- added C309: 10u, Capacitor_SMD:C_1210_3225Metric, F.Cu at (-56.5, -5.70)
- added C310: 10u, Capacitor_SMD:C_1210_3225Metric, F.Cu at (-56.5, -2.49)
- added C311: 10u, Capacitor_SMD:C_1210_3225Metric, F.Cu at (-56.5, 0.72)
- added C312: 10u, Capacitor_SMD:C_1210_3225Metric, F.Cu at (-56.5, 3.93)
- added D100: B345BE-13, Diode_SMD:D_SMB, F.Cu at (66.1, 147.3)
- added D101: B345BE-13, Diode_SMD:D_SMB, F.Cu at (36.4, 178.8)
- added D102: B345BE-13, Diode_SMD:D_SMB, F.Cu at (29.1, 178.8)
- added D200: ESDLIN1524BJ, Diode_SMD:D_SOD-323, F.Cu at (120.8, -0.39)
- added D201: ESDLIN1524BJ, Diode_SMD:D_SOD-323, F.Cu at (82.4, 21.7)
- added D202: ESDLIN1524BJ, Diode_SMD:D_SOD-323, F.Cu at (108.8, 8.61)
- added D203: NUP2105L, Package_TO_SOT_SMD:SOT-23, F.Cu at (108.9, 5.86)
- added D204: NUP2105L, Package_TO_SOT_SMD:SOT-23, F.Cu at (93.8, 21.9)
- added D205: SP0504BAJT, Package_TO_SOT_SMD:SOT-353_SC-70-5, F.Cu at (101.3, 16.7)
- added D206: SP0504BAJT, Package_TO_SOT_SMD:SOT-353_SC-70-5, F.Cu at (88.9, 22.2)
- added D207: SP0504BAJT, Package_TO_SOT_SMD:SOT-353_SC-70-5, F.Cu at (85.6, 22.2)
- added D208: SP0504BAJT, Package_TO_SOT_SMD:SOT-353_SC-70-5, F.Cu at (112.2, 5.51)
- added D209: SP0504BAJT, Package_TO_SOT_SMD:SOT-353_SC-70-5, F.Cu at (108.7, 11.0)
- added D210: SP0504BAJT, Package_TO_SOT_SMD:SOT-353_SC-70-5, F.Cu at (101.3, 19.5)
- added D300: B230, Diode_SMD:D_SMB, F.Cu at (-46.6, 10.2)
- added D301: B230, Diode_SMD:D_SMB, F.Cu at (-53.9, 10.2)
- added D302: B230, Diode_SMD:D_SMB, F.Cu at (-61.3, 10.2)
- added D303: SP0504BAJT, Package_TO_SOT_SMD:SOT-353_SC-70-5, F.Cu at (-27.9, 9.34)
- added D304: SP0504BAJT, Package_TO_SOT_SMD:SOT-353_SC-70-5, F.Cu at (-31.1, 9.34)
- added D305: SP0504BAJT, Package_TO_SOT_SMD:SOT-353_SC-70-5, F.Cu at (-34.4, 9.34)
- added FB100: 100R, Inductor_SMD:L_0603_1608Metric, F.Cu at (57.7, 155.5)
- added FB101: 100R, Inductor_SMD:L_0603_1608Metric, F.Cu at (61.6, 166.2)
- added FB200: 100R, Inductor_SMD:L_0603_1608Metric, F.Cu at (121.4, 8.89)
- added FB201: 100R, Inductor_SMD:L_0603_1608Metric, F.Cu at (106.1, 22.2)
- added FB202: 100R, Inductor_SMD:L_0603_1608Metric, F.Cu at (113.4, 15.7)
- added FB203: 100R, Inductor_SMD:L_0603_1608Metric, F.Cu at (110.4, 19.2)
- added FB204: 100R, Inductor_SMD:L_0603_1608Metric, F.Cu at (117.9, 10.9)
- added FB205: 100R, Inductor_SMD:L_0603_1608Metric, F.Cu at (111.6, 14.2)
- added FB206: 100R, Inductor_SMD:L_0603_1608Metric, F.Cu at (121.4, 7.38)
- added FB207: 100R, Inductor_SMD:L_0603_1608Metric, F.Cu at (107.4, 17.7)
- added FB208: 100R, Inductor_SMD:L_0603_1608Metric, F.Cu at (110.4, 16.2)
- added FB209: 100R, Inductor_SMD:L_0603_1608Metric, F.Cu at (113.4, 17.2)
- added FB210: 100R, Inductor_SMD:L_0603_1608Metric, F.Cu at (121.4, 5.87)
- added FB211: 100R, Inductor_SMD:L_0603_1608Metric, F.Cu at (118.4, 9.08)
- added FB212: 100R, Inductor_SMD:L_0603_1608Metric, F.Cu at (114.8, 12.4)
- added FB213: 100R, Inductor_SMD:L_0603_1608Metric, F.Cu at (110.4, 17.7)
- added FB214: 100R, Inductor_SMD:L_0603_1608Metric, F.Cu at (121.4, 4.36)
- added FB300: 100R, Inductor_SMD:L_0603_1608Metric, F.Cu at (-63.4, 6.54)
- added FB301: 100R, Inductor_SMD:L_0603_1608Metric, F.Cu at (-57.4, 6.54)
- added FB302: 100R, Inductor_SMD:L_0603_1608Metric, F.Cu at (69.4, -64.6)
- added FB303: 100R, Inductor_SMD:L_0603_1608Metric, F.Cu at (69.4, -67.6)
- added FB304: 100R, Inductor_SMD:L_0603_1608Metric, F.Cu at (-7.38, 11.7)
- added FB305: 100R, Inductor_SMD:L_0603_1608Metric, F.Cu at (-54.4, 6.29)
- added FB306: 100R, Inductor_SMD:L_0603_1608Metric, F.Cu at (-24.7, 10.2)
- added FB307: 100R, Inductor_SMD:L_0603_1608Metric, F.Cu at (-21.7, 8.67)
- added FB308: 100R, Inductor_SMD:L_0603_1608Metric, F.Cu at (75.4, -63.1)
- added FB309: 100R, Inductor_SMD:L_0603_1608Metric, F.Cu at (72.4, -63.1)
- added FB310: 100R, Inductor_SMD:L_0603_1608Metric, F.Cu at (75.4, -64.6)
- added FB311: 100R, Inductor_SMD:L_0603_1608Metric, F.Cu at (-10.4, 10.2)
- added FB312: 100R, Inductor_SMD:L_0603_1608Metric, F.Cu at (-13.4, 10.8)
- added FB313: 100R, Inductor_SMD:L_0603_1608Metric, F.Cu at (-16.4, 10.8)
- added FB314: 100R, Inductor_SMD:L_0603_1608Metric, F.Cu at (-15.7, 9.25)
- added FB315: 100R, Inductor_SMD:L_0603_1608Metric, F.Cu at (-12.5, 8.67)
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Connections:
- C1 pad 1: RESET -> VCCQ
- C100 pad 1: +3.3VP -> +BATT
- C100 pad 2: GND1 -> GND
- C101 pad 1: VCC -> Net-(C101-Pad1)
- C101 pad 2: GND1 -> Net-(C101-Pad2)
- C102 pad 1: +3.3VP -> +3V3
- C102 pad 2: GND1 -> GND
- C12 pad 1: GND1 -> VCCQ
- C12 pad 2: Net-(C12-Pad2) -> GND1
- C13 pad 1: GND1 -> VCCQ
- C13 pad 2: Net-(C13-Pad2) -> GND1
- C14 pad 1: GND -> GND1
- C14 pad 2: +3V3 -> VCCQ
- C15 pad 1: VCC -> GND1
- C15 pad 2: GND1 -> VCCQ
- C16 pad 1: GND -> GND1
- C16 pad 2: +BATT -> VCCQ
- C17 pad 1: GND -> GND1
- C17 pad 2: +BATT -> Net-(C17-Pad2)
- C18 pad 1: GND -> Net-(BT1-Pad1)
- C18 pad 2: +BATT -> GND1
- C19 pad 1: Net-(C19-Pad1) -> RESET
- C19 pad 2: GND -> GND1
- C2 pad 1: Net-(C2-Pad1) -> VCCQ
- C20 pad 1: Net-(C20-Pad1) -> VCCQ
- C20 pad 2: GND -> GND1
- C21 pad 2: GND -> GND1
- C22 pad 1: +3V3 -> Net-(C22-Pad1)
- C22 pad 2: GND -> GND1
- C23 pad 1: GND -> GND1
- C23 pad 2: +3V3 -> Net-(C23-Pad2)
- C24 pad 1: GND -> GND1
- C24 pad 2: +5V -> Net-(C24-Pad2)
- C25 pad 1: Net-(C25-Pad1) -> VCC
- C25 pad 2: GND -> GND1
- C26 pad 1: +BATT -> VCC
- C26 pad 2: GND -> GND1
- C27 pad 1: +BATT -> GND1
- C27 pad 2: GND -> VCC
- C28 pad 1: +BATT -> VCCQ
- C28 pad 2: GND -> GND1
- C29 pad 1: Net-(C29-Pad1) -> VCCQ
- C29 pad 2: GND -> GND1
- C3 pad 1: Net-(C3-Pad1) -> VCCQ
- C30 pad 1: Net-(C30-Pad1) -> VCCQ
- C30 pad 2: GND -> GND1
- C31 pad 1: Net-(C31-Pad1) -> VCCQ
- C31 pad 2: GND -> GND1
- C32 pad 1: Net-(C32-Pad1) -> VCCQ
- C32 pad 2: GND -> GND1
- C33 pad 1: Net-(C33-Pad1) -> VCCQ
- C33 pad 2: Net-(C33-Pad2) -> GND1
- C34 pad 1: Net-(C34-Pad1) -> +3.3VP
- C34 pad 2: Net-(C34-Pad2) -> GND1
- C35 pad 1: Net-(C35-Pad1) -> VCCQ
- C35 pad 2: Net-(C35-Pad2) -> GND1
- C36 pad 1: GND -> VCC
- C36 pad 2: Net-(C36-Pad2) -> GND1
- C37 pad 1: +3V3 -> +3.3VP
- C37 pad 2: GND -> GND1
- D1 pad 1: Net-(D1-Pad1) -> GND1
- D1 pad 2: LCD_LED-A -> Signal_LED
- FB1 pad 1: LIN3 -> VCCQ
- FB1 pad 2: Net-(C21-Pad1) -> Net-(FB1-Pad2)
- FB2 pad 1: LIN1 -> *LCD_LED-K
- FB2 pad 2: Net-(C19-Pad1) -> Net-(FB2-Pad2)
- FB3 pad 1: LIN2 -> Net-(FB3-Pad1)
- FB3 pad 2: Net-(C20-Pad1) -> +3.3VP
- FB4 pad 1: CAN-H -> Net-(FB4-Pad1)
- FB4 pad 2: Net-(D10-Pad2) -> VCC
- FB5 pad 1: CAN-L -> Net-(FB5-Pad1)
- FB5 pad 2: Net-(D10-Pad1) -> *LCD_LED-A
- J1 pad 1: Net-(J1-Pad1) -> GND1
- J1 pad 2: +4V -> GND1
- J1 pad 3: Net-(J1-Pad3) -> *LPUART_TX_RS485
- J1 pad 4: UART4_TX -> *USART1_TX_LIN1
- J1 pad 5: UART4_RX -> *LPUART_RX_RX485
- J1 pad 6: GND -> *USART1_RX_LIN1
- J2 pad 1: GND -> *LCD_LED-K
- J2 pad 10: USART2_RX_LIN2 -> LCD_R5
- J2 pad 11: CAN1_RX -> LCD_R6
- J2 pad 12: USART3_TX_LIN3 -> LCD_R7
- J2 pad 13: I2C2_SCL -> LCD_G0
- J2 pad 14: USART3_RX_LIN3 -> LCD_G1
- J2 pad 15: I2C2_SDA -> LCD_G2
- J2 pad 16: UART4_TX -> LCD_G3
- J2 pad 17: I2C4_SCL -> LCD_G4
- J2 pad 18: UART4_RX -> LCD_G5
- J2 pad 19: I2C4_SDA -> LCD_G6
- J2 pad 2: GND -> *LCD_LED-A
- J2 pad 20: UART5_TX -> LCD_G7
- J2 pad 21: PWR_Reset -> LCD_B0
- J2 pad 22: UART5_RX -> LCD_B1
- J2 pad 23: GND -> LCD_B2
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
Commit message: Bauteil Gruppierungen im Layout
Parts:
- moved R101 111.7 mm to (-19.7, 108.7), turned to 270 degrees
- moved R100 105.8 mm to (-19.7, 105.9), turned to 270 degrees
- moved C100 101.5 mm to (-12.8, 114.3)
- moved R102 101.0 mm to (-17.8, 115.6)
- moved L106 100.8 mm to (129.5, 101.6)
- moved C101 100.5 mm to (-8.89, 106.2), turned to 270 degrees
- moved C136 100.0 mm to (128.3, 114.3)
- moved C104 98.7 mm to (-7.62, 111.8)
- moved R104 98.3 mm to (-16.5, 111.8)
- moved U100 96.2 mm to (-12.2, 107.4)
- moved C137 93.6 mm to (128.1, 120.7), turned to 180 degrees
- moved R103 93.1 mm to (-7.14, 115.6)
- moved R105 89.4 mm to (6.83, 101.6)
- moved R128 88.4 mm to (123.2, 101.6)
- moved C106 85.5 mm to (17.0, 99.1)
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Connections:
- D101 pad 2: DC_Input -> Net-(D101-Pad2)
- D102 pad 2: DC_Input -> Net-(D101-Pad2)
- F1 pad 1: +BATT -> Net-(D101-Pad2)
- F1 pad 2: Net-(F1-Pad2) -> DC_Input
- L105 pad 1: Net-(F1-Pad2) -> +BATT
- L105 pad 2: DC_Input -> Net-(D101-Pad2)
Other:
- copper layers 2 -> 4
- net class Octo added: clearance 0.2, trace_width 0.25, via_dia 0.8, via_drill 0.4
