File: Hardware/Board/Womo.kicad_pcb (KiCad board)
At the start: 4 copper layers, 319 parts, among them IC1 MX25LM51245GXDI00, IC2 IS66WVH8M8BLL-100B1LI_0, IC3 TSC2007, J1 Conn_02x25_Odd_Even, J2 54104-4031, J3 52271-0679, J300 Power In, J301 1Wire 1-4, J302 1Wire 5-8, J303 LIN 1-3, J304 Truma, J305 Dormetic, J306 Analog 1-4, J307 Analog 5-8, J308 Wasser, J309 Abwasser, J310 CAN + RS485, J311 Schaudt EBL, J312 Spare, J313 CPU, J314 SIM800-1, J315 SIM800-2, J316 Raspberry_Pi_2_3, J4 Conn_02x06_Odd_Even, J5 Spare, J6 USB_B_Micro, J7 Conn_ARM_JTAG_SWD_20, Q100 2N7002, Q102 2N7002, Q103 2N7002, Q104 2N7002, Q300 2N7002, Q301 2N7002, SW1 Boot, SW2 Wakeup, SW3 Reset, U1 STM32L4R9ZITx, U100 MAX17572, U101 MAX17572, U102 MAX17572, U103 STLD40D, U104 MAX17574, U105 MAX17572, U2 USBLC6-2SC6, U200 TJA1029T, U201 TJA1029T, U202 TJA1029T, U203 TJA1049T-3, U204 MAX3072E, U205 DS2482S-800+, U206 PCF8574A, U207 PCF8574A, U208 MAX11615, U3 MOD-nRF8001, U300 ESP-12F, Y1 16 MHz, Y2 32.768

Commit message: Schaltplan: Pulldown bei den Mosfets zugefügt, Fehler Korrektur, Baulteil Footprints zugewiesen und Lib angepasst, Netztliste ohne Fehler zum Layout übertragbar. Board: Auf neues Design angepasst, Beginn der platzierung der Teile nach Funktionsgruppen
Parts:
- removed C115: 100n, Capacitor_SMD:C_0603_1608Metric
- removed C116, C118: 10n, Capacitor_SMD:C_0603_1608Metric
- removed C117, C119: 4u7, Capacitor_SMD:C_1210_3225Metric
- removed C307: 100pF, Capacitor_SMD:C_0603_1608Metric
- removed C308: 47u, Capacitor_SMD:C_1210_3225Metric
- removed C309, C310, C311, C312, C34: 10u, Capacitor_SMD:C_1210_3225Metric
- removed C32, C33: 100nF, Capacitor_SMD:C_0603_1608Metric
- removed C35, C36, C37: 1uF, Capacitor_SMD:C_0603_1608Metric
- removed D100: B345BE-13, Diode_SMD:D_SMB
- removed F1: KFZ 5A, Fuse:Fuseholder_Blade_ATO_Littelfuse_Pudenz_2_Pin
- removed FB100, FB101: 100R, Inductor_SMD:L_0603_1608Metric
- removed FB4, FB5: Ferrite, Inductor_SMD:L_0603_1608Metric
- removed IC2: IS66WVH8M8BLL-100B1LI_0, SamacSys_Parts:BGA24C100P5X5_600X800X35
- removed IC3: TSC2007, Package_SO:TSSOP-16_4.4x5mm_P0.65mm
- removed J4: Conn_02x06_Odd_Even, Connector_PinHeader_2.54mm:PinHeader_2x06_P2.54mm_Vertical
- removed J5: Spare, Connector_PinHeader_2.54mm:PinHeader_1x06_P2.54mm_Vertical
- removed J6: USB_B_Micro, Connector_USB:USB_Micro-B_Molex-105017-0001
- removed J7: Conn_ARM_JTAG_SWD_20, Connector_IDC:IDC-Header_2x10_P2.54mm_Vertical
- removed L103: 4uH7, Inductor_SMD:L_Coilcraft_XxL4030
- removed Q300, Q301: 2N7002, Package_TO_SOT_SMD:SOT-23
- removed R48, R49: 10K, Resistor_SMD:R_0603_1608Metric
- removed SW2: Wakeup, Button_Switch_THT:SW_PUSH_6mm_H8.5mm
- removed U103: STLD40D, Package_DFN_QFN:DFN-8-1EP_3x3mm_P0.65mm_EP1.55x2.4mm
- added C138: 47u, Capacitor_SMD:C_1210_3225Metric, F.Cu at (202.7, 209.6)
- added C139: 47u, Capacitor_SMD:C_1210_3225Metric, F.Cu at (198.0, 209.6)
- added C215: 100nF, Capacitor_SMD:C_0603_1608Metric, F.Cu at (341.7, 237.0)
- added C216: 100nF, Capacitor_SMD:C_0603_1608Metric, F.Cu at (304.5, 239.3)
- added C217: 100nF, Capacitor_SMD:C_0603_1608Metric, F.Cu at (186.7, 19.0)
- added C218: 100nF, Capacitor_SMD:C_0603_1608Metric, F.Cu at (199.5, 6.07)
- added C219: 5n6, Capacitor_SMD:C_0603_1608Metric, F.Cu at (201.2, 10.8)
- added C220: 10uF, Capacitor_SMD:C_1210_3225Metric, F.Cu at (161.8, 24.2)
- added C221: 100nF, Capacitor_SMD:C_0603_1608Metric, F.Cu at (209.2, 1.03)
- added C222: 100nF, Capacitor_SMD:C_0603_1608Metric, F.Cu at (203.1, 3.22)
- added C223: 100nF, Capacitor_SMD:C_0603_1608Metric, F.Cu at (180.5, 25.5)
- added C224: 100nF, Capacitor_SMD:C_0603_1608Metric, F.Cu at (183.5, 22.5)
- added C225: 100nF, Capacitor_SMD:C_0603_1608Metric, F.Cu at (205.6, 0.37)
- added C226: 100nF, Capacitor_SMD:C_0603_1608Metric, F.Cu at (208.9, -1.99)
- added C227: 47u, Capacitor_SMD:C_1210_3225Metric, F.Cu at (171.7, 244.9)
- added C228: 47u, Capacitor_SMD:C_1210_3225Metric, F.Cu at (181.2, 244.9)
- added C229: 47u, Capacitor_SMD:C_1210_3225Metric, F.Cu at (190.1, 244.9)
- added C230: 47u, Capacitor_SMD:C_1210_3225Metric, F.Cu at (199.0, 244.9)
- added C315: 10u, Capacitor_SMD:C_1210_3225Metric, F.Cu at (280.8, -48.3)
- added C316: 100nF, Capacitor_SMD:C_0603_1608Metric, F.Cu at (268.0, -48.5)
- added C317: 100nF, Capacitor_SMD:C_0603_1608Metric, F.Cu at (249.9, -59.9)
- added C318: 10u, Capacitor_SMD:C_1210_3225Metric, F.Cu at (273.7, -59.4)
- added C319: 10u, Capacitor_SMD:C_1210_3225Metric, F.Cu at (287.1, -59.2)
- added C320: 100nF, Capacitor_SMD:C_0603_1608Metric, F.Cu at (255.5, -42.7)
- added C321: 100pF, Capacitor_SMD:C_0603_1608Metric, F.Cu at (329.4, 260.9)
- added C322: 100pF, Capacitor_SMD:C_0603_1608Metric, F.Cu at (331.5, 260.9)
- added C323: 100pF, Capacitor_SMD:C_0603_1608Metric, F.Cu at (334.5, 260.9)
- added C324: 100pF, Capacitor_SMD:C_0603_1608Metric, F.Cu at (337.1, 260.8)
- added C325: 100pF, Capacitor_SMD:C_0603_1608Metric, F.Cu at (339.3, 260.6)
- added C326: 100pF, Capacitor_SMD:C_0603_1608Metric, F.Cu at (341.6, 260.6)
- added C327: 100pF, Capacitor_SMD:C_0603_1608Metric, F.Cu at (344.2, 260.8)
- added C328: 100pF, Capacitor_SMD:C_0603_1608Metric, F.Cu at (347.0, 261.1)
- added C400: 100nF, Capacitor_SMD:C_0603_1608Metric, F.Cu at (126.0, 248.6)
- added C401: 100nF, Capacitor_SMD:C_0603_1608Metric, F.Cu at (115.3, 264.7)
- added C402: 100nF, Capacitor_SMD:C_0603_1608Metric, F.Cu at (127.7, 264.9)
- added C403: 4u7, Capacitor_SMD:C_0603_1608Metric, F.Cu at (117.1, 245.8)
- added C404: 100nF, Capacitor_SMD:C_0603_1608Metric, F.Cu at (115.3, 245.9)
- added C405: 5n6, Capacitor_SMD:C_0603_1608Metric, F.Cu at (121.4, 237.2)
- added C500: 100nF, Capacitor_SMD:C_0603_1608Metric, F.Cu at (109.5, 172.7)
- added C501: 100nF, Capacitor_SMD:C_0603_1608Metric, F.Cu at (96.0, 173.0)
- added C502: 100nF, Capacitor_SMD:C_0603_1608Metric, F.Cu at (96.7, 178.6)
- added C503: 100nF, Capacitor_SMD:C_0603_1608Metric, F.Cu at (103.1, 173.0)
- added C504: 10uF, Capacitor_SMD:C_0603_1608Metric, F.Cu at (103.1, 179.1)
- added C505: 220nF, Capacitor_SMD:C_0603_1608Metric, F.Cu at (109.2, 179.6)
- added D211: SP0504BAJT, Package_TO_SOT_SMD:SOT-353_SC-70-5, F.Cu at (312.8, 258.1)
- added D212: NUP2105L, Package_TO_SOT_SMD:SOT-23, F.Cu at (208.7, -6.03)
- added D213: SP0504BAJT, Package_TO_SOT_SMD:SOT-353_SC-70-5, F.Cu at (192.0, 12.8)
- added D214: SP0504BAJT, Package_TO_SOT_SMD:SOT-353_SC-70-5, F.Cu at (169.7, 0.17)
- added D215: SP0504BAJT, Package_TO_SOT_SMD:SOT-353_SC-70-5, F.Cu at (188.0, 16.4)
- added D216: SP0504BAJT, Package_TO_SOT_SMD:SOT-353_SC-70-5, F.Cu at (205.7, -1.81)
- added D217: B345BE-13, Diode_SMD:D_SMB, F.Cu at (161.8, 233.7)
- added D218: B345BE-13, Diode_SMD:D_SMB, F.Cu at (167.4, 233.7)
- added D306: NUP2105L, Package_TO_SOT_SMD:SOT-23, F.Cu at (258.8, -23.4)
- added D400: NUP2105L, Package_TO_SOT_SMD:SOT-23, F.Cu at (121.4, 233.7)
- added D9: D, Diode_SMD:D_SOD-323, F.Cu at (169.7, 2.57)
- added F100: KFZ 5A, Fuse:Fuseholder_Blade_ATO_Littelfuse_Pudenz_2_Pin, F.Cu at (154.9, 244.3)
- added F200: KFZ 10A, Fuse:Fuseholder_Blade_ATO_Littelfuse_Pudenz_2_Pin, F.Cu at (164.8, 244.3)
- added FB215: 100R, Inductor_SMD:L_0603_1608Metric, F.Cu at (208.9, -3.50)
- added FB216: 100R, Inductor_SMD:L_0603_1608Metric, F.Cu at (189.5, 24.6)
- added FB217: 100R, Inductor_SMD:L_0603_1608Metric, F.Cu at (195.1, 11.6)
- added FB218: 100R, Inductor_SMD:L_0603_1608Metric, F.Cu at (186.7, 20.5)
- added FB219: 100R, Inductor_SMD:L_0603_1608Metric, F.Cu at (209.2, 5.56)
- added FB220: 100R, Inductor_SMD:L_0603_1608Metric, F.Cu at (200.9, 14.5)
- added FB221: 100R, Inductor_SMD:L_0603_1608Metric, F.Cu at (194.9, 15.0)
- added FB222: 100R, Inductor_SMD:L_0603_1608Metric, F.Cu at (183.5, 24.0)
- added FB223: 100R, Inductor_SMD:L_0603_1608Metric, F.Cu at (203.1, 4.73)
- added FB224: 100R, Inductor_SMD:L_0603_1608Metric, F.Cu at (189.8, 18.6)
- added FB225: 100R, Inductor_SMD:L_0603_1608Metric, F.Cu at (199.5, 9.09)
- added FB226: 100R, Inductor_SMD:L_0603_1608Metric, F.Cu at (208.9, -0.48)
- added FB227: 100R, Inductor_SMD:L_0603_1608Metric, F.Cu at (195.1, 13.1)
- added FB228: 100R, Inductor_SMD:L_0603_1608Metric, F.Cu at (191.1, 16.5)
- added FB229: 100R, Inductor_SMD:L_0603_1608Metric, F.Cu at (206.1, 1.88)
- added FB327: 100R, Inductor_SMD:L_0603_1608Metric, F.Cu at (309.1, 262.7)
- added FB328: 100R, Inductor_SMD:L_0603_1608Metric, F.Cu at (311.7, 262.7)
- added FB329: 100R, Inductor_SMD:L_0603_1608Metric, F.Cu at (314.2, 262.7)
- added FB330: 100R, Inductor_SMD:L_0603_1608Metric, F.Cu at (316.7, 262.7)
- added FB331: 100R, Inductor_SMD:L_0603_1608Metric, F.Cu at (249.9, -36.6)
- added FB332: 100R, Inductor_SMD:L_0603_1608Metric, F.Cu at (255.8, -59.4)
- added FB333: 100R, Inductor_SMD:L_0603_1608Metric, F.Cu at (261.8, -59.7)
- added FB334: 100R, Inductor_SMD:L_0603_1608Metric, F.Cu at (267.9, -36.8)
- added FB335: 100R, Inductor_SMD:L_0603_1608Metric, F.Cu at (280.6, -54.1)
- added FB336: 100R, Inductor_SMD:L_0603_1608Metric, F.Cu at (329.2, 256.5)
- added FB337: 100R, Inductor_SMD:L_0603_1608Metric, F.Cu at (331.5, 256.6)
- added FB338: 100R, Inductor_SMD:L_0603_1608Metric, F.Cu at (334.5, 256.6)
- added FB339: 100R, Inductor_SMD:L_0603_1608Metric, F.Cu at (337.1, 256.6)
- added FB340: 100R, Inductor_SMD:L_0603_1608Metric, F.Cu at (339.3, 256.8)
- added FB341: 100R, Inductor_SMD:L_0603_1608Metric, F.Cu at (341.6, 256.8)
- added FB342: 100R, Inductor_SMD:L_0603_1608Metric, F.Cu at (344.4, 256.8)
- added FB343: 100R, Inductor_SMD:L_0603_1608Metric, F.Cu at (347.0, 256.8)
- added FB400: 100R, Inductor_SMD:L_0603_1608Metric, F.Cu at (126.0, 244.9)
- added FB401: 100R, Inductor_SMD:L_0603_1608Metric, F.Cu at (118.6, 231.9)
- added FB402: 100R, Inductor_SMD:L_0603_1608Metric, F.Cu at (124.2, 231.9)
- added IC200: BTS6143D, Womo-Lin:BTS6143D, F.Cu at (173.7, 254.1)
- added IC201: BTS6143D, Womo-Lin:BTS6143D, F.Cu at (182.6, 254.1)
- added IC203: BTS6143D, Womo-Lin:BTS6143D, F.Cu at (191.5, 254.1)
- added IC204: BTS6143D, Womo-Lin:BTS6143D, F.Cu at (200.4, 254.0)
- added J317: RJ45_Shielded, Connector_RJ:RJ45_Amphenol_RJHSE5380, F.Cu at (-32.0, 186.9)
- added J318: Spare, Connector_PinHeader_2.54mm:PinHeader_2x10_P2.54mm_Vertical, F.Cu at (-64.3, 24.1)
- added J319: SENSOR, Connector_IDC:IDC-Header_2x05_P2.54mm_Vertical, F.Cu at (-57.2, 144.1)
- added J320: Raspberry_Pi_2_3, Connector_IDC:IDC-Header_2x20_P2.54mm_Vertical, F.Cu at (154.6, -65.7)
- added J321: Wasser, Womo-Lin:436500628, F.Cu at (321.1, 244.9)
- added J322: Abwasser, Womo-Lin:436500527, F.Cu at (354.1, 246.6)
- added J323: 733-370, WAGO Klemmleisten:SHDR10W80P0X250_1X10_2750X890X780P, F.Cu at (326.6, 267.0)
- added J324: Waveshare IoT Hat, Connector_IDC:IDC-Header_2x20_P2.54mm_Vertical, F.Cu at (-66.9, 144.1)
- added J325: 734-168, WAGO Klemmleisten:SHDR8W150P350X350_1X8_3040X1030X860P, F.Cu at (172.0, 265.7)
- added J326: 733-366, WAGO Klemmleisten:SHDR6W80P0X250_1X6_1750X890X780P, F.Cu at (163.4, -20.2)
- added J400: USB_B_Micro, Connector_USB:USB_Micro-B_Molex-105017-0001, F.Cu at (120.7, 270.8)
- added J401: RJ45_Shielded, Connector_RJ:RJ45_Amphenol_RJHSE5380, F.Cu at (118.6, 220.2)
- added J500: SENSOR, Connector_IDC:IDC-Header_2x05_P2.54mm_Vertical, F.Cu at (126.2, 181.9)
- added K300: 5-1393243-2, Womo-Lin:513932432, F.Cu at (237.0, 259.8)
- added K301: 5-1393243-2, Womo-Lin:513932432, F.Cu at (252.0, 259.8)
- added K302: 5-1393243-2, Womo-Lin:513932432, F.Cu at (267.0, 259.8)
- added K303: 5-1393243-2, Womo-Lin:513932432, F.Cu at (281.9, 259.8)
- added L200: L_Core_Ferrite, Inductor_SMD:L_Coilcraft_XxL4020, F.Cu at (174.2, 240.6)
- added L201: L_Core_Ferrite, Inductor_SMD:L_Coilcraft_XxL4020, F.Cu at (182.6, 240.6)
- added L202: L_Core_Ferrite, Inductor_SMD:L_Coilcraft_XxL4020, F.Cu at (191.5, 240.5)
- added L203: L_Core_Ferrite, Inductor_SMD:L_Coilcraft_XxL4020, F.Cu at (200.4, 240.4)
- added Q200: 2N7002, Package_TO_SOT_SMD:SOT-23, F.Cu at (173.2, 235.5)
- added Q201: 2N7002, Package_TO_SOT_SMD:SOT-23, F.Cu at (181.9, 234.9)
- added Q202: 2N7002, Package_TO_SOT_SMD:SOT-23, F.Cu at (191.3, 235.2)
- added Q203: 2N7002, Package_TO_SOT_SMD:SOT-23, F.Cu at (201.9, 235.7)
- added R131: 22k6, Resistor_SMD:R_0603_1608Metric, F.Cu at (206.5, 208.8)
- added R219: 47k, Resistor_SMD:R_0603_1608Metric, F.Cu at (195.8, 18.0)
- added R220: 10R, Resistor_SMD:R_0603_1608Metric, F.Cu at (205.5, 7.92)
- added R221: 120R, Resistor_SMD:R_0603_1608Metric, F.Cu at (201.2, 12.3)
- added R222: 10R, Resistor_SMD:R_0603_1608Metric, F.Cu at (197.1, 16.5)
- added R223: 47k, Resistor_SMD:R_0603_1608Metric, F.Cu at (209.2, 4.05)
- added R224: 47k, Resistor_SMD:R_0603_1608Metric, F.Cu at (192.8, 21.1)
- added R225: 10R, Resistor_SMD:R_0603_1608Metric, F.Cu at (192.8, 19.5)
- added R226: 120R, Resistor_SMD:R_0603_1608Metric, F.Cu at (205.5, 6.41)
- added R227: 10R, Resistor_SMD:R_0603_1608Metric, F.Cu at (189.8, 23.1)
- added R228: 10K, Resistor_SMD:R_0603_1608Metric, F.Cu at (326.9, 236.0)
- added R229: 10K, Resistor_SMD:R_0603_1608Metric, F.Cu at (323.1, 236.0)
- added R230: 60R, Resistor_SMD:R_0603_1608Metric, F.Cu at (209.2, 2.54)
- added R231: 60R, Resistor_SMD:R_0603_1608Metric, F.Cu at (189.8, 21.6)
- added R232: 4k7, Resistor_SMD:R_0603_1608Metric, F.Cu at (186.5, 25.0)
- added R234: 4k7, Resistor_SMD:R_0603_1608Metric, F.Cu at (206.1, 4.90)
- added R235: 4k7, Resistor_SMD:R_0603_1608Metric, F.Cu at (198.2, 13.0)
- added R236: 4k7, Resistor_SMD:R_0603_1608Metric, F.Cu at (206.1, 3.39)
- added R237: 4k7, Resistor_SMD:R_0603_1608Metric, F.Cu at (189.8, 20.1)
- added R238: 4k7, Resistor_SMD:R_0603_1608Metric, F.Cu at (202.5, 6.24)
- added R239: 4k7, Resistor_SMD:R_0603_1608Metric, F.Cu at (198.2, 11.5)
- added R240: 4k7, Resistor_SMD:R_0603_1608Metric, F.Cu at (186.5, 23.5)
- added R241: 10k, Resistor_SMD:R_0603_1608Metric, F.Cu at (177.0, 236.2)
- added R242: 1k, Resistor_SMD:R_0603_1608Metric, F.Cu at (194.1, 16.5)
- added R243: 100k, Resistor_SMD:R_0603_1608Metric, F.Cu at (177.0, 233.4)
- added R244: 10k, Resistor_SMD:R_0603_1608Metric, F.Cu at (185.6, 236.5)
- added R245: 1k, Resistor_SMD:R_0603_1608Metric, F.Cu at (186.7, 22.0)
- added R246: 100k, Resistor_SMD:R_0603_1608Metric, F.Cu at (185.7, 233.9)
- added R247: 10k, Resistor_SMD:R_0603_1608Metric, F.Cu at (195.8, 236.5)
- added R248: 1k, Resistor_SMD:R_0603_1608Metric, F.Cu at (169.6, 4.30)
- added R249: 100k, Resistor_SMD:R_0603_1608Metric, F.Cu at (195.6, 233.7)
- added R250: 10k, Resistor_SMD:R_0603_1608Metric, F.Cu at (206.0, 237.2)
- added R251: 1k, Resistor_SMD:R_0603_1608Metric, F.Cu at (196.5, 8.43)
- added R252: 100k, Resistor_SMD:R_0603_1608Metric, F.Cu at (206.0, 234.9)
- added R400: 60R, Resistor_SMD:R_0603_1608Metric, F.Cu at (119.6, 239.8)
- added R401: 60R, Resistor_SMD:R_0603_1608Metric, F.Cu at (122.9, 239.8)
- added R5: 47K, Resistor_SMD:R_0603_1608Metric, F.Cu at (286.0, 204.7)
- added R502: 10K, Resistor_SMD:R_0603_1608Metric, F.Cu at (105.4, 189.7)
- added R503: 10K, Resistor_SMD:R_0603_1608Metric, F.Cu at (109.7, 189.7)
- added R6: 47K, Resistor_SMD:R_0603_1608Metric, F.Cu at (293.5, 195.6)
- added R7: 47K, Resistor_SMD:R_0603_1608Metric, F.Cu at (293.5, 197.1)
- added R8: 47K, Resistor_SMD:R_0603_1608Metric, F.Cu at (289.8, 201.0)
- added U209: MAX3072E, Package_SO:SOIC-8_3.9x4.9mm_P1.27mm, F.Cu at (170.7, 19.3)
- added U210: MAX3072E, Package_SO:SOIC-8_3.9x4.9mm_P1.27mm, F.Cu at (183.8, 5.47)
- added U211: MAX11615, Package_SO:QSOP-16_3.9x4.9mm_P0.635mm, F.Cu at (337.7, 241.4)
- added U212: PCF8574A, Package_SO:SOIC-16W_7.5x10.3mm_P1.27mm, F.Cu at (307.8, 247.9)
- added U213: TJA1049T-3, Package_SO:SOIC-8_3.9x4.9mm_P1.27mm, F.Cu at (183.2, 10.9)
- added U214: DS2482S-800+, Package_SO:SOIC-16_3.9x9.9mm_P1.27mm, F.Cu at (163.2, 17.3)
- added U215: SN74LV4052A, Package_SO:TSSOP-16_4.4x5mm_P0.65mm, F.Cu at (49.6, 141.4)
- added U216: Si8642BB-B-IS1, Package_SO:SOIC-16_3.9x9.9mm_P1.27mm, F.Cu at (183.8, -2.53)
- added U217: Si8642BB-B-IS1, Package_SO:SOIC-16_3.9x9.9mm_P1.27mm, F.Cu at (191.2, -2.53)
- added U301: max4896atp+, Womo-Lin:max4896atp&plus_, F.Cu at (217.0, 255.1)
- added U302: TJA1049T-3, Package_SO:SOIC-8_3.9x4.9mm_P1.27mm, F.Cu at (243.5, -68.6)
- added U303: ESP-12F, RF_Module:ESP-12E, F.Cu at (375.2, 43.9)
- added U304: TJA1049T-3, Package_SO:SOIC-8_3.9x4.9mm_P1.27mm, F.Cu at (250.2, -23.9)
- added U4: MOD-nRF8001, RF_Module:MOD-nRF8001, F.Cu at (361.9, 177.0)
- added U400: USBLC6-2SC6, Package_TO_SOT_SMD:SOT-23-6, F.Cu at (119.5, 264.7)
- added U401: FT232RL, Package_SO:SSOP-28_5.3x10.2mm_P0.65mm, F.Cu at (120.9, 256.5)
- added U402: TJA1049T-3, Package_SO:SOIC-8_3.9x4.9mm_P1.27mm, F.Cu at (121.3, 245.8)
- added U5: USBLC6-2SC6, Package_TO_SOT_SMD:SOT-23-6, F.Cu at (346.4, 198.9)
- added U500: BME680, Package_LGA:Bosch_LGA-8_3x3mm_P0.8mm_ClockwisePinNumbering, F.Cu at (114.6, 189.7)
- added U501: LSM303AGR, Package_LGA:LGA-12_2x2mm_P0.5mm, F.Cu at (116.3, 183.1)
- added U6: TJA1049T-3, Package_SO:SOIC-8_3.9x4.9mm_P1.27mm, F.Cu at (340.1, 117.1)
- C128: value 100n -> 2u2; footprint Capacitor_SMD:C_0603_1608Metric -> Capacitor_SMD:C_1210_3225Metric
- C129: value 1u -> 2u2; footprint Capacitor_SMD:C_0603_1608Metric -> Capacitor_SMD:C_1210_3225Metric
- C130: value 47u -> 22nF; footprint Capacitor_SMD:C_1210_3225Metric -> Capacitor_SMD:C_0603_1608Metric
- C131: value 47u -> 100nF; footprint Capacitor_SMD:C_1210_3225Metric -> Capacitor_SMD:C_0603_1608Metric
- C132: value 2u2 -> 100nF; footprint Capacitor_SMD:C_1210_3225Metric -> Capacitor_SMD:C_0603_1608Metric
- C133: value 5n6 -> 22uF; footprint Capacitor_SMD:C_0603_1608Metric -> Capacitor_SMD:C_1210_3225Metric
- C134: value 100n -> 22uF; footprint Capacitor_SMD:C_0603_1608Metric -> Capacitor_SMD:C_1210_3225Metric
- C135: value 100nF -> 10u; footprint Capacitor_SMD:C_0603_1608Metric -> Capacitor_SMD:C_1210_3225Metric
- C136: value 10uF -> 100n; footprint Capacitor_SMD:C_1210_3225Metric -> Capacitor_SMD:C_0603_1608Metric
- C137: value 4u7 -> 1u; footprint Capacitor_SMD:C_1210_3225Metric -> Capacitor_SMD:C_0603_1608Metric
- C201, C203, C205: value 220pF -> 100nF
- C202, C204, C208: value 100nF -> 220pF
- C206: value 10uF -> 220pF; footprint Capacitor_SMD:C_1210_3225Metric -> Capacitor_SMD:C_0603_1608Metric
- C210: value 5n6 -> 100nF
- C23, C24: value 3p3 -> 4p7
- C25, C26: value 1uF -> 10u; footprint Capacitor_SMD:C_0603_1608Metric -> Capacitor_SMD:C_1210_3225Metric
- C27: value 100n -> 100nF
- C30: value 100nF -> 1u
- C300, C301, C304, C305: value 100pF -> 100nF
- C302: value 100pF -> 47u; footprint Capacitor_SMD:C_0603_1608Metric -> Capacitor_SMD:C_1210_3225Metric
- C303: value 100pF -> 10u; footprint Capacitor_SMD:C_0603_1608Metric -> Capacitor_SMD:C_1210_3225Metric
- C306: value 100pF -> 5n6
- D203: value NUP2105L -> ESDLIN1524BJ; footprint Package_TO_SOT_SMD:SOT-23 -> Diode_SMD:D_SOD-323
- D205, D206, D207: value SP0504BAJT -> NUP2105L; footprint Package_TO_SOT_SMD:SOT-353_SC-70-5 -> Package_TO_SOT_SMD:SOT-23
- D300, D301, D302: value B230 -> SP0504BAJT; footprint Diode_SMD:D_SMB -> Package_TO_SOT_SMD:SOT-353_SC-70-5
- FB1, FB2, FB3: value Ferrite -> 100R
- IC1: value MX25LM51245GXDI00 -> SPSGRFC-868; footprint SamacSys_Parts:BGA24C100P5X5_600X800X35 -> Womo-Lin:SPSGRFC868
- J1: value Conn_02x25_Odd_Even -> USB_B_Micro; footprint Connector_PinHeader_2.54mm:PinHeader_2x25_P2.54mm_Vertical -> Connector_USB:USB_Micro-B_Molex-105017-0001
- J2: value 54104-4031 -> Conn_ARM_JTAG_SWD_20; footprint SamacSys_Parts:54104-4031 -> Connector_IDC:IDC-Header_2x10_P2.54mm_Vertical
- J3: value 52271-0679 -> SD_Card; footprint SamacSys_Parts:52271-0679 -> Connector_Card:10067847-001RLF
- J300: value Power In -> 734-264; footprint WAGO Klemmleisten:WAGO_Klemmleiste_Hebel4mm²Vertikal_RM5mm_4-pol -> WAGO Klemmleisten:SHDR4W120P0X381_1X4_1640X1030X850P
- J301: value 1Wire 1-4 -> 733-368; footprint WAGO Klemmleisten:WAGO_Klemmleiste_Hebel4mm²Vertikal_RM5mm_8-pol -> WAGO Klemmleisten:SHDR8W80P0X250_1X8_2250X890X780P
- J302: value 1Wire 5-8 -> 733-368; footprint WAGO Klemmleisten:WAGO_Klemmleiste_Hebel4mm²Vertikal_RM5mm_8-pol -> WAGO Klemmleisten:SHDR8W80P0X250_1X8_2250X890X780P
- J303: value LIN 1-3 -> 733-368; footprint WAGO Klemmleisten:WAGO_Klemmleiste_Hebel4mm²Vertikal_RM5mm_6-pol -> WAGO Klemmleisten:SHDR8W80P0X250_1X8_2250X890X780P
- J306: value Analog 1-4 -> 733-366; footprint WAGO Klemmleisten:WAGO_Klemmleiste_Hebel4mm²Vertikal_RM5mm_8-pol -> WAGO Klemmleisten:SHDR6W80P0X250_1X6_1750X890X780P
- J307: value Analog 5-8 -> 733-366; footprint WAGO Klemmleisten:WAGO_Klemmleiste_Hebel4mm²Vertikal_RM5mm_8-pol -> WAGO Klemmleisten:SHDR6W80P0X250_1X6_1750X890X780P
- J308: value Wasser -> 733-366; footprint SamacSys_Parts:436500628 -> WAGO Klemmleisten:SHDR6W80P0X250_1X6_1750X890X780P
- J309: value Abwasser -> 733-366; footprint SamacSys_Parts:436500527 -> WAGO Klemmleisten:SHDR6W80P0X250_1X6_1750X890X780P
- J310: value CAN + RS485 -> 733-370; footprint WAGO Klemmleisten:WAGO_Klemmleiste_Hebel4mm²Vertikal_RM5mm_6-pol -> WAGO Klemmleisten:SHDR10W80P0X250_1X10_2750X890X780P
- J311: value Schaudt EBL -> 734-163; footprint Connectors_Molex:Molex_Microfit3_Header_02x03_Straight_43045-0628 -> WAGO Klemmleisten:SHDR3W100P0X350_1X3_1290X1030X850P
- J312: value Spare -> 734-163; footprint Connector_PinHeader_2.54mm:PinHeader_2x10_P2.54mm_Vertical -> WAGO Klemmleisten:SHDR3W100P0X350_1X3_1290X1030X850P
- J313: value CPU -> 734-163; footprint Connector_PinSocket_2.54mm:PinSocket_2x25_P2.54mm_Vertical -> WAGO Klemmleisten:SHDR3W100P0X350_1X3_1290X1030X850P
- J314: value SIM800-1 -> 734-163; footprint Connector_PinHeader_2.54mm:PinHeader_1x06_P2.54mm_Vertical -> WAGO Klemmleisten:SHDR3W100P0X350_1X3_1290X1030X850P
- J315: value SIM800-2 -> 734-168; footprint Connector_PinSocket_2.54mm:PinSocket_1x06_P2.54mm_Vertical -> WAGO Klemmleisten:SHDR8W150P350X350_1X8_3040X1030X860P
- J316: value Raspberry_Pi_2_3 -> 733-363; footprint Connector_IDC:IDC-Header_2x20_P2.54mm_Vertical -> WAGO Klemmleisten:SHDR3W80P0X250_1X3_1000X890X780P
- L104: footprint SamacSys_Parts:XAL8080 -> Womo-Lin:XAL8080
- L105: value L_Core_Ferrite -> 10uH; footprint Inductor_SMD:L_Coilcraft_XxL4020 -> Womo-Lin:XAL8080
- L106: value 15uH -> L_Core_Ferrite; footprint Inductor_SMD:L_Coilcraft_XxL4040 -> Inductor_SMD:L_Coilcraft_XxL4020
- R105, R125: value 10k -> 100k
- R106, R113, R126: value 40k2 -> 10k
- R108: value 4r7 -> 40k2
- R109: value 178k -> 4r7
- R110: value 39k -> 178k
- R111: value 10k -> 39k
- R112: value 40k2 -> 100k
- R114: value 86k6 -> 40k2
- R115: value 32k4 -> 40k2
- R116: value 100K -> 86k6
- R117: value 10R 1% -> 32k4
- R118: value 32k4 -> 100k
- R128: value 178k -> 49k9
- R129: value 39k -> 4r7
- R130: value 4r7 -> 105k
- R2: value 10K -> 1k
- R206: value 60R -> 10K
- R207: value 60R -> 1K
- R208: value 10R -> 47k
- R209: value 120R -> 47k
- R211, R216: value 4k7 -> 120R
- R212, R215, R217: value 4k7 -> 10R
- R213, R214, R218: value 4k7 -> 47k
- R3, R4: value 10K -> 47K
- R300, R301: value 1K -> 60R
- R304, R305, R312, R313: value 10k -> 1K
- R308, R309, R317: value 1K -> 10k
- R318, R320, R321: value 10k -> 47K
- R319: value 1K -> 47K
- U1: value STM32L4R9ZITx -> STM32L476ZGTx
- U105: value MAX17572 -> MAX17574; footprint Package_DFN_QFN:DFN-12-1EP_3x3mm_P0.5mm_EP2.05x2.86mm -> Package_DFN_QFN:QFN-24-1EP_4x5mm_P0.5mm_EP2.65x3.65mm
- U2: value USBLC6-2SC6 -> M25Q128A; footprint Package_TO_SOT_SMD:SOT-23-6 -> Package_SO:SOIJ-8_5.3x5.3mm_P1.27mm
- U200: value TJA1029T -> SN74LV4052A; footprint Package_SO:SOIC-8_3.9x4.9mm_P1.27mm -> Package_SO:TSSOP-16_4.4x5mm_P0.65mm
- U203: value TJA1049T-3 -> TJA1029T
- U204: value MAX3072E -> TJA1029T
- U205: value DS2482S-800+ -> SN74LV4052A; footprint Package_SO:SOIC-16_3.9x9.9mm_P1.27mm -> Package_SO:TSSOP-16_4.4x5mm_P0.65mm
- U206: value PCF8574A -> SN74LV4052A; footprint Package_SO:SOIC-16W_7.5x10.3mm_P1.27mm -> Package_SO:TSSOP-16_4.4x5mm_P0.65mm
- U207: value PCF8574A -> MAX3072E; footprint Package_SO:SOIC-16W_7.5x10.3mm_P1.27mm -> Package_SO:SOIC-8_3.9x4.9mm_P1.27mm
- U208: value MAX11615 -> MAX3072E; footprint Package_SO:QSOP-16_3.9x4.9mm_P0.635mm -> Package_SO:SOIC-8_3.9x4.9mm_P1.27mm
- U3: value MOD-nRF8001 -> 24AA02UID; footprint RF_Module:MOD-nRF8001 -> Package_TO_SOT_SMD:SOT-23-5
- U300: value ESP-12F -> max4896atp+; footprint RF_Module:ESP-12E -> Womo-Lin:max4896atp&plus_
- Y1: value 16 MHz -> 25 MHz
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Connections:
- net Net-(U200-Pad3) renamed UART4_TX_LIN
- BT1 pad 2: GND1 -> GND
- C1 pad 1: VCCQ -> +3V3
- C1 pad 2: GND1 -> Net-(C1-Pad2)
- C10 pad 1: VCCQ -> +3V3
- C10 pad 2: GND1 -> GND
- C11 pad 1: VCCQ -> +3V3
- C11 pad 2: GND1 -> GND
- C12 pad 1: VCCQ -> +3V3
- C12 pad 2: GND1 -> GND
- C128 pad 1: DC_Input -> +BATT
- C129 pad 1: DC_Input -> +BATT
- C13 pad 1: VCCQ -> +3V3
- C13 pad 2: GND1 -> Net-(C13-Pad2)
- C130 pad 1: +BATT -> Net-(C130-Pad1)
- C131 pad 1: +BATT -> Net-(C131-Pad1)
- C131 pad 2: GND -> Net-(C131-Pad2)
- C132 pad 1: +BATT -> +5VL
- C133 pad 1: Net-(C133-Pad1) -> +5VL
- C134 pad 1: Net-(C134-Pad1) -> +5VL
- C135 pad 1: Net-(C135-Pad1) -> GND
- C136 pad 1: +VSW -> DC_Input
- C137 pad 1: GND -> DC_Input
- C137 pad 2: Net-(C137-Pad2) -> GND
- C14 pad 1: GND1 -> Net-(C13-Pad2)
- C14 pad 2: VCCQ -> +3V3
- C15 pad 1: GND1 -> Net-(C13-Pad2)
- C15 pad 2: VCCQ -> +3V3
- C16 pad 1: GND1 -> Net-(C13-Pad2)
- C16 pad 2: VCCQ -> Net-(C16-Pad2)
- C17 pad 1: GND1 -> Net-(C13-Pad2)
- C17 pad 2: Net-(C17-Pad2) -> Net-(C16-Pad2)
- C18 pad 2: GND1 -> GND
- C19 pad 2: GND1 -> GND
- C2 pad 1: VCCQ -> +3V3
- C2 pad 2: GND1 -> Net-(C1-Pad2)
- C20 pad 1: VCCQ -> Net-(C20-Pad1)
- C20 pad 2: GND1 -> GND
- C200 pad 1: GND -> +3.3VA
- C200 pad 2: +BATT -> GND
- C201 pad 1: Net-(C201-Pad1) -> GND
- C201 pad 2: GND -> +BATT
- C202 pad 1: GND -> Net-(C202-Pad1)
- C202 pad 2: +BATT -> GND
- C203 pad 1: Net-(C203-Pad1) -> GND
- C203 pad 2: GND -> +BATT
- C204 pad 1: GND -> Net-(C204-Pad1)
- C204 pad 2: +BATT -> GND
- C205 pad 1: Net-(C205-Pad1) -> GND
- C205 pad 2: GND -> +BATT
- C206 pad 1: +3.3VA -> Net-(C206-Pad1)
- C207 pad 1: +3.3VA -> GND
- C207 pad 2: GND -> +BATT
- C208 pad 1: +3V3 -> Net-(C208-Pad1)
- C209 pad 1: GND -> +3.3VA
- C209 pad 2: +5V -> GND
- C21 pad 2: GND1 -> GND
- C210 pad 1: Net-(C210-Pad1) -> +3.3VA
- C211 pad 2: +3V3 -> +3.3VA
- C212 pad 2: +3V3 -> +3.3VA
- C213 pad 2: +3V3 -> +3.3VA
- C214 pad 2: +3V3 -> +3.3VA
- C22 pad 2: GND1 -> GND
- C23 pad 1: GND1 -> GND
- C24 pad 1: GND1 -> GND
- C25 pad 1: VCC -> +3.3VA
- C25 pad 2: GND1 -> GND
- C26 pad 1: VCC -> +3.3VA
- C26 pad 2: GND1 -> GND
- C27 pad 1: GND1 -> +3V3
- C27 pad 2: VCC -> GND
- C28 pad 1: VCCQ -> +3.3VA
- C28 pad 2: GND1 -> GND
- C29 pad 1: VCCQ -> GND
- C29 pad 2: GND1 -> +5V
- C3 pad 1: VCCQ -> +3V3
- C3 pad 2: GND1 -> Net-(C1-Pad2)
- C30 pad 1: VCCQ -> GND
- C30 pad 2: GND1 -> +3.3VA
- C300 pad 1: Net-(C300-Pad1) -> GND
- C300 pad 2: GND -> +3.3VA
- C301 pad 1: Net-(C301-Pad1) -> GND
- C301 pad 2: GND -> +3.3VA
- C302 pad 1: Net-(C302-Pad1) -> +5VD
- C304 pad 1: Net-(C304-Pad1) -> Net-(C303-Pad1)
- C305 pad 1: Net-(C305-Pad1) -> GND
- C305 pad 2: GND -> +5VD
- C31 pad 1: VCCQ -> +3V3
- C31 pad 2: GND1 -> GND
- C4 pad 1: VCCQ -> +3V3
- C4 pad 2: GND1 -> Net-(C1-Pad2)
- C5 pad 1: VCCQ -> +3V3
- C5 pad 2: GND1 -> Net-(C1-Pad2)
- C6 pad 1: VCCQ -> +3V3
- C6 pad 2: GND1 -> Net-(C1-Pad2)
- C7 pad 1: VCCQ -> +3V3
- C7 pad 2: GND1 -> Net-(C1-Pad2)
- C8 pad 1: VCCQ -> +3V3
- C8 pad 2: GND1 -> Net-(C1-Pad2)
- C9 pad 1: VCCQ -> +3V3
- C9 pad 2: GND1 -> Net-(C1-Pad2)
- D1 pad 1: GND1 -> GND
- D200 pad 1: Net-(C201-Pad1) -> Net-(C202-Pad1)
- D201 pad 1: Net-(C203-Pad1) -> Net-(C204-Pad1)
- D202 pad 1: Net-(C205-Pad1) -> Net-(C206-Pad1)
- D203 pad 1: Net-(D203-Pad1) -> Net-(C208-Pad1)
- D203 pad 2: Net-(D203-Pad2) -> GND
- D205 pad 2: GND -> Net-(D205-Pad2)
- D205 pad 3: Net-(D205-Pad3) -> GND
- D206 pad 2: GND -> Net-(D206-Pad2)
- D206 pad 3: Net-(D206-Pad3) -> GND
- D207 pad 1: P0 -> Net-(D207-Pad1)
- D207 pad 2: GND -> Net-(D207-Pad2)
- D207 pad 3: P1 -> GND
- D208 pad 1: P4 -> AIN0
- D208 pad 3: P5 -> AIN1
- D208 pad 4: P6 -> AIN2
- D208 pad 5: P7 -> AIN3
- D209 pad 1: AIN0 -> AIN4
- D209 pad 3: AIN1 -> AIN5
- D209 pad 4: AIN2 -> AIN6
- D209 pad 5: AIN3 -> AIN7
- D210 pad 1: AIN4 -> P0
- D210 pad 3: AIN5 -> P1
- D210 pad 4: AIN6 -> P2
- D210 pad 5: AIN7 -> P3
- D300 pad 1: Net-(D300-Pad1) -> PF4
- D300 pad 2: +5VD -> GND
- D301 pad 1: Net-(D301-Pad1) -> PF0
- D301 pad 2: Net-(D300-Pad1) -> GND
- D302 pad 1: +4V -> PF8
- D302 pad 2: Net-(D301-Pad1) -> GND
- D303 pad 1: PC6 -> PF12
- D303 pad 3: PC7 -> PF13
- D303 pad 4: Net-(D303-Pad4) -> I2C1_SDA
- D303 pad 5: PB2 -> I2C1SCL
- D304 pad 1: P4 -> INt_2_XL
- D304 pad 3: P5 -> INT_MAG_DRDY
- D304 pad 4: P6 -> INT_1_XL
- D304 pad 5: P7 -> I2C3_SCL
- D305 pad 1: I2C4_SDA -> I2C3_SDA
- D305 pad 3: I2C4_SCL -> I2C1_SDA
- D305 pad 4: PF11 -> I2C1_SCL
- FB1 pad 1: VCCQ -> Net-(C16-Pad2)
- FB1 pad 2: Net-(FB1-Pad2) -> Net-(C20-Pad1)
- FB2 pad 1: *LCD_LED-K -> Net-(C16-Pad2)
- FB2 pad 2: Net-(FB2-Pad2) -> +3V3
- FB200 pad 2: Net-(C201-Pad1) -> Net-(C202-Pad1)
- FB201 pad 2: Net-(C203-Pad1) -> Net-(C204-Pad1)
- FB202 pad 2: Net-(C205-Pad1) -> Net-(C206-Pad1)
- FB203 pad 1: 1Wire_P7 -> LIN4
- FB203 pad 2: Net-(D206-Pad1) -> Net-(C208-Pad1)
- FB204 pad 1: 1Wire_P6 -> RS485_1_A
- FB204 pad 2: Net-(D206-Pad3) -> Net-(D204-Pad2)
- FB205 pad 1: 1Wire_P5 -> RS485_1_B
- FB205 pad 2: Net-(D206-Pad4) -> Net-(D204-Pad1)
- FB206 pad 1: 1Wire_P4 -> RS485_2_A
- FB206 pad 2: Net-(D206-Pad5) -> Net-(D205-Pad2)
- FB207 pad 1: 1Wire_P3 -> RS485_2_B
- FB208 pad 1: 1Wire_P2 -> RS485_3_A
- FB208 pad 2: Net-(D205-Pad3) -> Net-(D206-Pad2)
- FB209 pad 1: 1Wire_P1 -> RS485_3_B
- FB209 pad 2: Net-(D205-Pad4) -> Net-(D206-Pad1)
- FB210 pad 1: 1Wire_P0 -> RS485_4_A
- FB210 pad 2: Net-(D205-Pad5) -> Net-(D207-Pad2)
- FB211 pad 1: CAN-H -> RS485_4_B
- FB211 pad 2: Net-(D203-Pad2) -> Net-(D207-Pad1)
- FB212 pad 1: CAN-L -> CAN-H
- FB212 pad 2: Net-(D203-Pad1) -> Net-(D212-Pad2)
- FB213 pad 1: RS485-A -> CAN-L
- FB213 pad 2: Net-(D204-Pad2) -> Net-(D212-Pad1)
- FB214 pad 1: RS485-B -> 1Wire_P7
- FB214 pad 2: Net-(D204-Pad1) -> Net-(D214-Pad1)
- FB3 pad 2: +3.3VP -> +3.3VA
- FB300 pad 1: Net-(C300-Pad1) -> Net-(FB300-Pad1)
- FB300 pad 2: Net-(FB300-Pad2) -> PF0
- FB301 pad 1: Net-(C301-Pad1) -> Net-(FB301-Pad1)
- FB301 pad 2: Net-(FB301-Pad2) -> PF1
- FB302 pad 1: Net-(C302-Pad1) -> Net-(FB302-Pad1)
- FB302 pad 2: Net-(FB302-Pad2) -> PF2
- FB303 pad 1: Net-(C303-Pad1) -> Net-(FB303-Pad1)
- FB303 pad 2: Net-(FB303-Pad2) -> PF3
- FB304 pad 1: Net-(C304-Pad1) -> Net-(FB304-Pad1)
- FB304 pad 2: Net-(FB304-Pad2) -> PF4
- FB305 pad 1: Net-(C305-Pad1) -> Net-(FB305-Pad1)
- FB305 pad 2: Net-(FB305-Pad2) -> PF5
- FB306 pad 1: Net-(C306-Pad1) -> Net-(FB306-Pad1)
- FB306 pad 2: Net-(FB306-Pad2) -> PF6
- FB307 pad 1: Net-(C307-Pad1) -> Net-(FB307-Pad1)
- FB307 pad 2: Net-(FB307-Pad2) -> PF7
- FB308 pad 2: Net-(FB308-Pad2) -> +3V3
- FB309 pad 2: Net-(FB309-Pad2) -> +3.3VA
- FB310 pad 2: Net-(FB310-Pad2) -> PF8
- FB311 pad 2: Net-(FB311-Pad2) -> PF9
- FB312 pad 2: P4 -> PF10
- FB313 pad 2: P5 -> PF11
- FB314 pad 2: P6 -> PF12
- FB315 pad 2: P7 -> PF13
- FB316 pad 2: PC6 -> I2C1_SDA
- FB317 pad 2: PC7 -> I2C1SCL
- FB318 pad 1: Net-(FB318-Pad1) -> INt_2_XL
- FB318 pad 2: Net-(D303-Pad4) -> Net-(FB318-Pad2)
- FB319 pad 1: Net-(FB319-Pad1) -> INT_MAG_DRDY
- FB319 pad 2: PB2 -> Net-(FB319-Pad2)
- FB320 pad 1: Net-(FB320-Pad1) -> INT_1_XL
- FB320 pad 2: +3V3 -> Net-(FB320-Pad2)
- FB321 pad 1: Net-(FB321-Pad1) -> I2C3_SCL
- FB321 pad 2: +5V -> Net-(FB321-Pad2)
- FB322 pad 1: Net-(FB322-Pad1) -> I2C3_SDA
- FB322 pad 2: +VSW -> Net-(FB322-Pad2)
- FB323 pad 2: +3.3VA -> P0
- FB324 pad 2: PF11 -> P1
- FB325 pad 2: I2C4_SCL -> P2
- FB326 pad 2: I2C4_SDA -> P3
- J1 pad 1: GND1 -> Net-(J1-Pad1)
- J1 pad 2: GND1 -> Net-(J1-Pad2)
- J1 pad 3: *LPUART_TX_RS485 -> Net-(J1-Pad3)
- J1 pad 4: *USART1_TX_LIN1 -> USB_ID
- J1 pad 5: *LPUART_RX_RX485 -> GND
- J1 pad 6: *USART1_RX_LIN1 -> GND
- J2 pad 1: *LCD_LED-K -> Net-(J2-Pad1)
- J2 pad 10: LCD_R5 -> GND
- J2 pad 11: LCD_R6 -> Net-(J2-Pad11)
- J2 pad 12: LCD_R7 -> GND
- J2 pad 13: LCD_G0 -> JTAG_TDO
- J2 pad 14: LCD_G1 -> GND
- J2 pad 15: LCD_G2 -> Net-(J2-Pad15)
- J2 pad 16: LCD_G3 -> GND
- J2 pad 17: LCD_G4 -> Net-(J2-Pad17)
- J2 pad 18: LCD_G5 -> GND
- J2 pad 19: LCD_G6 -> Net-(J2-Pad19)
- J2 pad 2: *LCD_LED-A -> +3V3
- J2 pad 20: LCD_G7 -> GND
- J2 pad 3: GND1 -> JTAG_RES
- J2 pad 4: VCC -> GND
- J2 pad 5: LCD_R0 -> JTAG_TDI
- J2 pad 6: LCD_R1 -> GND
- J2 pad 7: LCD_R2 -> JTAG_TMS
- J2 pad 8: LCD_R3 -> GND
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
Commit message: Schaltplan: Kleinere Korrekturen Layout: I/O Ports Gröstenteils platziert
Parts:
- removed D204, D206: NUP2105L, Package_TO_SOT_SMD:SOT-23
- removed D4, D5: D, Diode_SMD:D_SOD-323
- added D219: SP0504BAJT, Package_TO_SOT_SMD:SOT-353_SC-70-5, F.Cu at (254.1, 136.3)
- added D220: SP0504BAJT, Package_TO_SOT_SMD:SOT-353_SC-70-5, F.Cu at (234.2, 136.3)
- added D221: B345BE-13, Diode_SMD:D_SMB, F.Cu at (175.3, 222.9)
- added D222: B345BE-13, Diode_SMD:D_SMB, F.Cu at (167.9, 222.9)
- D200, D202: value ESDLIN1524BJ -> D
- D205, D207: value NUP2105L -> ESDLIN1524BJ; footprint Package_TO_SOT_SMD:SOT-23 -> Diode_SMD:D_SOD-323
- D208, D209, D210, D211, D216: value SP0504BAJT -> NUP2105L; footprint Package_TO_SOT_SMD:SOT-353_SC-70-5 -> Package_TO_SOT_SMD:SOT-23
- D212: value NUP2105L -> SP0504BAJT; footprint Package_TO_SOT_SMD:SOT-23 -> Package_TO_SOT_SMD:SOT-353_SC-70-5
- D217, D218: value B345BE-13 -> SP0504BAJT; footprint Diode_SMD:D_SMB -> Package_TO_SOT_SMD:SOT-353_SC-70-5
- D6: value D -> 204
- D9: value D -> 206
- moved FB306 522.8 mm to (477.9, 153.7)
- moved C306 522.8 mm to (504.3, 155.2)
- moved D303 522.8 mm to (474.8, 152.8)
- moved FB304 522.8 mm to (495.3, 155.2)
- moved FB307 522.8 mm to (481.0, 152.2)
- moved FB311 522.8 mm to (492.3, 153.7)
- moved FB312 522.8 mm to (489.3, 154.3)
- moved FB313 522.8 mm to (486.3, 154.3)
- moved FB314 522.8 mm to (487.0, 152.8)
- moved FB315 522.8 mm to (490.2, 152.2)
- moved FB316 522.8 mm to (484.0, 152.8)
- moved R300 522.8 mm to (507.3, 153.7)
- moved R301 522.8 mm to (498.3, 152.2)
- moved R319 522.8 mm to (504.3, 153.7)
- moved R320 522.8 mm to (501.3, 153.7)
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Connections:
- D200 pad 1: Net-(C202-Pad1) -> Net-(D200-Pad1)
- D200 pad 2: GND -> +BATT
- D201 pad 1: Net-(C204-Pad1) -> Net-(C202-Pad1)
- D202 pad 1: Net-(C206-Pad1) -> Net-(D202-Pad1)
- D202 pad 2: GND -> +BATT
- D203 pad 1: Net-(C208-Pad1) -> Net-(C204-Pad1)
- D205 pad 1: Net-(D205-Pad1) -> Net-(C206-Pad1)
- D205 pad 2: Net-(D205-Pad2) -> GND
- D207 pad 1: Net-(D207-Pad1) -> Net-(C208-Pad1)
- D207 pad 2: Net-(D207-Pad2) -> GND
- D208 pad 1: AIN0 -> Net-(D208-Pad1)
- D208 pad 2: GND -> Net-(D208-Pad2)
- D208 pad 3: AIN1 -> GND
- D209 pad 1: AIN4 -> Net-(D209-Pad1)
- D209 pad 2: GND -> Net-(D209-Pad2)
- D209 pad 3: AIN5 -> GND
- D210 pad 1: P0 -> Net-(D210-Pad1)
- D210 pad 2: GND -> Net-(D210-Pad2)
- D210 pad 3: P1 -> GND
- D211 pad 1: P4 -> Net-(D211-Pad1)
- D211 pad 2: GND -> Net-(D211-Pad2)
- D211 pad 3: P5 -> GND
- D212 pad 1: Net-(D212-Pad1) -> AIN0
- D212 pad 2: Net-(D212-Pad2) -> GND
- D212 pad 3: GND -> AIN1
- D213 pad 1: Net-(D213-Pad1) -> AIN4
- D213 pad 3: Net-(D213-Pad3) -> AIN5
- D213 pad 4: Net-(D213-Pad4) -> AIN6
- D213 pad 5: Net-(D213-Pad5) -> AIN7
- D214 pad 1: Net-(D214-Pad1) -> P0
- D214 pad 3: Net-(D214-Pad3) -> P1
- D214 pad 4: Net-(D214-Pad4) -> P2
- D214 pad 5: Net-(D214-Pad5) -> P3
- D215 pad 1: Net-(D215-Pad1) -> P4
- D215 pad 3: Net-(D215-Pad3) -> P5
- D215 pad 4: Net-(D215-Pad4) -> P6
- D215 pad 5: Net-(D215-Pad5) -> P7
- D216 pad 2: GND -> Net-(D216-Pad2)
- D216 pad 3: Net-(D216-Pad3) -> GND
- D217 pad 1: GND -> Net-(D217-Pad1)
- D217 pad 2: Net-(D217-Pad2) -> GND
- D218 pad 1: GND -> Net-(D218-Pad1)
- D218 pad 2: Net-(D217-Pad2) -> GND
- F200 pad 1: Net-(D217-Pad2) -> Net-(D221-Pad2)
- FB204 pad 2: Net-(D204-Pad2) -> Net-(D208-Pad1)
- FB205 pad 2: Net-(D204-Pad1) -> Net-(D208-Pad2)
- FB206 pad 2: Net-(D205-Pad2) -> Net-(D209-Pad1)
- FB207 pad 2: Net-(D205-Pad1) -> Net-(D209-Pad2)
- FB208 pad 2: Net-(D206-Pad2) -> Net-(D210-Pad1)
- FB209 pad 2: Net-(D206-Pad1) -> Net-(D210-Pad2)
- FB210 pad 2: Net-(D207-Pad2) -> Net-(D211-Pad1)
- FB211 pad 2: Net-(D207-Pad1) -> Net-(D211-Pad2)
- FB212 pad 2: Net-(D212-Pad2) -> Net-(D216-Pad1)
- FB213 pad 2: Net-(D212-Pad1) -> Net-(D216-Pad2)
- FB214 pad 2: Net-(D214-Pad1) -> Net-(D218-Pad1)
- FB215 pad 2: Net-(D214-Pad3) -> Net-(D218-Pad3)
- FB216 pad 2: Net-(D214-Pad4) -> Net-(D218-Pad4)
- FB217 pad 2: Net-(D214-Pad5) -> Net-(D218-Pad5)
- FB218 pad 2: Net-(D213-Pad1) -> Net-(D217-Pad1)
- FB219 pad 2: Net-(D213-Pad3) -> Net-(D217-Pad3)
- FB220 pad 2: Net-(D213-Pad4) -> Net-(D217-Pad4)
- FB221 pad 2: Net-(D213-Pad5) -> Net-(D217-Pad5)
- FB222 pad 2: Net-(D215-Pad1) -> Net-(D219-Pad1)
- FB223 pad 2: Net-(D215-Pad3) -> Net-(D219-Pad3)
- FB224 pad 2: Net-(D215-Pad4) -> Net-(D219-Pad4)
- FB225 pad 2: Net-(D215-Pad5) -> Net-(D219-Pad5)
- FB226 pad 2: Net-(D216-Pad1) -> Net-(D220-Pad1)
- FB227 pad 2: Net-(D216-Pad3) -> Net-(D220-Pad3)
- FB228 pad 2: Net-(D216-Pad4) -> Net-(D220-Pad4)
- FB229 pad 2: Net-(D216-Pad5) -> Net-(D220-Pad5)
- L200 pad 2: Net-(D217-Pad2) -> Net-(D221-Pad2)
- L201 pad 2: Net-(D217-Pad2) -> Net-(D221-Pad2)
- L202 pad 2: Net-(D217-Pad2) -> Net-(D221-Pad2)
- L203 pad 2: Net-(D217-Pad2) -> Net-(D221-Pad2)
- R201 pad 1: Net-(D4-Pad1) -> Net-(D200-Pad1)
- R203 pad 1: Net-(D5-Pad1) -> Net-(D202-Pad1)
- R210 pad 1: Net-(D204-Pad2) -> Net-(D208-Pad1)
- R211 pad 1: Net-(D204-Pad2) -> Net-(D208-Pad1)
- R211 pad 2: Net-(D204-Pad1) -> Net-(D208-Pad2)
- R212 pad 1: Net-(D204-Pad1) -> Net-(D208-Pad2)
- R215 pad 1: Net-(D205-Pad2) -> Net-(D209-Pad1)
- R216 pad 1: Net-(D205-Pad2) -> Net-(D209-Pad1)
- R216 pad 2: Net-(D205-Pad1) -> Net-(D209-Pad2)
- R217 pad 1: Net-(D205-Pad1) -> Net-(D209-Pad2)
- R220 pad 1: Net-(D206-Pad2) -> Net-(D210-Pad1)
- R221 pad 1: Net-(D206-Pad2) -> Net-(D210-Pad1)
- R221 pad 2: Net-(D206-Pad1) -> Net-(D210-Pad2)
- R222 pad 1: Net-(D206-Pad1) -> Net-(D210-Pad2)
- R225 pad 1: Net-(D207-Pad2) -> Net-(D211-Pad1)
- R226 pad 1: Net-(D207-Pad2) -> Net-(D211-Pad1)
- R226 pad 2: Net-(D207-Pad1) -> Net-(D211-Pad2)
- R227 pad 1: Net-(D207-Pad1) -> Net-(D211-Pad2)
- R230 pad 1: Net-(D212-Pad2) -> Net-(D216-Pad1)
- R231 pad 2: Net-(D212-Pad1) -> Net-(D216-Pad2)
- R232 pad 2: Net-(D214-Pad1) -> Net-(D218-Pad1)
- R234 pad 2: Net-(D214-Pad3) -> Net-(D218-Pad3)
- R235 pad 2: Net-(D214-Pad4) -> Net-(D218-Pad4)
- R236 pad 2: Net-(D214-Pad5) -> Net-(D218-Pad5)
- R237 pad 2: Net-(D213-Pad1) -> Net-(D217-Pad1)
- R238 pad 2: Net-(D213-Pad3) -> Net-(D217-Pad3)
- R239 pad 2: Net-(D213-Pad4) -> Net-(D217-Pad4)
- R240 pad 2: Net-(D213-Pad5) -> Net-(D217-Pad5)
- U213 pad 6: Net-(D212-Pad1) -> Net-(D216-Pad2)
- U213 pad 7: Net-(D212-Pad2) -> Net-(D216-Pad1)
- U214 pad 1: Net-(D213-Pad1) -> Net-(D217-Pad1)
- U214 pad 10: Net-(D214-Pad3) -> Net-(D218-Pad3)
- U214 pad 11: Net-(D214-Pad4) -> Net-(D218-Pad4)
- U214 pad 12: Net-(D214-Pad5) -> Net-(D218-Pad5)
- U214 pad 14: Net-(D213-Pad5) -> Net-(D217-Pad5)
- U214 pad 15: Net-(D213-Pad4) -> Net-(D217-Pad4)
- U214 pad 16: Net-(D213-Pad3) -> Net-(D217-Pad3)
- U214 pad 9: Net-(D214-Pad1) -> Net-(D218-Pad1)
- U216 pad 11: Net-(D215-Pad5) -> Net-(D219-Pad5)
- U216 pad 12: Net-(D215-Pad4) -> Net-(D219-Pad4)
- U216 pad 13: Net-(D215-Pad3) -> Net-(D219-Pad3)
- U216 pad 14: Net-(D215-Pad1) -> Net-(D219-Pad1)
- U217 pad 11: Net-(D216-Pad5) -> Net-(D220-Pad5)
- U217 pad 12: Net-(D216-Pad4) -> Net-(D220-Pad4)
- U217 pad 13: Net-(D216-Pad3) -> Net-(D220-Pad3)
- U217 pad 14: Net-(D216-Pad1) -> Net-(D220-Pad1)

Commit message: Grobplatzierung abgeschlossen, Raspberry und GSM/GNSS Bohrungen Platziert, Befestigungsbohrungen festgelegt, Board Outline festgelegt
Parts:
- removed C302: 47u, Capacitor_SMD:C_1210_3225Metric
- removed C318, C319: 10u, Capacitor_SMD:C_1210_3225Metric
- J320: footprint Connector_IDC:IDC-Header_2x20_P2.54mm_Vertical -> Connector_PinSocket_2.54mm:PinSocket_2x20_P2.54mm_Vertical
- moved C502 317.1 mm to (413.3, 198.4), turned to 90 degrees
- moved C501 314.1 mm to (408.9, 200.4), turned to 90 degrees
- moved R503 306.9 mm to (416.6, 195.8), turned to 180 degrees
- moved C504 303.2 mm to (405.9, 195.3), turned to 90 degrees
- moved C505 301.4 mm to (410.2, 194.8), turned to 90 degrees
- moved U500 300.9 mm to (415.4, 191.4), turned to 90 degrees
- moved R502 299.7 mm to (405.1, 190.0), turned to 180 degrees
- moved C503 298.9 mm to (401.6, 190.2), turned to 90 degrees
- moved R242 296.3 mm to (165.9, 261.9), turned to 90 degrees
- moved C500 294.5 mm to (403.1, 195.1), turned to 90 degrees
- moved U501 293.0 mm to (409.2, 191.3), turned to 90 degrees
- moved U402 287.8 mm to (409.1, 244.0)
- moved C400 287.8 mm to (413.8, 246.9)
- moved C403 287.8 mm to (404.9, 244.1)
- moved FB400 287.8 mm to (413.8, 243.2)
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Connections:
- D306 pad 1: CTRL_L -> CTRL_H
- D306 pad 2: CTRL_H -> CTRL_L
Routing:
- net GND: vias 0 -> 14
Other:
- board outline added: 255 x 150 mm
- net class Octo: via_dia 0.8 -> 1; via_drill 0.4 -> 0.5
- net class Power added: clearance 0.2, trace_width 1, via_dia 1, via_drill 0.5
