File: Hardware/Displayunit/MCU.sch (KiCad schematic (older format))
At the start: 66 parts, among them J1 Conn_02x25_Odd_Even, U3 MOD-nRF8001

Commit message: Display Unit Lib Fehler behoben, und noch Zeug raus geworfen Library jetzt projekt spezifisch im Hardware root.. Hauptplatine rund um den Prozessor a bissl was getan, vorbereitung Quadspi Flash und SD Karte.
Parts:
- removed C? (x3): 1uF, Capacitor_SMD:C_0603_1608Metric, symbol Device:C
- removed FB? (x5): Ferrite, Inductor_SMD:L_0603_1608Metric, symbol Device:Ferrite_Bead_Small
- removed J1: Conn_02x25_Odd_Even, Connector_PinHeader_2.54mm:PinHeader_2x25_P2.54mm_Vertical, symbol Connector_Generic:Conn_02x25_Odd_Even
- IC?: symbol Womo-rescue:IS66WVH8M8BLL-100B1LI_0-SamacSys_Parts -> Womo-Lin:IS66WVH8M8BLL-100B1LI_0
- IC?: symbol Womo-rescue:MX25LM51245GXDI00-SamacSys_Parts -> Womo-Lin:MX25LM51245GXDI00
- IC?: symbol Womo-rescue:TSC2007-opendous -> opendous:TSC2007
- J?: symbol Womo-rescue:54104-4031-SamacSys_Parts -> Womo-Lin:54104-4031
- J?: symbol Womo-rescue:52271-0679-SamacSys_Parts -> Womo-Lin:52271-0679
Connections:
- net labels added: GND
- net labels removed: *PWR_Reset
- wire segments 524 -> 448
Other:
- note removed: "Connection to Mainboard"
