File: Hardware/Displayunit/Displayunit.sch (KiCad schematic (older format))
At the start: 0 parts

Commit message: Displayunit: Fix Libs, fix, Footprints, PCB angelegt, Auf eine Schaltplanseite reduziert.
Parts:
- added BT1: Battery_Cell, Battery:BatteryHolder_Keystone_1058_1x2032, symbol Device:Battery_Cell
- added C1, C22, C26, C31, C5: 1uF, Capacitor_SMD:C_0603_1608Metric, symbol Device:C
- added C10, C11, C12, C13, C14, C18, C19, C20, C25, C27, C36, C6, C7, C8, C9: 100n, Capacitor_SMD:C_0603_1608Metric, symbol Device:C
- added C15, C17: 10uF, Capacitor_SMD:C_1210_3225Metric, symbol Device:C
- added C16: 10nF, Capacitor_SMD:C_0603_1608Metric, symbol Device:C
- added C2, C28, C30, C34, C40, C41, C45, C48, C50: 100nF, Capacitor_SMD:C_0603_1608Metric, symbol Device:C
- added C21, C32, C33: 2u2, Capacitor_SMD:C_1210_3225Metric, symbol Device:C
- added C23, C24: 3p3, Capacitor_SMD:C_0603_1608Metric, symbol Device:C
- added C29, C43: 10n, Capacitor_SMD:C_0603_1608Metric, symbol Device:C
- added C3, C4: 6p8, Capacitor_SMD:C_0603_1608Metric, symbol Device:C
- added C35, C47: 4u7, Capacitor_SMD:C_1210_3225Metric, symbol Device:C
- added C37: 1u, Capacitor_SMD:C_0603_1608Metric, symbol Device:C
- added C38, C39: 5n6, Capacitor_SMD:C_0603_1608Metric, symbol Device:C
- added C42, C44: 22uF, Capacitor_SMD:C_1210_3225Metric, symbol Device:C
- added C46, C49: 47u, Capacitor_SMD:C_1210_3225Metric, symbol Device:C
- added D1: LED, LED_SMD:LED_1206_3216Metric, symbol Device:LED
- added D2, D3, D4: B345BE-13, Diode_SMD:D_SMB, symbol pspice:DIODE
- added F1: KFZ 5A, Fuse:Fuseholder_Blade_ATO_Littelfuse_Pudenz_2_Pin, symbol Device:Fuse
- added FB1, FB2: 100R, Inductor_SMD:L_0603_1608Metric, symbol Device:Ferrite_Bead_Small
- added IC1: TSC2007, Package_SO:TSSOP-16_4.4x5mm_P0.65mm, symbol opendous:TSC2007
- added IC2: MX25LM51245GXDI00, Womo-Lin:BGA24C100P5X5_600X800X35, symbol Womo-Lin:MX25LM51245GXDI00
- added IC3: IS66WVH8M8BLL-100B1LI_0, Womo-Lin:BGA24C100P5X5_600X800X35, symbol Womo-Lin:IS66WVH8M8BLL-100B1LI_0
- added J1: USB_B_Micro, Connector_USB:USB_Micro-B_Molex-105017-0001, symbol Connector:USB_B_Micro
- added J2: 8P8C_Shielded, Connector_RJ:RJ45_Hanrun_HR911105A, symbol Connector:8P8C_Shielded
- added J3: 54104-4031, Womo-Lin:54104-4031, symbol Womo-Lin:54104-4031
- added J4: Conn_ARM_JTAG_SWD_20, Connector_IDC:IDC-Header_2x10_P2.54mm_Vertical, symbol Connector:Conn_ARM_JTAG_SWD_20
- added J5: 52271-0679, Womo-Lin:52271-0679, symbol Womo-Lin:52271-0679
- added J6: Conn_02x06_Odd_Even, Connector_PinHeader_2.54mm:PinHeader_2x06_P2.54mm_Vertical, symbol Connector_Generic:Conn_02x06_Odd_Even
- added L1: 4uH7, Inductor_SMD:L_Coilcraft_XxL4030, symbol Device:L
- added L2: L_Core_Ferrite, Inductor_SMD:L_Coilcraft_XxL4020, symbol Device:L_Core_Ferrite
- added L3, L4: 15uH, Inductor_SMD:L_Coilcraft_XxL4040, symbol Device:L
- added Q1: 2N7002, Package_TO_SOT_SMD:SOT-23, symbol Transistor_FET:2N7002
- added R1, R2, R3, R4: 10K, Resistor_SMD:R_0603_1608Metric, symbol Device:R
- added R10: 10R 1%, Resistor_SMD:R_0603_1608Metric, symbol Device:R
- added R11, R12, R9: 40k2, Resistor_SMD:R_0603_1608Metric, symbol Device:R
- added R13, R15, R17: 32k4, Resistor_SMD:R_0603_1608Metric, symbol Device:R
- added R14, R16: 86k6, Resistor_SMD:R_0603_1608Metric, symbol Device:R
- added R5: 10k, Resistor_SMD:R_0603_1608Metric, symbol Device:R
- added R6: 100K, Resistor_SMD:R_0603_1608Metric, symbol Device:R
- added R7: 3M3, Resistor_SMD:R_0603_1608Metric, symbol Device:R
- added R8: 432k, Resistor_SMD:R_0603_1608Metric, symbol Device:R
- added SW1: Boot, Button_Switch_THT:SW_PUSH_6mm, symbol Switch:SW_Push
- added SW2: Reset, Button_Switch_THT:SW_PUSH_6mm, symbol Switch:SW_Push
- added SW3: Wakeup, Button_Switch_THT:SW_PUSH_6mm_H8.5mm, symbol Switch:SW_Push
- added U1: STM32L4R9ZITx, Package_QFP:LQFP-144_20x20mm_P0.5mm, symbol MCU_ST_STM32L4+:STM32L4R9ZITx
- added U2: USBLC6-2SC6, Package_TO_SOT_SMD:SOT-23-6, symbol Power_Protection:USBLC6-2SC6
- added U3: STLD40D, Package_DFN_QFN:DFN-8-1EP_3x3mm_P0.65mm_EP1.55x2.4mm, symbol Womo-Lin:STLD40D
- added U4, U5: MAX17572, Package_DFN_QFN:DFN-12-1EP_3x3mm_P0.5mm_EP2.05x2.86mm, symbol Regulator_Switching:MAX17572
- added Y1: 16 MHz, Crystal:Crystal_SMD_3225-4Pin_3.2x2.5mm, symbol Device:Crystal_GND24
- added Y2: 32.768, Crystal:Crystal_SMD_MicroCrystal_CC7V-T1A-2Pin_3.2x1.5mm, symbol Device:Crystal
Connections:
- net labels added: *I2C2_SCL, *I2C2_SDA, *I2C4_SCL, *I2C4_SDA, *LCD_BL_CTR, *LCD_LED-A, *LCD_LED-K, +3.3V, +3.3VA, +BATT, +VSW, 3VA_EN, Boot0, GND, GND1, I2C3_SCL, I2C3_SDA, JTAG_RES, JTAG_TCK, JTAG_TDI, JTAG_TDO, JTAG_TMS, LCD_37, LCD_38, LCD_39, LCD_40, LCD_B0, LCD_B1, LCD_B2, LCD_B3, LCD_B4, LCD_B5, LCD_B6, LCD_B7, LCD_BL_CTRL, LCD_CLK, LCD_DE, LCD_EN, LCD_G0, LCD_G1, LCD_G2, LCD_G3, LCD_G4, LCD_G5, LCD_G6, LCD_G7, LCD_HSYNC, LCD_INT, LCD_LED-A, LCD_LED-K, LCD_R0, LCD_R1, LCD_R2, LCD_R3, LCD_R4, LCD_R5, LCD_R6, LCD_R7, LCD_VSYNC, OctoSPI_P1_CLK, OctoSPI_P1_DQS, OctoSPI_P1_IO0, OctoSPI_P1_IO1, OctoSPI_P1_IO2, OctoSPI_P1_IO3, OctoSPI_P1_IO4, OctoSPI_P1_IO5, OctoSPI_P1_IO6, OctoSPI_P1_IO7, OctoSPI_P1_NCS, OctoSPI_P2_CLK, OctoSPI_P2_DQS, OctoSPI_P2_IO0, OctoSPI_P2_IO1, OctoSPI_P2_IO2, OctoSPI_P2_IO3, OctoSPI_P2_IO4, OctoSPI_P2_IO5, OctoSPI_P2_IO6, OctoSPI_P2_IO7, OctoSPI_P2_NCS, PWR_Reset, RESET, SPI1_MISO, SPI1_MOSI, SPI1_NSS, SPI1_SCK, Signal_LED, TOUCH_INT, TOUCH_RESET, USB_D+, USB_D-, USB_ID, USB_NOE, USB_SOF, VCC, VCCQ, Wakeup, X+, X-, Y+, Y-
- wire segments 0 -> 508
- no-connect marks 0 -> 22
Other:
- note added: "I2C ADR: 1001000"
- note added: "Touchconfig"
- note added: "Touchcontroller"
- note added: "Touchdisplay RGB TFT"

Commit message: Fix Womo BRD für Produktion, Displayboard Schaltplan weitere Arbeiten.
Parts:
- added C?: 100n, Capacitor_SMD:C_0603_1608Metric, symbol Device:C
- added C?: 5n6, Capacitor_SMD:C_0603_1608Metric, symbol Device:C
- added D?: NUP2105L, symbol Device:D_TVS_x2_AAC
- added FB? (x2): 100R, Inductor_SMD:L_0603_1608Metric, symbol Device:Ferrite_Bead_Small
- added R? (x2): 60R, Resistor_SMD:R_0603_1608Metric, symbol Device:R
- added U?: TJA1049T-3, Package_SO:SOIC-8_3.9x4.9mm_P1.27mm, symbol Interface_CAN_LIN:TJA1049T-3
Connections:
- net labels removed: VCCQ
- wire segments 508 -> 529
Other:
- moved on the sheet: J3

Commit message: Fix: Produktionsdaten Board Arbeiten Schaltplan Displayunit
Parts:
- removed U?: TJA1049T-3, Package_SO:SOIC-8_3.9x4.9mm_P1.27mm, symbol Interface_CAN_LIN:TJA1049T-3
- added C53, C54: 100n, Capacitor_SMD:C_0603_1608Metric, symbol Displayunit-rescue:C-Device
- added J7: 734-264, SHDR4W120P0X381_1X4_1640X1030X850P, symbol WAGO:734-264
- added U6: SN65HVD231, Package_SO:SOIC-8_3.9x4.9mm_P1.27mm, symbol Interface_CAN_LIN:SN65HVD231
- BT1: symbol Device:Battery_Cell -> Displayunit-rescue:Battery_Cell-Device
- C1, C10, C11, C12, C13, C14, C15, C16, C17, C18, C19, C2, C20, C21, C22, C23, C24, C25, C26, C27, C28, C29, C3, C30, C31, C32, C33, C34, C35, C36, C37, C38, C39, C4, C40, C41, C42, C43, C44, C45, C46, C47, C48, C49, C5, C50, C6, C7, C8, C9: symbol Device:C -> Displayunit-rescue:C-Device
- C51, C52: renamed from C?; symbol Device:C -> Displayunit-rescue:C-Device
- D1: symbol Device:LED -> Displayunit-rescue:LED-Device
- D2, D3, D4: symbol pspice:DIODE -> Displayunit-rescue:DIODE-pspice
- D5: renamed from D?; symbol Device:D_TVS_x2_AAC -> Displayunit-rescue:D_TVS_x2_AAC-Device
- F1: symbol Device:Fuse -> Displayunit-rescue:Fuse-Device
- FB1, FB2: symbol Device:Ferrite_Bead_Small -> Displayunit-rescue:Ferrite_Bead_Small-Device
- FB3, FB4: renamed from FB?; symbol Device:Ferrite_Bead_Small -> Displayunit-rescue:Ferrite_Bead_Small-Device
- J1: symbol Connector:USB_B_Micro -> Displayunit-rescue:USB_B_Micro-Connector
- J2: symbol Connector:8P8C_Shielded -> Displayunit-rescue:8P8C_Shielded-Connector
- J4: symbol Connector:Conn_ARM_JTAG_SWD_20 -> Displayunit-rescue:Conn_ARM_JTAG_SWD_20-Connector
- J6: symbol Connector_Generic:Conn_02x06_Odd_Even -> Displayunit-rescue:Conn_02x06_Odd_Even-Connector_Generic
- L1, L3, L4: symbol Device:L -> Displayunit-rescue:L-Device
- L2: symbol Device:L_Core_Ferrite -> Displayunit-rescue:L_Core_Ferrite-Device
- Q1: symbol Transistor_FET:2N7002 -> Displayunit-rescue:2N7002-Transistor_FET
- R1, R10, R11, R12, R13, R14, R15, R16, R17, R2, R3, R4, R5, R6, R7, R8, R9: symbol Device:R -> Displayunit-rescue:R-Device
- R18, R19: renamed from R?; symbol Device:R -> Displayunit-rescue:R-Device
- SW1, SW2, SW3: symbol Switch:SW_Push -> Displayunit-rescue:SW_Push-Switch
- U1: symbol MCU_ST_STM32L4+:STM32L4R9ZITx -> Displayunit-rescue:STM32L4R9ZITx-MCU_ST_STM32L4+
- U2: symbol Power_Protection:USBLC6-2SC6 -> Displayunit-rescue:USBLC6-2SC6-Power_Protection
- U4, U5: symbol Regulator_Switching:MAX17572 -> Displayunit-rescue:MAX17572-Regulator_Switching
- Y1: symbol Device:Crystal_GND24 -> Displayunit-rescue:Crystal_GND24-Device
- Y2: symbol Device:Crystal -> Displayunit-rescue:Crystal-Device
Connections:
- net labels added: CAN_STB, Control+, USART1_RX, USART1_TX, VrefCAN
- wire segments 529 -> 554

Commit message: Display Board kleinere Schaltplan Anpassung , Board Design an New Heaven Display angepasst, Platzierung zu 95 % abgeschlossen
Parts:
- removed D2, D3, D4: B345BE-13, Diode_SMD:D_SMB, symbol Displayunit-rescue:DIODE-pspice
- added D2, D3, D4: B250, Diode_SMD:D_SMB, symbol Diode:B250
- added R20: 100k, Resistor_SMD:R_0603_1608Metric, symbol Displayunit-rescue:R-Device
- C1, C22, C26, C31, C37: footprint Capacitor_SMD:C_0603_1608Metric -> Capacitor_SMD:C_1210_3225Metric
- D5: footprint (none) -> Package_TO_SOT_SMD:SOT-23
- F1: value KFZ 5A -> PFUF.150.2 30V 1.5A; footprint Fuse:Fuseholder_Blade_ATO_Littelfuse_Pudenz_2_Pin -> Fuse:Fuse_1210_3225Metric
- J2: footprint Connector_RJ:RJ45_Hanrun_HR911105A -> Connector_RJ:RJ45_Amphenol_RJHSE5380
- J7: footprint SHDR4W120P0X381_1X4_1640X1030X850P -> WAGO:SHDR4W120P0X381_1X4_1640X1030X850P
Connections:
- net +VSW is gone; now on net +3.3VA: R13.1
- net GND1 is gone; now on net GND: C17.2, C18.1, C19.1, C20.1, C21.1
- net VCC is gone; now on net +3.3VA: C25.2, C31.1, IC1.1 (VDD), J5.1, R3.1, R4.1
- net +3.3VA: now also C44.1, L4.2, R16.1
- net +BATT: now also R9.1
- net 3VA_EN: now also R20.1
- net Control+: now also C54.1, D3.2 (A)
- net GND: now also J5.2, R20.2
- net LCD_LED-A: now also D4.1 (K)
- net at Q1.3 (D), U5.2 (EN/UVLO): now also R9.2
- net at L1.2, U3.8 (SW): now also D4.2 (A)
- net at F1.2: now also D2.1 (K), D3.1 (K)
- net at C53.1, J7.1, J7.2: now also D2.2 (A)
Other:
- moved on the sheet: R9
