File: Hardware/Displayunit/Displayunit.sch (KiCad schematic (older format))
At the start: 122 parts, among them IC1 TSC2007, IC2 MX25LM51245GXDI00, IC3 IS66WVH8M8BLL-100B1LI_0, J1 8P8C_Shielded, J2 8P8C_Shielded, J3 54104-4031, J4 Conn_ARM_JTAG_SWD_20, J5 52271-0679, J6 Conn_02x06_Odd_Even, J7 WAGO_Klemmleiste_2-pol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

Commit message: Weitere Arbeiten am Layout, UID i2c Eeprom hinzugefügt.
Parts:
- added C59: 100n, Capacitor_SMD:C_0603_1608Metric, symbol Displayunit-rescue:C-Device
- added U8: 24AA02-OT, Package_TO_SOT_SMD:SOT-23-5, symbol Memory_EEPROM:24AA02-OT
- gave numbers to parts that had none: 2
Connections:
- wire segments 607 -> 613
Changed lines of the file:
@@
 AR Path="/5D80EC74/5E2BD8A4" Ref="C?"  Part="1"
 AR Path="/5D80E6E8/5E2BD8A4" Ref="C?"  Part="1"
-AR Path="/5E2BD8A4" Ref="C?"  Part="1"
-F 0 "C?" V 20098 4350 50  0000 C CNN
+AR Path="/5E2BD8A4" Ref="C58"  Part="1"
+F 0 "C58" V 20098 4350 50  0000 C CNN
 F 1 "4u7" V 20189 4350 50  0000 C CNN
 F 2 "Capacitor_SMD:C_0603_1608Metric" H 20388 4200 50  0001 C CNN
@@
 AR Path="/5D80EC74/5E337A65" Ref="C?"  Part="1"
 AR Path="/5D80E6E8/5E337A65" Ref="C?"  Part="1"
-AR Path="/5E337A65" Ref="C?"  Part="1"
-F 0 "C?" V 20450 2350 50  0000 C CNN
+AR Path="/5E337A65" Ref="C57"  Part="1"
+F 0 "C57" V 20450 2350 50  0000 C CNN
 F 1 "4u7" V 20550 2350 50  0000 C CNN
 F 2 "Capacitor_SMD:C_0603_1608Metric" H 20338 2200 50  0001 C CNN
@@
 Wire Wire Line
 	20500 4350 20800 4350
+$Comp
+L Memory_EEPROM:24AA02-OT U8
+U 1 1 5E4A9EFD
+P 11900 11900
+F 0 "U8" H 11571 11946 50  0000 R CNN
+F 1 "24AA02-OT" H 11571 11855 50  0000 R CNN
+F 2 "Package_TO_SOT_SMD:SOT-23-5" H 11900 11900 50  0001 C CNN
+F 3 "http://ww1.microchip.com/downloads/en/DeviceDoc/21709J.pdf" H 11900 11900 50  0001 C CNN
+	1    11900 11900
+	1    0    0    -1
+$EndComp
+Text GLabel 12450 11900 2    50   Input ~ 0
+I2C4_SCL
+Text GLabel 12450 11800 2    50   BiDi ~ 0
+I2C4_SDA
+$Comp
+L Displayunit-rescue:GND-power #PWR?
+U 1 1 5E5A04AA
+P 11900 12250
+AR Path="/5C8BBC9A/5E5A04AA" Ref="#PWR?"  Part="1"
+AR Path="/5E0C5EEA/5E5A04AA" Ref="#PWR?"  Part="1"
+AR Path="/5D80EC74/5E5A04AA" Ref="#PWR?"  Part="1"
+AR Path="/5D80E6E8/5E5A04AA" Ref="#PWR?"  Part="1"
+AR Path="/5D80E2A0/5E5A04AA" Ref="#PWR?"  Part="1"
+AR Path="/5E5A04AA" Ref="#PWR0127"  Part="1"
+F 0 "#PWR0127" H 11900 12000 50  0001 C CNN
+F 1 "GND" H 11900 12050 50  0000 C CNN
+F 2 "" H 11900 12250 50  0001 C CNN
+F 3 "" H 11900 12250 50  0001 C CNN
+	1    11900 12250
+	1    0    0    -1
+$EndComp
+$Comp
+L Displayunit-rescue:C-Device C?
+U 1 1 5E61BCF5
+P 12100 11400
+AR Path="/5C8BBC9A/5E61BCF5" Ref="C?"  Part="1"
+AR Path="/5E0C5EEA/5E61BCF5" Ref="C?"  Part="1"
+AR Path="/5D80EC74/5E61BCF5" Ref="C?"  Part="1"
+AR Path="/5D80E6E8/5E61BCF5" Ref="C?"  Part="1"
+AR Path="/5E61BCF5" Ref="C59"  Part="1"
+F 0 "C59" H 12300 11450 50  0000 L CNN
+F 1 "100n" H 12300 11350 50  0000 L CNN
+F 2 "Capacitor_SMD:C_0603_1608Metric" H 12138 11250 50  0001 C CNN
+F 3 "~" H 12100 11400 50  0001 C CNN
+	1    12100 11400
+	1    0    0    -1
+$EndComp
+$Comp
+L Displayunit-rescue:+3.3V-power #PWR?
+U 1 1 5E61BCFB
+P 11900 11200
+AR Path="/5D80E2A0/5E61BCFB" Ref="#PWR?"  Part="1"
+AR Path="/5E61BCFB" Ref="#PWR0128"  Part="1"
+F 0 "#PWR0128" H 11900 11050 50  0001 C CNN
+F 1 "+3.3V" H 11915 11373 50  0000 C CNN
+F 2 "" H 11900 11200 50  0001 C CNN
+F 3 "" H 11900 11200 50  0001 C CNN
+	1    11900 11200
+	1    0    0    -1
+$EndComp
+Wire Wire Line
+	11900 11600 11900 11250
+Wire Wire Line
+	12100 11250 11900 11250
+Connection ~ 11900 11250
+Wire Wire Line
+	11900 11250 11900 11200
+$Comp
+L Displayunit-rescue:GND-power #PWR?
+U 1 1 5E80DCAB
+P 12100 11550
+AR Path="/5C8BBC9A/5E80DCAB" Ref="#PWR?"  Part="1"
+AR Path="/5E0C5EEA/5E80DCAB" Ref="#PWR?"  Part="1"
+AR Path="/5D80EC74/5E80DCAB" Ref="#PWR?"  Part="1"
+AR Path="/5D80E6E8/5E80DCAB" Ref="#PWR?"  Part="1"
+AR Path="/5D80E2A0/5E80DCAB" Ref="#PWR?"  Part="1"
+AR Path="/5E80DCAB" Ref="#PWR0129"  Part="1"
+F 0 "#PWR0129" H 12100 11300 50  0001 C CNN
+F 1 "GND" H 12250 11500 50  0000 C CNN
+F 2 "" H 12100 11550 50  0001 C CNN
+F 3 "" H 12100 11550 50  0001 C CNN
+	1    12100 11550
+	1    0    0    -1
+$EndComp
+Wire Wire Line
+	11900 12250 11900 12200
+Wire Wire Line
+	12450 11800 12300 11800
+Wire Wire Line
+	12450 11900 12300 11900
 $EndSCHEMATC

Commit message: Displayboard fertig layoutet, kleinere Fehler beseitigt, WomoLin Biblothek senkrechter Würth RJ 45 zugefügt
Parts:
- removed J1, J2: 8P8C_Shielded, Connector_RJ:RJ45_Amphenol_RJHSE5380, symbol Displayunit-rescue:8P8C_Shielded-Connector
- added J1, J2: 615008138221, Womo-Lin:615008138221, symbol Womo-Lin:615008138221
Connections:
- net labels removed: LCD_BL_CTR, Wakeup
- wire segments 613 -> 622
Changed lines of the file:
@@
 	1    0    0    -1
 $EndComp
-Text GLabel 11350 5750 0    50   Input ~ 0
-USB_D-
 Text GLabel 12350 5750 2    50   Input ~ 0
+USB_D-
+Text GLabel 11350 5750 0    50   Input ~ 0
 USB_D+
 Text GLabel 10800 5200 2    50   Input ~ 0
@@
 Touchdisplay RGB TFT
 $Comp
-L Displayunit-rescue:USBLC6-2SC6-Power_Protection U?
-U 1 1 5E312514
-P 11850 5650
-AR Path="/5D80E2A0/5E312514" Ref="U?"  Part="1"
-AR Path="/5E312514" Ref="U2"  Part="1"
-F 0 "U2" H 12150 5250 50  0000 C CNN
-F 1 "USBLC6-2SC6" H 12350 5150 50  0000 C CNN
-F 2 "Package_TO_SOT_SMD:SOT-23-6" H 11100 6050 50  0001 C CNN
-F 3 "http://www2.st.com/resource/en/datasheet/CD00050750.pdf" H 12050 6000 50  0001 C CNN
-	1    11850 5650
-	1    0    0    -1
-$EndComp
-$Comp
 L Womo-Lin:54104-4031 J?
 U 1 1 5E31251F
@@
 	11850 4800 11850 5150
 Wire Wire Line
-	11350 5100 11350 5550
-Wire Wire Line
-	10700 5100 11350 5100
-Wire Wire Line
-	10700 5000 12350 5000
-Wire Wire Line
-	12350 5000 12350 5550
+	10700 5000 11350 5000
 Wire Wire Line
 	10700 4800 11850 4800
@@
 	7400 8300 7250 8300
 Text GLabel 7400 8300 2    50   Input ~ 0
-Wakeup
+3VA_EN
 Connection ~ 2950 6100
 Wire Wire Line
@@
 	6350 12900 6350 13000
 Text GLabel 7400 6600 2    50   Output ~ 0
-LCD_BL_CTR
+LCD_BL_CTRL
 Text GLabel 7400 10200 2    50   Input ~ 0
 TOUCH_INT
@@
 Y-
 $Comp
-L Displayunit-rescue:8P8C_Shielded-Connector J1
-U 1 1 5F96FCE3
-P 15900 8450
-F 0 "J1" H 15957 9117 50  0000 C CNN
-F 1 "8P8C_Shielded" H 15957 9026 50  0000 C CNN
-F 2 "Connector_RJ:RJ45_Amphenol_RJHSE5380" V 15900 8475 50  0001 C CNN
-F 3 "~" V 15900 8475 50  0001 C CNN
-	1    15900 8450
-	-1   0    0    1
-$EndComp
-$Comp
 L Displayunit-rescue:R-Device R?
 U 1 1 5E2C30E1
@@
 $EndComp
 $Comp
-L Displayunit-rescue:GND-power #PWR?
-U 1 1 5EA2EB1F
-P 15900 7950
-AR Path="/5C8BBC9A/5EA2EB1F" Ref="#PWR?"  Part="1"
-AR Path="/5E0C5EEA/5EA2EB1F" Ref="#PWR?"  Part="1"
-AR Path="/5D80EC74/5EA2EB1F" Ref="#PWR?"  Part="1"
-AR Path="/5D80E6E8/5EA2EB1F" Ref="#PWR?"  Part="1"
-AR Path="/5D80E2A0/5EA2EB1F" Ref="#PWR?"  Part="1"
-AR Path="/5EA2EB1F" Ref="#PWR0104"  Part="1"
-F 0 "#PWR0104" H 15900 7700 50  0001 C CNN
-F 1 "GND" H 15900 7750 50  0000 C CNN
-F 2 "" H 15900 7950 50  0001 C CNN
-F 3 "" H 15900 7950 50  0001 C CNN
-	1    15900 7950
-	-1   0    0    1
-$EndComp
-$Comp
 L Displayunit-rescue:Ferrite_Bead_Small-Device FB?
 U 1 1 5EA91CC4
@@
 L Displayunit-rescue:GND-power #PWR?
 U 1 1 5ECB14B9
-P 15350 9000
+P 16500 8700
 AR Path="/5C8BBC9A/5ECB14B9" Ref="#PWR?"  Part="1"
 AR Path="/5E0C5EEA/5ECB14B9" Ref="#PWR?"  Part="1"
@@
 AR Path="/5D80E2A0/5ECB14B9" Ref="#PWR?"  Part="1"
 AR Path="/5ECB14B9" Ref="#PWR0114"  Part="1"
-F 0 "#PWR0114" H 15350 8750 50  0001 C CNN
-F 1 "GND" H 15350 8800 50  0000 C CNN
-F 2 "" H 15350 9000 50  0001 C CNN
-F 3 "" H 15350 9000 50  0001 C CNN
-	1    15350 9000
+F 0 "#PWR0114" H 16500 8450 50  0001 C CNN
+F 1 "GND" H 16500 8500 50  0000 C CNN
+F 2 "" H 16500 8700 50  0001 C CNN
+F 3 "" H 16500 8700 50  0001 C CNN
+	1    16500 8700
 	1    0    0    -1
 $EndComp
@@
 Wire Wire Line
 	17500 4150 17400 4150
-$Comp
-L Displayunit-rescue:8P8C_Shielded-Connector J2
-U 1 1 5DED998B
-P 15900 9850
-F 0 "J2" H 15957 10517 50  0000 C CNN
-F 1 "8P8C_Shielded" H 15957 10426 50  0000 C CNN
-F 2 "Connector_RJ:RJ45_Amphenol_RJHSE5380" V 15900 9875 50  0001 C CNN
-F 3 "~" V 15900 9875 50  0001 C CNN
-	1    15900 9850
-	-1   0    0    1
-$EndComp
-$Comp
-L Displayunit-rescue:GND-power #PWR?
-U 1 1 5DEDCC16
-P 15250 10400
-AR Path="/5C8BBC9A/5DEDCC16" Ref="#PWR?"  Part="1"
-AR Path="/5E0C5EEA/5DEDCC16" Ref="#PWR?"  Part="1"
-AR Path="/5D80EC74/5DEDCC16" Ref="#PWR?"  Part="1"
-AR Path="/5D80E6E8/5DEDCC16" Ref="#PWR?"  Part="1"
-AR Path="/5D80E2A0/5DEDCC16" Ref="#PWR?"  Part="1"
-AR Path="/5DEDCC16" Ref="#PWR0122"  Part="1"
-F 0 "#PWR0122" H 15250 10150 50  0001 C CNN
-F 1 "GND" H 15250 10200 50  0000 C CNN
-F 2 "" H 15250 10400 50  0001 C CNN
-F 3 "" H 15250 10400 50  0001 C CNN
-	1    15250 10400
-	1    0    0    -1
-$EndComp
-Wire Wire Line
-	15500 10150 15250 10150
-Wire Wire Line
-	15250 10150 15250 10250
-Wire Wire Line
-	15500 10250 15250 10250
-Connection ~ 15250 10250
-Wire Wire Line
-	15250 10250 15250 10400
 Wire Wire Line
 	15500 9950 15050 9950
@@
 	15150 8450 15500 8450
 Wire Wire Line
-	15350 8750 15350 8850
-Wire Wire Line
-	15500 8750 15350 8750
-Wire Wire Line
-	15500 8850 15350 8850
-Connection ~ 15350 8850
-Wire Wire Line
-	15350 8850 15350 9000
-Wire Wire Line
 	15500 9650 15250 9650
 Wire Wire Line
@@
 	15250 9550 15250 8250
 NoConn ~ 15500 8350
-NoConn ~ 15500 8650
+NoConn ~ 16400 8150
 NoConn ~ 15500 9750
-NoConn ~ 15500 10050
+NoConn ~ 16400 9550
 $Comp
 L Displayunit-rescue:GND-power #PWR?
 U 1 1 5E47C766
-P 15900 9350
+P 16500 10100
 AR Path="/5C8BBC9A/5E47C766" Ref="#PWR?"  Part="1"
 AR Path="/5E0C5EEA/5E47C766" Ref="#PWR?"  Part="1"
@@
 AR Path="/5D80E2A0/5E47C766" Ref="#PWR?"  Part="1"
 AR Path="/5E47C766" Ref="#PWR0123"  Part="1"
-F 0 "#PWR0123" H 15900 9100 50  0001 C CNN
-F 1 "GND" H 15700 9350 50  0000 C CNN
-F 2 "" H 15900 9350 50  0001 C CNN
-F 3 "" H 15900 9350 50  0001 C CNN
-	1    15900 9350
-	-1   0    0    1
+F 0 "#PWR0123" H 16500 9850 50  0001 C CNN
+F 1 "GND" H 16500 9900 50  0000 C CNN
+F 2 "" H 16500 10100 50  0001 C CNN
+F 3 "" H 16500 10100 50  0001 C CNN
+	1    16500 10100
+	1    0    0    -1
 $EndComp
 $Comp
@@
 Wire Wire Line
 	12450 11900 12300 11900
+$Comp
+L Womo-Lin:615008138221 J1
+U 1 1 5E552771
+P 15500 8150
+F 0 "J1" H 15950 8415 50  0000 C CNN
+F 1 "615008138221" H 15950 8324 50  0000 C CNN
+F 2 "Womo-Lin:615008138221" H 16250 8250 50  0001 L CNN
+F 3 "https://componentsearchengine.com/Datasheets/1/615008138221.pdf" H 16250 8150 50  0001 L CNN
+F 4 "Modular Connectors / Ethernet Connectors WR-MJ Feml Shielded 8P8C Vert Front Post" H 16250 8050 50  0001 L CNN "Description"
+F 5 "16.85" H 16250 7950 50  0001 L CNN "Height"
+F 6 "710-615008138221" H 16250 7850 50  0001 L CNN "Mouser Part Number"
+F 7 "https://www.mouser.com/Search/Refine.aspx?Keyword=710-615008138221" H 16250 7750 50  0001 L CNN "Mouser Price/Stock"
+F 8 "Wurth Elektronik" H 16250 7650 50  0001 L CNN "Manufacturer_Name"
+F 9 "615008138221" H 16250 7550 50  0001 L CNN "Manufacturer_Part_Number"
+	1    15500 8150
+	1    0    0    -1
+$EndComp
+$Comp
+L Womo-Lin:615008138221 J2
+U 1 1 5E555A7A
+P 15500 9550
+F 0 "J2" H 15950 9815 50  0000 C CNN
+F 1 "615008138221" H 15950 9724 50  0000 C CNN
+F 2 "Womo-Lin:615008138221" H 16250 9650 50  0001 L CNN
+F 3 "https://componentsearchengine.com/Datasheets/1/615008138221.pdf" H 16250 9550 50  0001 L CNN
+F 4 "Modular Connectors / Ethernet Connectors WR-MJ Feml Shielded 8P8C Vert Front Post" H 16250 9450 50  0001 L CNN "Description"
+F 5 "16.85" H 16250 9350 50  0001 L CNN "Height"
+F 6 "710-615008138221" H 16250 9250 50  0001 L CNN "Mouser Part Number"
+F 7 "https://www.mouser.com/Search/Refine.aspx?Keyword=710-615008138221" H 16250 9150 50  0001 L CNN "Mouser Price/Stock"
+F 8 "Wurth Elektronik" H 16250 9050 50  0001 L CNN "Manufacturer_Name"
+F 9 "615008138221" H 16250 8950 50  0001 L CNN "Manufacturer_Part_Number"
+	1    15500 9550
+	1    0    0    -1
+$EndComp
+Wire Wire Line
+	16400 9650 16500 9650
+Wire Wire Line
+	16500 9650 16500 9750
+Wire Wire Line
+	16400 9750 16500 9750
+Connection ~ 16500 9750
+Wire Wire Line
+	16500 9750 16500 9850
+Wire Wire Line
+	16400 9850 16500 9850
+Connection ~ 16500 9850
+Wire Wire Line
+	16500 9850 16500 9950
+Wire Wire Line
+	16400 9950 16500 9950
+Connection ~ 16500 9950
+Wire Wire Line
+	16500 9950 16500 10100
+Wire Wire Line
+	16400 8250 16500 8250
+Wire Wire Line
+	16500 8250 16500 8350
+Wire Wire Line
+	16400 8350 16500 8350
+Connection ~ 16500 8350
+Wire Wire Line
+	16500 8350 16500 8450
+Wire Wire Line
+	16400 8450 16500 8450
+Connection ~ 16500 8450
+Wire Wire Line
+	16500 8450 16500 8550
+Wire Wire Line
+	16400 8550 16500 8550
+Connection ~ 16500 8550
+Wire Wire Line
+	16500 8550 16500 8700
+$Comp
+L Displayunit-rescue:USBLC6-2SC6-Power_Protection U?
+U 1 1 5E312514
+P 11850 5650
+AR Path="/5D80E2A0/5E312514" Ref="U?"  Part="1"
+AR Path="/5E312514" Ref="U2"  Part="1"
+F 0 "U2" H 12150 5250 50  0000 C CNN
+F 1 "USBLC6-2SC6" H 12350 5150 50  0000 C CNN
+F 2 "Package_TO_SOT_SMD:SOT-23-6" H 11100 6050 50  0001 C CNN
+F 3 "http://www2.st.com/resource/en/datasheet/CD00050750.pdf" H 12050 6000 50  0001 C CNN
+	1    11850 5650
+	1    0    0    -1
+$EndComp
+Wire Wire Line
+	11350 5000 11350 5550
+Wire Wire Line
+	10700 5100 12350 5100
+Wire Wire Line
+	12350 5100 12350 5550
+Text GLabel 7400 9500 2    50   Output ~ 0
+CAN_STB
+Wire Wire Line
+	7400 9500 7250 9500
 $EndSCHEMATC

Commit message: Commit Foo beseitigt, Änderung auf Displayboard auf Protofertiger Teile.
Parts:
- removed U4, U5: MAX17572, Package_DFN_QFN:DFN-12-1EP_3x3mm_P0.5mm_EP2.05x2.86mm, symbol Displayunit-rescue:MAX17572-Regulator_Switching
- added C60, C61: 2u2, Capacitor_SMD:C_1210_3225Metric, symbol Displayunit-rescue:C-Device
- added C62, C63: 100n, Capacitor_SMD:C_1210_3225Metric, symbol Displayunit-rescue:C-Device
- added C64, C65: 2n7, Capacitor_SMD:C_0603_1608Metric, symbol Displayunit-rescue:C-Device
- added D6, D7: B260A-13-F, Diode_SMD:D_SMB, symbol Diode:B250
- added R2: 10K, Resistor_SMD:R_0603_1608Metric, symbol Displayunit-rescue:R-Device
- added R21, R22: 76K8, Resistor_SMD:R_0603_1608Metric, symbol Displayunit-rescue:R-Device
- added U4, U5: TPS54160DGQR, Womo-Lin:SOP50P490X110-11N, symbol Womo-Lin:TPS54160DGQR
- C38, C39: value 5n6 -> 10n
- C40, C41: value 100nF -> 100n
- C44: value 22uF -> 47u
- C57, C58: value 4u7 -> 6p8
- D2, D3: value B250 -> B260A-13-F
- FB10, FB5, FB6, FB7, FB8, FB9: value 100R -> BLM18PG121SN1D
- L3, L4: value 15uH -> 10uH
- R11, R12: value 40k2 -> 90k9
- R14: value 86k6 -> 31K6
- R15: value 32k4 -> 10K
- R16: value 86k6 -> 31k6
- R17: value 32k4 -> 10k
- R7: value 3M3 -> 332k
- R8: value 432k -> 61k9
- R9: value 40k2 -> 332k
- U6: value SN65HVD231 -> SN65HVD231DR
- U7: value AT25xxx -> AT25SF161-SHD-T
- U8: value 24AA02-OT -> 24AA02E48T-I/OT
- Y1: value 16 MHz -> X322516MLB4SI
- Y2: value 32.768 -> Q13FC1350000400
Connections:
- wire segments 622 -> 646
Other:
- moved on the sheet: C25, C27, C28, C29, C30, C31, C32, C33, C34, C35, C36, C37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

Commit message: Änderung PSU Displayboard, Lib angepast.
Parts:
- BT1: footprint Battery:BatteryHolder_Keystone_1058_1x2032 -> Womo-Lin:QJ.BS-6
- L1: footprint Inductor_SMD:L_Coilcraft_XxL4030 -> Womo-Lin:MWSA0603
- L2: footprint Inductor_SMD:L_Coilcraft_XxL4020 -> Womo-Lin:MWSA0603
- L3, L4: footprint Inductor_SMD:L_Coilcraft_XxL4040 -> Womo-Lin:MWSA0603
- SW1, SW2: footprint Button_Switch_THT:SW_PUSH_6mm -> Womo-Lin:TS-1187A
Changed lines of the file:
@@
 EESchema Schematic File Version 4
 LIBS:Displayunit-cache
-EELAYER 30 0
+EELAYER 29 0
 EELAYER END
 $Descr A2 23386 16535
@@
 F 0 "L4" V 21000 3650 50  0000 C CNN
 F 1 "10uH" V 20900 3600 50  0000 C CNN
-F 2 "Inductor_SMD:L_Coilcraft_XxL4040" H 20800 3750 50  0001 C CNN
+F 2 "Womo-Lin:MWSA0603" H 20800 3750 50  0001 C CNN
 F 3 "~" H 20800 3750 50  0001 C CNN
 	1    20800 3750
@@
 F 0 "L1" V 19840 6200 50  0000 C CNN
 F 1 "4uH7" V 19749 6200 50  0000 C CNN
-F 2 "Inductor_SMD:L_Coilcraft_XxL4030" H 19650 6200 50  0001 C CNN
+F 2 "Womo-Lin:MWSA0603" H 19650 6200 50  0001 C CNN
 F 3 "~" H 19650 6200 50  0001 C CNN
 	1    19650 6200
@@
 F 0 "L2" V 20400 8650 50  0000 C CNN
 F 1 "L_Core_Ferrite" V 20500 8650 50  0000 C CNN
-F 2 "Inductor_SMD:L_Coilcraft_XxL4020" H 20600 8550 50  0001 C CNN
+F 2 "Womo-Lin:MWSA0603" H 20600 8550 50  0001 C CNN
 F 3 "~" H 20600 8550 50  0001 C CNN
 	1    20600 8550
@@
 F 0 "SW1" V 2950 4635 50  0000 C CNN
 F 1 "Boot" V 2850 4600 50  0000 C CNN
-F 2 "Button_Switch_THT:SW_PUSH_6mm" H 2950 4550 50  0001 C CNN
+F 2 "Womo-Lin:TS-1187A" H 2950 4550 50  0001 C CNN
 F 3 "" H 2950 4550 50  0001 C CNN
 	1    2950 4350
@@
 F 0 "BT1" H 3668 5646 50  0000 L CNN
 F 1 "Battery_Cell" H 3668 5555 50  0000 L CNN
-F 2 "Battery:BatteryHolder_Keystone_1058_1x2032" V 3550 5610 50  0001 C CNN
+F 2 "Womo-Lin:QJ.BS-6" V 3550 5610 50  0001 C CNN
 F 3 "~" V 3550 5610 50  0001 C CNN
 	1    3550 5550
@@
 F 0 "SW2" V 2950 6585 50  0000 C CNN
 F 1 "Reset" V 2850 6550 50  0000 C CNN
-F 2 "Button_Switch_THT:SW_PUSH_6mm" H 2950 6500 50  0001 C CNN
+F 2 "Womo-Lin:TS-1187A" H 2950 6500 50  0001 C CNN
 F 3 "" H 2950 6500 50  0001 C CNN
 	1    2950 6300
@@
 F 0 "L3" V 21000 900 50  0000 C CNN
 F 1 "10uH" V 20900 900 50  0000 C CNN
-F 2 "Inductor_SMD:L_Coilcraft_XxL4040" H 20800 1050 50  0001 C CNN
+F 2 "Womo-Lin:MWSA0603" H 20800 1050 50  0001 C CNN
 F 3 "~" H 20800 1050 50  0001 C CNN
 	1    20800 1050

Commit message: PCB Prototypen Produktions Stand
Parts:
- removed C60, C61: 2u2, Capacitor_SMD:C_1210_3225Metric, symbol Displayunit-rescue:C-Device
- C62, C63: footprint Capacitor_SMD:C_1210_3225Metric -> Capacitor_SMD:C_0603_1608Metric
Changed lines of the file:
@@
 	1    0    0    -1
 $EndComp
-Wire Wire Line
-	17000 4100 17350 4100
 $Comp
 L Displayunit-rescue:R-Device R?
@@
 $Comp
 L Displayunit-rescue:C-Device C?
-U 1 1 60BFC24B
-P 17350 4250
-AR Path="/5C8BBC9A/60BFC24B" Ref="C?"  Part="1"
-AR Path="/5E0C5EEA/60BFC24B" Ref="C?"  Part="1"
-AR Path="/5D80EC74/60BFC24B" Ref="C?"  Part="1"
-AR Path="/5D80E6E8/60BFC24B" Ref="C?"  Part="1"
-AR Path="/60BFC24B" Ref="C61"  Part="1"
-F 0 "C61" H 17350 4650 50  0000 L CNN
-F 1 "2u2" H 17350 4550 50  0000 L CNN
-F 2 "Capacitor_SMD:C_1210_3225Metric" H 17388 4100 50  0001 C CNN
-F 3 "~" H 17350 4250 50  0001 C CNN
-	1    17350 4250
-	1    0    0    -1
-$EndComp
-$Comp
-L Displayunit-rescue:C-Device C?
 U 1 1 60C7DAA7
 P 17700 4250
@@
 F 0 "C63" H 17650 4650 50  0000 L CNN
 F 1 "100n" H 17650 4550 50  0000 L CNN
-F 2 "Capacitor_SMD:C_1210_3225Metric" H 17738 4100 50  0001 C CNN
+F 2 "Capacitor_SMD:C_0603_1608Metric" H 17738 4100 50  0001 C CNN
 F 3 "~" H 17700 4250 50  0001 C CNN
 	1    17700 4250
@@
 F 0 "C62" H 17650 1900 50  0000 L CNN
 F 1 "100n" H 17650 1800 50  0000 L CNN
-F 2 "Capacitor_SMD:C_1210_3225Metric" H 17738 1400 50  0001 C CNN
+F 2 "Capacitor_SMD:C_0603_1608Metric" H 17738 1400 50  0001 C CNN
 F 3 "~" H 17700 1550 50  0001 C CNN
 	1    17700 1550
 	1    0    0    -1
 $EndComp
-$Comp
-L Displayunit-rescue:C-Device C?
-U 1 1 60D8104E
-P 17350 1550
-AR Path="/5C8BBC9A/60D8104E" Ref="C?"  Part="1"
-AR Path="/5E0C5EEA/60D8104E" Ref="C?"  Part="1"
-AR Path="/5D80EC74/60D8104E" Ref="C?"  Part="1"
-AR Path="/5D80E6E8/60D8104E" Ref="C?"  Part="1"
-AR Path="/60D8104E" Ref="C60"  Part="1"
-F 0 "C60" H 17300 1900 50  0000 L CNN
-F 1 "2u2" H 17300 1800 50  0000 L CNN
-F 2 "Capacitor_SMD:C_1210_3225Metric" H 17388 1400 50  0001 C CNN
-F 3 "~" H 17350 1550 50  0001 C CNN
-	1    17350 1550
-	1    0    0    -1
-$EndComp
-Connection ~ 17350 1400
-Wire Wire Line
-	17350 1400 17000 1400
-Connection ~ 17350 4100
 Wire Wire Line
 	18050 4100 17700 4100
 Connection ~ 18050 4100
-Wire Wire Line
-	17350 4100 17700 4100
 Connection ~ 17700 4100
-Wire Wire Line
-	17350 1400 17700 1400
 Wire Wire Line
 	17700 1400 18050 1400
@@
 $Comp
 L Displayunit-rescue:GND-power #PWR?
-U 1 1 61118551
-P 17350 1700
-AR Path="/5C8BBC9A/61118551" Ref="#PWR?"  Part="1"
-AR Path="/5E0C5EEA/61118551" Ref="#PWR?"  Part="1"
-AR Path="/5D80EC74/61118551" Ref="#PWR?"  Part="1"
-AR Path="/5D80E6E8/61118551" Ref="#PWR?"  Part="1"
-AR Path="/61118551" Ref="#PWR0132"  Part="1"
-F 0 "#PWR0132" H 17350 1450 50  0001 C CNN
-F 1 "GND" H 17350 1500 50  0000 C CNN
-F 2 "" H 17350 1700 50  0001 C CNN
-F 3 "" H 17350 1700 50  0001 C CNN
-	1    17350 1700
-	1    0    0    -1
-$EndComp
-$Comp
-L Displayunit-rescue:GND-power #PWR?
-U 1 1 6119AFF7
-P 17350 4400
-AR Path="/5C8BBC9A/6119AFF7" Ref="#PWR?"  Part="1"
-AR Path="/5E0C5EEA/6119AFF7" Ref="#PWR?"  Part="1"
-AR Path="/5D80EC74/6119AFF7" Ref="#PWR?"  Part="1"
-AR Path="/5D80E6E8/6119AFF7" Ref="#PWR?"  Part="1"
-AR Path="/6119AFF7" Ref="#PWR0133"  Part="1"
-F 0 "#PWR0133" H 17350 4150 50  0001 C CNN
-F 1 "GND" H 17350 4200 50  0000 C CNN
-F 2 "" H 17350 4400 50  0001 C CNN
-F 3 "" H 17350 4400 50  0001 C CNN
-	1    17350 4400
-	1    0    0    -1
-$EndComp
-$Comp
-L Displayunit-rescue:GND-power #PWR?
 U 1 1 6121D9DF
 P 17700 4400
@@
 Wire Wire Line
 	10150 2300 10900 2300
+Wire Wire Line
+	17000 4100 17700 4100
+Wire Wire Line
+	17000 1400 17700 1400
 $EndSCHEMATC

Commit message: Display Board: Fix JTAG REF, LED Treiber > TPS61165, Spulen zurück auf XAL4040 Footprint, Auf Version 2.0 gehoben
Parts:
- removed R6: 100K, Resistor_SMD:R_0603_1608Metric, symbol Displayunit-rescue:R-Device
- removed U3: STLD40D, Package_DFN_QFN:DFN-8-1EP_3x3mm_P0.65mm_EP1.55x2.4mm, symbol Womo-Lin:STLD40D
- added IC4: TPS61165DRVR, Package_SON:WSON-6-1EP_2x2mm_P0.65mm_EP1x1.6mm, symbol opendous:TPS61160
- C1, C22, C31, C5, C55: value 1uF -> 1u
- C15: value 10uF -> 10u
- C16: value 10nF -> 10n
- C2, C28, C30, C34, C45, C48, C50: value 100nF -> 100n
- C43: value 10n -> 220n
- C46, C49: value 47u -> 10u
- C47: value 4u7 -> 1u
- D4: value B250 -> B260A-13-F
- L1: value 4uH7 -> 10uH; footprint Womo-Lin:MWSA0603 -> Inductor_SMD:L_Coilcraft_XxL4020
- L2: value L_Core_Ferrite -> 2uH2; footprint Womo-Lin:MWSA0603 -> Inductor_SMD:L_Coilcraft_XxL4020
- L3, L4: footprint Womo-Lin:MWSA0603 -> Inductor_SMD:L_Coilcraft_XxL4020
- R10: value 10R 1% -> 1R1; footprint Resistor_SMD:R_0603_1608Metric -> Resistor_SMD:R_1206_3216Metric
- R13: value 32k4 -> 10K
Connections:
- net +3V3: now also J4.1 (VTREF)
- net LCD_BL_CTRL: now also IC4.5 (CTRL)
- net LCD_LED-A: no longer C43.1
- net LCD_LED-K: now also R10.1, IC4.1 (FB); no longer C27.2, C29.2, C35.2, C43.2, FB2.2, R10.2
- net at D4.2 (A), L1.2: now also IC4.4 (SW)
- net at C27.1, C29.1, C35.1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: now also IC4.6 (VIN)
- new net: C43.1, IC4.2 (COMP)
- new net: C27.2, C29.2, C35.2, C43.2, FB2.2, IC4.3 (GND), IC4.7 (GND-Pad), R10.2
Other:
- moved on the sheet: C43, C47, R10, R13
