File: Hardware/Displayunit/Displayunit.sch (KiCad schematic (older format))
At the start: 132 parts, among them IC1 TSC2007, IC2 MX25LM51245GXDI00, IC3 IS66WVH8M8BLL-100B1LI_0, IC4 TPS61165DRVR, J1 615008138221, J2 615008138221, J3 54104-4031, J4 Conn_ARM_JTAG_SWD_20, J5 52271-0679, J6 Conn_02x06_Odd_Even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

Commit message: Fix Lib gedrehte FPC Stecker, 10 Pin FPC hinzu gefügt (Buydisplay.com Alternative) Displayboard RS485 und CAN Option hinzu. Beginn Änderung Layout.
Parts:
- added C60: 100n, Capacitor_SMD:C_0603_1608Metric, symbol Displayunit-rescue:C-Device
- added D8: NUP2105L, Package_TO_SOT_SMD:SOT-23, symbol Displayunit-rescue:D_TVS_x2_AAC-Device
- added FB11, FB12: 100R, Inductor_SMD:L_0603_1608Metric, symbol Displayunit-rescue:Ferrite_Bead_Small-Device
- added J10: ER-CON10HT-1, Womo-Lin:ER-CON10HT-1, symbol Womo-Lin:ER-CON10HT-1
- added R23, R24, R25, R6: 0R, Resistor_SMD:R_0603_1608Metric, symbol Displayunit-rescue:R-Device
- added R26: 120R, Resistor_SMD:R_0603_1608Metric, symbol Displayunit-rescue:R-Device
- added U3: HD588E, Package_SO:SOIC-8_3.9x4.9mm_P1.27mm, symbol Interface_UART:ST485EBDR
- IC4: footprint Package_SON:WSON-6-1EP_2x2mm_P0.65mm_EP1x1.6mm -> Package_SON:WSON-6-1EP_2x2mm_P0.65mm_EP1x1.6mm_ThermalVias
- L1, L2, L3, L4: footprint Inductor_SMD:L_Coilcraft_XxL4020 -> Womo-Lin:MWSA0603
- U7: footprint Package_SO:SO-8_3.9x4.9mm_P1.27mm -> Package_SO:SO-8_5.3x6.2mm_P1.27mm
Connections:
- net +3.3VA: now also J10.7, J10.9
- net +3V3: now also C60.1, U3.8 (VCC); no longer C10.1, C17.1, C18.2, C19.2, C20.2, U1.108 (VDDUSB), U1.131 (VDDIO2), U1.30 (VDDA), U1.68 (VDD), U1.73 (VDDDSI)
- net EXT_1: now also U1.65 (PB10); no longer U1.139 (PB8)
- net EXT_2: now also U1.66 (PB11); no longer U1.140 (PB9)
- net EXT_3: now also U1.69 (PB12); no longer U1.65 (PB10)
- net GND: now also C60.2, D8.3 (common), J10.1, J10.10, J10.8, U3.5 (GND); no longer IC1.13 (A1), IC1.14 (A0)
- net I2C2_SCL: now also J10.3
- net I2C2_SDA: now also J10.2
- net TOUCH_INT: now also J10.5
- net TOUCH_RESET: now also J10.4
- net USART1_RX: now also R24.2; no longer U6.4 (R)
- net USART1_TX: now also R23.2; no longer U6.1 (D)
- net USART2_CTS_NSS: now reaches U1.31 (PA0)
- net USART2_CTS_NSS: now also U3.1 (RO)
- net USART2_RTS_DE: now reaches U1.32 (PA1)
- net USART2_RTS_DE: now also U3.2 (~RE)
- net USART2_TX: now reaches U1.33 (PA2)
- net USART2_TX: now also U3.3 (DE)
- net USART2_RX: now reaches U1.34 (PA3)
- net USART2_RX: now also U3.4 (DI)
- net at J1.3: now also J1.6, J2.6, FB11.1
- net at J2.3: now also FB12.1
- new net: R23.1, R6.1, U6.1 (D)
- new net: R24.1, R25.1, U6.4 (R)
- new net: C17.1, C18.2, C19.2, C20.2, U1.131 (VDDIO2), U1.30 (VDDA), U1.73 (VDDDSI)
- new net: IC1.13 (A1), IC1.14 (A0)
- new net: D8.1 (A1), FB12.2, R26.2, U3.6 (A)
- new net: D8.2 (A2), FB11.2, R26.1, U3.7 (B)
- new net CAN1_RX: R25.2, U1.139 (PB8)
- new net CAN1_TX: R6.2, U1.140 (PB9)
- no-connect marks 26 -> 23
Other:
- moved on the sheet: C31, J5, J8, U2

Commit message: Fix Womolin Lib, ein paar Bauteile fehlte Lötstopmaske. Displayboard stand zweite Prototyp Bestellung.
Parts:
- removed C20: 100n, Capacitor_SMD:C_0603_1608Metric, symbol Displayunit-rescue:C-Device
- C1, C15, C22, C31, C37, C55: footprint Capacitor_SMD:C_1210_3225Metric -> Capacitor_SMD:C_1206_3216Metric
- C17: value 10uF -> 10u; footprint Capacitor_SMD:C_1210_3225Metric -> Capacitor_SMD:C_1206_3216Metric
- C26: value 1uF -> 1u; footprint Capacitor_SMD:C_1210_3225Metric -> Capacitor_SMD:C_1206_3216Metric
- C42: value 22uF -> 22u
- C44: value 47u -> 22u
- FB5, FB6, FB7, FB8, FB9: value BLM18PG121SN1D -> 100r
- L1, L3, L4: footprint Womo-Lin:MWSA0603 -> Womo-Lin:MWSA0503
- R1, R13, R15, R2, R3, R4: value 10K -> 10k
- R14: value 31K6 -> 31k6
Connections:
- net +3V3: now also C10.1, C17.1, C18.2, C19.2, U1.108 (VDDUSB), U1.131 (VDDIO2), U1.30 (VDDA), U1.68 (VDD), U1.73 (VDDDSI)
- net GND: now also IC1.13 (A1), IC1.14 (A0)
- net at FB11.1, J1.6, J2.6: no longer J1.3
- net at FB12.1, J2.3: now also J1.3
